File: pc slots.sch (KiCad schematic (older format))
At the start: 0 parts

Commit message: Use correct source rev6. mostly all schematics done for first pass...
Parts:
- added C700, C702, C703, C704, C705: 0.22uF, symbol Device:C
- added C701: 22uF 16V, symbol Device:CP
- added C711, C713, C714, C716, C717, C719, C720, C722, C726, C728, C730, C732, C734, C736, C738, C740, C742, C744, C746, C748, C750, C752, C754, C756, C758, C760, C762, C764, C766, C768, C770, C776, C778, C780, C782, C784, C786, C787, C789, C790, C791, C793, C794, C796: 1000pF, symbol Device:C_Small
- added CN700, CN701, CN702, CN703: IBM_8_BIT_EXPANSION_BUS, symbol amiga_customs:IBM_8_BIT_EXPANSION_BUS
- added CN704, CN705, CN706, CN707: IBM_16_BIT_EXTENDED_BUS, symbol amiga_customs:IBM_16_BIT_EXTENDED_BUS
- added RP700, RP701, RP702, RP703, RP704: 1k, Resistor_THT:R_Array_SIP10, symbol Device:R_Network09
- added RP705: 4.7k, Resistor_THT:R_Array_SIP10, symbol Device:R_Network09
Connections:
- new net: C711.1, RP700.10 (R9)
- new net: C713.1, RP700.9 (R8)
- new net: C714.1, RP700.8 (R7)
- new net: C716.1, RP700.7 (R6)
- new net: C717.1, RP700.6 (R5)
- new net: C719.1, RP700.5 (R4)
- new net: C720.1, RP700.4 (R3)
- new net: C722.1, RP700.3 (R2)
- new net: C726.1, RP700.2 (R1)
- new net: C728.1, RP701.10 (R9)
- new net: C744.1, RP701.2 (R1)
- new net: C742.1, RP701.3 (R2)
- new net: C740.1, RP701.4 (R3)
- new net: C738.1, RP701.5 (R4)
- new net: C736.1, RP701.6 (R5)
- new net: C734.1, RP701.7 (R6)
- new net: C732.1, RP701.8 (R7)
- new net: C730.1, RP701.9 (R8)
- new net: C746.1, RP702.10 (R9)
- new net: C791.1, RP702.2 (R1)
- new net: C790.1, RP702.3 (R2)
- new net: C758.1, RP702.4 (R3)
- new net: C756.1, RP702.5 (R4)
- new net: C754.1, RP702.6 (R5)
- new net: C752.1, RP702.7 (R6)
- new net: C750.1, RP702.8 (R7)
- new net: C748.1, RP702.9 (R8)
- new net: C793.1, RP703.10 (R9)
- new net: C770.1, RP703.2 (R1)
- new net: C768.1, RP703.3 (R2)
- new net: C766.1, RP703.4 (R3)
- new net: C764.1, RP703.5 (R4)
- new net: C762.1, RP703.6 (R5)
- new net: C760.1, RP703.7 (R6)
- new net: C796.1, RP703.8 (R7)
- new net: C794.1, RP703.9 (R8)
- new net: C789.1, RP704.2 (R1)
- new net: C787.1, RP704.3 (R2)
- new net: C786.1, RP704.4 (R3)
- new net: C784.1, RP704.5 (R4)
- new net: C782.1, RP704.6 (R5)
- new net: C780.1, RP704.7 (R6)
- new net: C778.1, RP704.8 (R7)
- new net: C776.1, RP704.9 (R8)
- new net +12V: C704.1, CN700.~ (B9), CN701.~ (B9), CN702.~ (B9), CN703.~ (B9)
- new net +5V: C700.1, C701.1, C705.1, CN700.~ (B9), CN701.~ (B9), CN702.~ (B9), CN703.~ (B9), CN704.~ (D9), CN705.~ (D9), CN706.~ (D9), CN707.~ (D9), RP705.1 (common)
- new net -12V: C703.1, CN700.~ (B9), CN701.~ (B9), CN702.~ (B9), CN703.~ (B9)
- new net -5V: C702.1, CN700.~ (B9), CN701.~ (B9), CN702.~ (B9), CN703.~ (B9)
- new net A0: C793.2, CN700.~ (B9), CN701.~ (B9), CN702.~ (B9), CN703.~ (B9)
- new net A1: C791.2, CN700.~ (B9), CN701.~ (B9), CN702.~ (B9), CN703.~ (B9)
- new net A10: C744.2, CN700.~ (B9), CN701.~ (B9), CN702.~ (B9), CN703.~ (B9)
- new net A11: C742.2, CN700.~ (B9), CN701.~ (B9), CN702.~ (B9), CN703.~ (B9)
- new net A12: C740.2, CN700.~ (B9), CN701.~ (B9), CN702.~ (B9), CN703.~ (B9)
- new net A13: C738.2, CN700.~ (B9), CN701.~ (B9), CN702.~ (B9), CN703.~ (B9)
- new net A14: C736.2, CN700.~ (B9), CN701.~ (B9), CN702.~ (B9), CN703.~ (B9)
- new net A15: C734.2, CN700.~ (B9), CN701.~ (B9), CN702.~ (B9), CN703.~ (B9)
- new net A16: C732.2, CN700.~ (B9), CN701.~ (B9), CN702.~ (B9), CN703.~ (B9)
- new net A17: C730.2, CN700.~ (B9), CN701.~ (B9), CN702.~ (B9), CN703.~ (B9)
- new net A18: C728.2, CN700.~ (B9), CN701.~ (B9), CN702.~ (B9), CN703.~ (B9)
- new net A19: C726.2, CN700.~ (B9), CN701.~ (B9), CN702.~ (B9), CN703.~ (B9)
- new net A2: C790.2, CN700.~ (B9), CN701.~ (B9), CN702.~ (B9), CN703.~ (B9)
- new net A3: C758.2, CN700.~ (B9), CN701.~ (B9), CN702.~ (B9), CN703.~ (B9)
- new net A4: C756.2, CN700.~ (B9), CN701.~ (B9), CN702.~ (B9), CN703.~ (B9)
- new net A5: C754.2, CN700.~ (B9), CN701.~ (B9), CN702.~ (B9), CN703.~ (B9)
- new net A6: C752.2, CN700.~ (B9), CN701.~ (B9), CN702.~ (B9), CN703.~ (B9)
- new net A7: C750.2, CN700.~ (B9), CN701.~ (B9), CN702.~ (B9), CN703.~ (B9)
- new net A8: C748.2, CN700.~ (B9), CN701.~ (B9), CN702.~ (B9), CN703.~ (B9)
- new net A9: C746.2, CN700.~ (B9), CN701.~ (B9), CN702.~ (B9), CN703.~ (B9)
- new net AEN: CN700.~ (B9), CN701.~ (B9), CN702.~ (B9), CN703.~ (B9)
- new net ALE: CN700.~ (B9), CN701.~ (B9), CN702.~ (B9), CN703.~ (B9)
- new net CD_SEL: CN700.~ (B9), CN701.~ (B9), CN702.~ (B9), CN703.~ (B9)
- new net CLK: CN700.~ (B9), CN701.~ (B9), CN702.~ (B9), CN703.~ (B9)
- new net D0: C722.2, CN700.~ (B9), CN701.~ (B9), CN702.~ (B9), CN703.~ (B9)
- new net D1: C720.2, CN700.~ (B9), CN701.~ (B9), CN702.~ (B9), CN703.~ (B9)
- new net D10: C780.2, CN704.~ (D9), CN705.~ (D9), CN706.~ (D9), CN707.~ (D9)
- new net D11: C782.2, CN704.~ (D9), CN705.~ (D9), CN706.~ (D9), CN707.~ (D9)
- new net D12: C784.2, CN704.~ (D9), CN705.~ (D9), CN706.~ (D9), CN707.~ (D9)
- new net D13: C786.2, CN704.~ (D9), CN705.~ (D9), CN706.~ (D9), CN707.~ (D9)
- new net D14: C787.2, CN704.~ (D9), CN705.~ (D9), CN706.~ (D9), CN707.~ (D9)
- new net D15: C789.2, CN704.~ (D9), CN705.~ (D9), CN706.~ (D9), CN707.~ (D9)
- new net D2: C719.2, CN700.~ (B9), CN701.~ (B9), CN702.~ (B9), CN703.~ (B9)
- new net D3: C717.2, CN700.~ (B9), CN701.~ (B9), CN702.~ (B9), CN703.~ (B9)
- new net D4: C716.2, CN700.~ (B9), CN701.~ (B9), CN702.~ (B9), CN703.~ (B9)
- new net D5: C714.2, CN700.~ (B9), CN701.~ (B9), CN702.~ (B9), CN703.~ (B9)
- new net D6: C713.2, CN700.~ (B9), CN701.~ (B9), CN702.~ (B9), CN703.~ (B9)
- new net D7: C711.2, CN700.~ (B9), CN701.~ (B9), CN702.~ (B9), CN703.~ (B9)
- new net D8: C776.2, CN704.~ (D9), CN705.~ (D9), CN706.~ (D9), CN707.~ (D9)
- new net D9: C778.2, CN704.~ (D9), CN705.~ (D9), CN706.~ (D9), CN707.~ (D9)
- new net DRQ0: CN704.~ (D9), CN705.~ (D9), CN706.~ (D9), CN707.~ (D9)
- new net DRQ1: CN700.~ (B9), CN701.~ (B9), CN702.~ (B9), CN703.~ (B9)
- new net DRQ2: CN700.~ (B9), CN701.~ (B9), CN702.~ (B9), CN703.~ (B9)
- new net DRQ3: CN700.~ (B9), CN701.~ (B9), CN702.~ (B9), CN703.~ (B9)
- new net DRQ5: CN704.~ (D9), CN705.~ (D9), CN706.~ (D9), CN707.~ (D9)
- new net DRQ6: CN704.~ (D9), CN705.~ (D9), CN706.~ (D9), CN707.~ (D9)
- new net DRQ7: CN704.~ (D9), CN705.~ (D9), CN706.~ (D9), CN707.~ (D9)
- new net GND: C700.2, C701.2, C702.2, C703.2, C704.2, C705.2, CN700.~ (B9), CN701.~ (B9), CN702.~ (B9), CN703.~ (B9), CN704.~ (D9), CN705.~ (D9), CN706.~ (D9), CN707.~ (D9), RP700.1 (common), RP701.1 (common), RP702.1 (common), RP703.1 (common), RP704.1 (common)
- new net IOREADY: CN700.~ (B9), CN701.~ (B9), CN702.~ (B9), CN703.~ (B9)
- new net IRQ10: CN704.~ (D9), CN705.~ (D9), CN706.~ (D9), CN707.~ (D9)
- new net IRQ11: CN704.~ (D9), CN705.~ (D9), CN706.~ (D9), CN707.~ (D9)
- new net IRQ12: CN704.~ (D9), CN705.~ (D9), CN706.~ (D9), CN707.~ (D9)
- new net IRQ14: CN704.~ (D9), CN705.~ (D9), CN706.~ (D9), CN707.~ (D9)
- new net IRQ15: CN704.~ (D9), CN705.~ (D9), CN706.~ (D9), CN707.~ (D9)
- new net IRQ2: CN700.~ (B9), CN701.~ (B9), CN702.~ (B9), CN703.~ (B9)
- new net IRQ3: CN700.~ (B9), CN701.~ (B9), CN702.~ (B9), CN703.~ (B9)
- new net IRQ4: CN700.~ (B9), CN701.~ (B9), CN702.~ (B9), CN703.~ (B9)
- new net IRQ5: CN700.~ (B9), CN701.~ (B9), CN702.~ (B9), CN703.~ (B9)
- new net IRQ6: CN700.~ (B9), CN701.~ (B9), CN702.~ (B9), CN703.~ (B9)
- new net IRQ7: CN700.~ (B9), CN701.~ (B9), CN702.~ (B9), CN703.~ (B9)
- new net LA17: C770.2, CN704.~ (D9), CN705.~ (D9), CN706.~ (D9), CN707.~ (D9)
- new net LA18: C768.2, CN704.~ (D9), CN705.~ (D9), CN706.~ (D9), CN707.~ (D9)
- new net LA19: C766.2, CN704.~ (D9), CN705.~ (D9), CN706.~ (D9), CN707.~ (D9)
- new net LA20: C764.2, CN704.~ (D9), CN705.~ (D9), CN706.~ (D9), CN707.~ (D9)
- new net LA21: C762.2, CN704.~ (D9), CN705.~ (D9), CN706.~ (D9), CN707.~ (D9)
- new net LA22: C760.2, CN704.~ (D9), CN705.~ (D9), CN706.~ (D9), CN707.~ (D9)
- new net LA23: C796.2, CN704.~ (D9), CN705.~ (D9), CN706.~ (D9), CN707.~ (D9)
- new net OSC: CN700.~ (B9), CN701.~ (B9), CN702.~ (B9), CN703.~ (B9)
- new net RESDRV: CN700.~ (B9), CN701.~ (B9), CN702.~ (B9), CN703.~ (B9)
- new net SHBE: C794.2, CN704.~ (D9), CN705.~ (D9), CN706.~ (D9), CN707.~ (D9)
- new net SHITHEAD: CN700.~ (B9), CN701.~ (B9), CN702.~ (B9), CN703.~ (B9)
- new net TC: CN700.~ (B9), CN701.~ (B9), CN702.~ (B9), CN703.~ (B9)
- new net _DACK0: CN704.~ (D9), CN705.~ (D9), CN706.~ (D9), CN707.~ (D9)
- new net _DACK1: CN700.~ (B9), CN701.~ (B9), CN702.~ (B9), CN703.~ (B9)
- new net _DACK2: CN700.~ (B9), CN701.~ (B9), CN702.~ (B9), CN703.~ (B9)
- new net _DACK3: CN700.~ (B9), CN701.~ (B9), CN702.~ (B9), CN703.~ (B9)
- new net _DACK5: CN704.~ (D9), CN705.~ (D9), CN706.~ (D9), CN707.~ (D9)
- new net _DACK6: CN704.~ (D9), CN705.~ (D9), CN706.~ (D9), CN707.~ (D9)
- new net _DACK7: CN704.~ (D9), CN705.~ (D9), CN706.~ (D9), CN707.~ (D9)
- new net _IO16: CN704.~ (D9), CN705.~ (D9), CN706.~ (D9), CN707.~ (D9), RP705.8 (R7)
- new net _IOCHK: CN700.~ (B9), CN701.~ (B9), CN702.~ (B9), CN703.~ (B9)
- new net _IOR: CN700.~ (B9), CN701.~ (B9), CN702.~ (B9), CN703.~ (B9), RP705.4 (R3)
- new net _IOW: CN700.~ (B9), CN701.~ (B9), CN702.~ (B9), CN703.~ (B9), RP705.5 (R4)
- new net _MASTER: CN704.~ (D9), CN705.~ (D9), CN706.~ (D9), CN707.~ (D9)
- new net _MEM16: CN704.~ (D9), CN705.~ (D9), CN706.~ (D9), CN707.~ (D9), RP705.9 (R8)
- new net _MEMR: CN700.~ (B9), CN701.~ (B9), CN702.~ (B9), CN703.~ (B9), CN704.~ (D9), CN705.~ (D9), CN706.~ (D9), CN707.~ (D9), RP705.2 (R1), RP705.3 (R2), RP705.6 (R5)
- new net _MEMW: CN700.~ (B9), CN701.~ (B9), CN702.~ (B9), CN703.~ (B9), RP705.7 (R6)
- no-connect marks 0 -> 2
Other:
- note added: "Note: R6 PCB - C789 is noted C788 and connected to _MASTER instead of D15"
