File: pc slots.sch (KiCad schematic (older format))
At the start: 64 parts, among them CN700 IBM_8_BIT_EXPANSION_BUS, CN701 IBM_8_BIT_EXPANSION_BUS, CN702 IBM_8_BIT_EXPANSION_BUS, CN703 IBM_8_BIT_EXPANSION_BUS, CN704 IBM_16_BIT_EXTENDED_BUS, CN705 IBM_16_BIT_EXTENDED_BUS, CN706 IBM_16_BIT_EXTENDED_BUS, CN707 IBM_16_BIT_EXTENDED_BUS

Commit message: Associate more components
Parts:
- C701: footprint (none) -> Capacitor_THT:CP_Radial_D8.0mm_P5.00mm
Changed lines of the file:
@@
 F 0 "C701" H 1968 9046 50  0000 L CNN
 F 1 "22uF 16V" H 1968 8955 50  0000 L CNN
-F 2 "" H 1888 8850 50  0001 C CNN
+F 2 "Capacitor_THT:CP_Radial_D8.0mm_P5.00mm" H 1888 8850 50  0001 C CNN
 F 3 "~" H 1850 9000 50  0001 C CNN
 	1    1850 9000

Commit message: Associate ISA slots
Parts:
- CN700, CN701, CN702, CN703: footprint (none) -> ISA:ISA8
- CN704, CN705, CN706, CN707: footprint (none) -> ISA:ISA16
Changed lines of the file:
@@
 F 0 "CN700" H 4450 3283 50  0000 C CNN
 F 1 "IBM_8_BIT_EXPANSION_BUS" H 4450 3284 50  0001 C CNN
-F 2 "" H 4450 3250 50  0001 C CNN
+F 2 "ISA:ISA8" H 4450 3250 50  0001 C CNN
 F 3 "" H 4450 3250 50  0001 C CNN
 	1    4450 3200
@@
 F 0 "CN704" H 4475 10033 50  0000 C CNN
 F 1 "IBM_16_BIT_EXTENDED_BUS" H 4475 10034 50  0001 C CNN
-F 2 "" H 4500 10000 50  0001 C CNN
+F 2 "ISA:ISA16" H 4500 10000 50  0001 C CNN
 F 3 "" H 4500 10000 50  0001 C CNN
 	1    4500 9950
@@
 F 0 "CN701" H 7100 3283 50  0000 C CNN
 F 1 "IBM_8_BIT_EXPANSION_BUS" H 7100 3284 50  0001 C CNN
-F 2 "" H 7100 3250 50  0001 C CNN
+F 2 "ISA:ISA8" H 7100 3250 50  0001 C CNN
 F 3 "" H 7100 3250 50  0001 C CNN
 	1    7100 3200
@@
 F 0 "CN705" H 7125 10033 50  0000 C CNN
 F 1 "IBM_16_BIT_EXTENDED_BUS" H 7125 10034 50  0001 C CNN
-F 2 "" H 7150 10000 50  0001 C CNN
+F 2 "ISA:ISA16" H 7150 10000 50  0001 C CNN
 F 3 "" H 7150 10000 50  0001 C CNN
 	1    7150 9950
@@
 F 0 "CN702" H 9600 3283 50  0000 C CNN
 F 1 "IBM_8_BIT_EXPANSION_BUS" H 9600 3284 50  0001 C CNN
-F 2 "" H 9600 3250 50  0001 C CNN
+F 2 "ISA:ISA8" H 9600 3250 50  0001 C CNN
 F 3 "" H 9600 3250 50  0001 C CNN
 	1    9600 3200
@@
 F 0 "CN706" H 9625 10033 50  0000 C CNN
 F 1 "IBM_16_BIT_EXTENDED_BUS" H 9625 10034 50  0001 C CNN
-F 2 "" H 9650 10000 50  0001 C CNN
+F 2 "ISA:ISA16" H 9650 10000 50  0001 C CNN
 F 3 "" H 9650 10000 50  0001 C CNN
 	1    9650 9950
@@
 F 0 "CN703" H 12050 3283 50  0000 C CNN
 F 1 "IBM_8_BIT_EXPANSION_BUS" H 12050 3284 50  0001 C CNN
-F 2 "" H 12050 3250 50  0001 C CNN
+F 2 "ISA:ISA8" H 12050 3250 50  0001 C CNN
 F 3 "" H 12050 3250 50  0001 C CNN
 	1    12050 3200
@@
 F 0 "CN707" H 12075 10033 50  0000 C CNN
 F 1 "IBM_16_BIT_EXTENDED_BUS" H 12075 10034 50  0001 C CNN
-F 2 "" H 12100 10000 50  0001 C CNN
+F 2 "ISA:ISA16" H 12100 10000 50  0001 C CNN
 F 3 "" H 12100 10000 50  0001 C CNN
 	1    12100 9950

Commit message: Update footprints
Parts:
- C700, C702, C703, C704, C705, C711, C713, C714, C716, C717, C719, C720, C722, C726, C728, C730, C732, C734, C736, C738, C740, C742, C744, C746, C748, C750, C752, C754, C756, C758, C760, C762, C764, C766, C768, C770, C776, C778, C780, C782, C784, C786, C787, C789, C790, C791, C793, C794, C796: footprint (none) -> Capacitor_THT:C_Rect_L11.0mm_W2.8mm_P10.00mm_MKT

Commit message: hmmmm
Parts:
- CN700, CN701, CN702, CN703: symbol amiga_customs:IBM_8_BIT_EXPANSION_BUS -> amiga2000-rescue:IBM_8_BIT_EXPANSION_BUS-amiga_customs
Connections:
- net A0: now also CN700.63 (A31), CN701.63 (A31), CN702.63 (A31), CN703.63 (A31); no longer CN700.62 (A31), CN701.62 (A31), CN702.62 (A31), CN703.62 (A31)
- net GND: now also CN700.62 (B31), CN701.62 (B31), CN702.62 (B31), CN703.62 (B31); no longer CN700.61 (B31), CN701.61 (B31), CN702.61 (B31), CN703.61 (B31)
Changed lines of the file:
@@
 D7
 $Comp
-L amiga_customs:IBM_8_BIT_EXPANSION_BUS CN700
+L amiga2000-rescue:IBM_8_BIT_EXPANSION_BUS-amiga_customs CN700
 U 1 1 682158CF
 P 4450 3200
+AR Path="/682158CF" Ref="CN700"  Part="1"
+AR Path="/5CEA7188/682158CF" Ref="CN700"  Part="1"
 F 0 "CN700" H 4450 3283 50  0000 C CNN
 F 1 "IBM_8_BIT_EXPANSION_BUS" H 4450 3284 50  0001 C CNN
@@
 $EndComp
 $Comp
-L amiga_customs:IBM_8_BIT_EXPANSION_BUS CN701
+L amiga2000-rescue:IBM_8_BIT_EXPANSION_BUS-amiga_customs CN701
 U 1 1 682288F0
 P 7100 3200
+AR Path="/682288F0" Ref="CN701"  Part="1"
+AR Path="/5CEA7188/682288F0" Ref="CN701"  Part="1"
 F 0 "CN701" H 7100 3283 50  0000 C CNN
 F 1 "IBM_8_BIT_EXPANSION_BUS" H 7100 3284 50  0001 C CNN
@@
 $EndComp
 $Comp
-L amiga_customs:IBM_8_BIT_EXPANSION_BUS CN702
+L amiga2000-rescue:IBM_8_BIT_EXPANSION_BUS-amiga_customs CN702
 U 1 1 6822BC0D
 P 9600 3200
+AR Path="/6822BC0D" Ref="CN702"  Part="1"
+AR Path="/5CEA7188/6822BC0D" Ref="CN702"  Part="1"
 F 0 "CN702" H 9600 3283 50  0000 C CNN
 F 1 "IBM_8_BIT_EXPANSION_BUS" H 9600 3284 50  0001 C CNN
@@
 $EndComp
 $Comp
-L amiga_customs:IBM_8_BIT_EXPANSION_BUS CN703
+L amiga2000-rescue:IBM_8_BIT_EXPANSION_BUS-amiga_customs CN703
 U 1 1 6822E618
 P 12050 3200
+AR Path="/6822E618" Ref="CN703"  Part="1"
+AR Path="/5CEA7188/6822E618" Ref="CN703"  Part="1"
 F 0 "CN703" H 12050 3283 50  0000 C CNN
 F 1 "IBM_8_BIT_EXPANSION_BUS" H 12050 3284 50  0001 C CNN

Commit message: fix fuckup
Parts:
- CN700, CN701, CN702, CN703: symbol amiga2000-rescue:IBM_8_BIT_EXPANSION_BUS-amiga_customs -> amiga_customs:IBM_8_BIT_EXPANSION_BUS
Connections:
- net A0: now also CN700.62 (A31), CN701.62 (A31), CN702.62 (A31), CN703.62 (A31); no longer CN700.63 (A31), CN701.63 (A31), CN702.63 (A31), CN703.63 (A31)
- net GND: now also CN700.61 (B31), CN701.61 (B31), CN702.61 (B31), CN703.61 (B31); no longer CN700.62 (B31), CN701.62 (B31), CN702.62 (B31), CN703.62 (B31)

Commit message: Make caps footprint smaller
Parts:
- C700, C702, C703, C704, C705, C711, C713, C714, C716, C717, C719, C720, C722, C726, C728, C730, C732, C734, C736, C738, C740, C742, C744, C746, C748, C750, C752, C754, C756, C758, C760, C762, C764, C766, C768, C770, C776, C778, C780, C782, C784, C786, C787, C789, C790, C791, C793, C794, C796: footprint Capacitor_THT:C_Rect_L11.0mm_W2.8mm_P10.00mm_MKT -> Capacitor_THT:C_Rect_L11.5mm_W2.0mm_P10.00mm_MKT

Commit message: Add DoNotPopulate field for components which shouldn't be fitted
Parts:
- CN704, CN705: DoNotPopulate (none) -> yes
Changed lines of the file:
@@
 F 2 "ISA:ISA16" H 4500 10000 50  0001 C CNN
 F 3 "" H 4500 10000 50  0001 C CNN
+F 4 "yes" H 4500 9950 50  0001 C CNN "DoNotPopulate"
 	1    4500 9950
 	1    0    0    -1
@@
 F 2 "ISA:ISA16" H 7150 10000 50  0001 C CNN
 F 3 "" H 7150 10000 50  0001 C CNN
+F 4 "yes" H 7150 9950 50  0001 C CNN "DoNotPopulate"
 	1    7150 9950
 	1    0    0    -1
