File: pc slots.sch (KiCad schematic (older format))
At the start: 64 parts, among them CN700 IBM_8_BIT_EXPANSION_BUS, CN701 IBM_8_BIT_EXPANSION_BUS, CN702 IBM_8_BIT_EXPANSION_BUS, CN703 IBM_8_BIT_EXPANSION_BUS, CN704 IBM_16_BIT_EXTENDED_BUS, CN705 IBM_16_BIT_EXTENDED_BUS, CN706 IBM_16_BIT_EXTENDED_BUS, CN707 IBM_16_BIT_EXTENDED_BUS

Commit message: Switch footprints for suitable modern replacements
Parts:
- C700, C702, C703, C704, C705: footprint Capacitor_THT:C_Rect_L11.5mm_W2.0mm_P10.00mm_MKT -> Capacitor_THT:C_Rect_L11.5mm_W4.0mm_P10.00mm_MKT
- C711, C713, C714, C716, C717, C719, C720, C722, C726, C728, C730, C732, C734, C736, C738, C740, C742, C744, C746, C748, C750, C752, C754, C756, C758, C760, C762, C764, C766, C768, C770, C776, C778, C780, C782, C784, C786, C787, C789, C790, C791, C793, C794, C796: footprint Capacitor_THT:C_Rect_L11.5mm_W2.0mm_P10.00mm_MKT -> Capacitor_THT:C_Rect_L11.5mm_W2.6mm_P10.00mm_MKT

Commit message: Some footprints updates; Add all Mouser references
Parts:
- C700, C702, C703, C704, C705: RefOrder (none) -> 594-A224K20X7RF5TAA
- C701: RefOrder (none) -> 667-ECA-1CM220B
- C711, C713, C714, C716, C717, C719, C720, C722, C726, C728, C730, C732, C734, C736, C738, C740, C742, C744, C746, C748, C750, C752, C754, C756, C758, C760, C762, C764, C766, C768, C770, C776, C778, C780, C782, C784, C786, C787, C789, C790, C791, C793, C794, C796: RefOrder (none) -> 581-SA105C102KAR
- RP700, RP701, RP702, RP703, RP704: RefOrder (none) -> 652-4610X-1LF-1K
- RP705: RefOrder (none) -> 858-L101S472LF

Commit message: Got the components, reduce some footprints
Parts:
- C700, C702, C703, C704, C705: footprint Capacitor_THT:C_Rect_L11.5mm_W4.0mm_P10.00mm_MKT -> Capacitor_THT:C_Rect_L11.5mm_W2.6mm_P10.00mm_MKT
- C701: footprint Capacitor_THT:CP_Radial_D8.0mm_P5.00mm -> Capacitor_THT:CP_Radial_Tantal_D5.0mm_P5.00mm
Changed lines of the file:
@@
 F 0 "C700" H 2865 9046 50  0000 L CNN
 F 1 "0.22uF" H 2865 8955 50  0000 L CNN
-F 2 "Capacitor_THT:C_Rect_L11.5mm_W4.0mm_P10.00mm_MKT" H 2788 8850 50  0001 C CNN
+F 2 "Capacitor_THT:C_Rect_L11.5mm_W2.6mm_P10.00mm_MKT" H 2788 8850 50  0001 C CNN
 F 3 "~" H 2750 9000 50  0001 C CNN
 F 4 "594-A224K20X7RF5TAA" H 2750 9000 50  0001 C CNN "RefOrder"
@@
 F 0 "C703" H 2915 5346 50  0000 L CNN
 F 1 "0.22uF" H 2915 5255 50  0000 L CNN
-F 2 "Capacitor_THT:C_Rect_L11.5mm_W4.0mm_P10.00mm_MKT" H 2838 5150 50  0001 C CNN
+F 2 "Capacitor_THT:C_Rect_L11.5mm_W2.6mm_P10.00mm_MKT" H 2838 5150 50  0001 C CNN
 F 3 "~" H 2800 5300 50  0001 C CNN
 F 4 "594-A224K20X7RF5TAA" H 2800 5300 50  0001 C CNN "RefOrder"
@@
 F 0 "C704" H 2665 5846 50  0000 L CNN
 F 1 "0.22uF" H 2665 5755 50  0000 L CNN
-F 2 "Capacitor_THT:C_Rect_L11.5mm_W4.0mm_P10.00mm_MKT" H 2588 5650 50  0001 C CNN
+F 2 "Capacitor_THT:C_Rect_L11.5mm_W2.6mm_P10.00mm_MKT" H 2588 5650 50  0001 C CNN
 F 3 "~" H 2550 5800 50  0001 C CNN
 F 4 "594-A224K20X7RF5TAA" H 2550 5800 50  0001 C CNN "RefOrder"
@@
 F 0 "C702" H 3165 5846 50  0000 L CNN
 F 1 "0.22uF" H 3165 5755 50  0000 L CNN
-F 2 "Capacitor_THT:C_Rect_L11.5mm_W4.0mm_P10.00mm_MKT" H 3088 5650 50  0001 C CNN
+F 2 "Capacitor_THT:C_Rect_L11.5mm_W2.6mm_P10.00mm_MKT" H 3088 5650 50  0001 C CNN
 F 3 "~" H 3050 5800 50  0001 C CNN
 F 4 "594-A224K20X7RF5TAA" H 3050 5800 50  0001 C CNN "RefOrder"
@@
 F 0 "C701" H 1968 9046 50  0000 L CNN
 F 1 "22uF 16V" H 1968 8955 50  0000 L CNN
-F 2 "Capacitor_THT:CP_Radial_D8.0mm_P5.00mm" H 1888 8850 50  0001 C CNN
+F 2 "Capacitor_THT:CP_Radial_Tantal_D5.0mm_P5.00mm" H 1888 8850 50  0001 C CNN
 F 3 "~" H 1850 9000 50  0001 C CNN
 F 4 "667-ECA-1CM220B" H 1850 9000 50  0001 C CNN "RefOrder"
@@
 F 0 "C705" H 1365 9046 50  0000 L CNN
 F 1 "0.22uF" H 1365 8955 50  0000 L CNN
-F 2 "Capacitor_THT:C_Rect_L11.5mm_W4.0mm_P10.00mm_MKT" H 1288 8850 50  0001 C CNN
+F 2 "Capacitor_THT:C_Rect_L11.5mm_W2.6mm_P10.00mm_MKT" H 1288 8850 50  0001 C CNN
 F 3 "~" H 1250 9000 50  0001 C CNN
 F 4 "594-A224K20X7RF5TAA" H 1250 9000 50  0001 C CNN "RefOrder"

Commit message: Some footprint changes; Tidy pcb
Parts:
- C711, C713, C714, C716, C717, C719, C720, C722, C726, C728, C730, C732, C734, C736, C738, C740, C742, C744, C746, C748, C750, C752, C754, C756, C758, C760, C762, C764, C766, C768, C770, C776, C778, C780, C782, C784, C786, C787, C789, C790, C791, C793, C794, C796: footprint Capacitor_THT:C_Rect_L11.5mm_W2.6mm_P10.00mm_MKT -> Capacitor_THT:C_Rect_L11.5mm_W2.0mm_P10.00mm_MKT
