File: agnus.sch (KiCad schematic (older format))
At the start: 0 parts

Commit message: Use correct source rev6. mostly all schematics done for first pass...
Parts:
- added C101, C102, C107, C110, C918: 0.1uF, symbol Device:C
- added C415: 4.7uF 16V, symbol Device:CP
- added C905, C907, C908: 100pF, symbol Device:C
- added FB101, FB102, FB907: Ferrite_Bead_Small, symbol Device:Ferrite_Bead_Small
- added J102, J900: Jumper_2_Bridged, symbol Jumper:Jumper_2_Bridged
- added R101, R109, R916: 4.7k, symbol Device:R
- added R105, R106: 22, symbol Device:R
- added R110, R114, R115: 330, symbol Device:R
- added RP102, RP902, RP907: 47, Resistor_THT:R_Array_SIP8, symbol Device:R_Pack04_SIP
- added U101: AGNUS8372, symbol amiga_customs:AGNUS8372
- added U102: GARY5719, symbol amiga_customs:GARY5719
- added U107: 74F04, symbol 74xx:74LS04
- added U108: 74LS74A, symbol 74xx:74LS74
- added U302: 74LS32, symbol 74xx:74LS32
- added U900: 74F00, symbol 74xx:74LS00
- added X1: 28.63636MHz, Oscillator:Oscillator_DIP-14, symbol Oscillator:ACO-xxxMHz
Connections:
- new net: U101.52 (_LDS), U102.10 (_LDS)
- new net: U101.53 (_UDS), U102.11 (_UDS)
- new net: U101.22 (R/W), U102.12 (R/W)
- new net: U101.24 (_AS), U102.13 (_AS)
- new net: J900.2 (B), R916.1, U102.14 (_BGACK)
- new net: U102.15 (_BLIT), U900.8
- new net: U101.23 (_REGEN), U102.18 (_REGEN)
- new net: U101.19 (_BLISS), U102.19 (_BLISS)
- new net: R105.1, U102.2 (_VPA)
- new net: U101.25 (_RAMEN), U102.20 (_RAMEN)
- new net: C905.2, FB102.1, U102.25 (_LATCH)
- new net: R106.1, U102.43 (_DTACK)
- new net: U101.20 (_BLIT), U900.12
- new net: RP907.3 (R2.1), RP907.5 (R3.1), U101.38 (7MHz), U302.9
- new net: J102.1 (A), R101.1, U101.41 (PAL/_NTSC)
- new net: U900.10, U900.11
- new net: FB101.2, X1.8 (OUT)
- new net: RP907.2 (R1.2), U302.8
- new net: RP902.7 (R4.1), U107.2
- new net: RP902.6 (R3.2), U107.10
- new net: RP102.6 (R3.2), RP102.7 (R4.1), U107.4
- new net: RP902.3 (R2.1), U107.12
- new net: RP102.3 (R2.1), U107.6
- new net: RP102.2 (R1.2), U107.8
- new net: FB907.2, RP102.1 (R1.1)
- new net +5V: C101.1, C102.1, C107.1, C110.1, C415.1, C918.1, R101.2, R109.2, R114.1, R115.1, R916.2, U101.15 (+5V), U102.17 (VCC), U102.48 (VCC), U102.6 (VCC), U108.14 (VCC), U900.13, U900.14 (VCC), X1.14 (Vcc)
- new net 28M: FB101.1, U101.34 (28MHZ)
- new net 7M: RP907.6 (R3.2)
- new net A17: U102.33 (A17)
- new net A18: U102.34 (A18)
- new net A19: U102.35 (A19)
- new net A20: U102.36 (A20)
- new net A21: U102.37 (A21)
- new net A22: U102.38 (A22)
- new net A23: U102.39 (A23)
- new net C1: C907.1, U101.40 (CCK), U102.28 (CCK), U107.13, U107.3
- new net C3: C908.1, U101.39 (CCKQ), U102.27 (CCKQ), U107.5, U107.9
- new net DMAL: U101.18 (DMAL)
- new net DRA0: U101.43 (DRA0)
- new net DRA1: U101.44 (DRA1)
- new net DRA2: U101.45 (DRA2)
- new net DRA3: U101.46 (DRA3)
- new net DRA4: U101.47 (DRA4)
- new net DRA5: U101.48 (DRA5)
- new net DRA6: U101.49 (DRA6)
- new net DRA7: U101.50 (DRA7)
- new net DRA8: U101.51 (DRA8)
- new net E7M: RP907.1 (R1.1)
- new net ECDAC: RP902.8 (R4.2)
- new net GND: C101.2, C102.2, C107.2, C110.2, C415.2, C905.1, C907.2, C908.2, C918.2, J102.2 (B), R110.2, U101.42 (VSS1), U101.58 (VSS2), U101.82 (VSS3), U102.1 (GND), U102.24 (GND), U102.40 (NC), U108.7 (GND), U302.10, U900.7 (GND), X1.7 (GND)
- new net OVL: U102.30 (OVL)
- new net RGA1: U101.33 (RGA1)
- new net RGA2: U101.32 (RGA2)
- new net RGA3: U101.31 (RGA3)
- new net RGA4: U101.30 (RGA4)
- new net RGA5: U101.29 (RGA5)
- new net RGA6: U101.28 (RGA6)
- new net RGA7: U101.27 (RGA7)
- new net RGA8: U101.26 (RGA8)
- new net V7M: RP907.4 (R2.2)
- new net VCDAC: RP902.5 (R3.1)
- new net XCLK: R110.1, U101.35 (XCLK)
- new net XRDY: R114.2, U102.31 (XRDY)
- new net _BGACK: J900.1 (A)
- new net _CASL: U101.54 (_CASL)
- new net _CASU: U101.55 (_CASU)
- new net _CDAC: U101.37 (_CDAC), U102.26 (_CDAC), U107.1, U107.11
- new net _CLKRD: U102.22 (_CLKRD)
- new net _CLKWR: U102.23 (_CLKWR)
- new net _CSYNC: U101.80 (_CSYNC)
- new net _DTACK: R106.2
- new net _EC1: RP902.4 (R2.2)
- new net _EC3: FB907.1
- new net _EXRAM: U102.32 (_EXRAM)
- new net _HLT: U102.42 (_HLT)
- new net _HSYNC: U101.81 (_HSYNC)
- new net _INT3: U101.17 (_INTR)
- new net _LATCH: FB102.2
- new net _LPEN: U101.78 (_LPEN)
- new net _MC1: RP102.8 (R4.2)
- new net _OEB: U102.4 (_OEB)
- new net _OEL: U102.3 (_OEL)
- new net _OVR: R115.2, U102.29 (_OVR)
- new net _RAS1: U101.56 (_RAS1)
- new net _ROMEN: U102.21 (_ROMEN), U900.9
- new net _RST: U101.16 (_RESET), U102.41 (_RST)
- new net _VC1: RP102.5 (R3.1)
- new net _VC3: RP102.4 (R2.2)
- new net _VPA: R105.2
- new net _VSYNC: U101.79 (_VSYNC)
- new net _WE: U101.21 (_WE)
- new net _XCLKEN: R109.1, U101.36 (_XCLKEN)
- new net __RAS0: U101.57 (_RAS0)
- no-connect marks 0 -> 4
Other:
- note added: "J102\nopen : PAL\nclosed : NTSC"
