File: agnus.sch (KiCad schematic (older format))
At the start: 32 parts, among them J102 Jumper_2_Bridged, J900 Jumper_2_Bridged, U101 AGNUS8372, U102 GARY5719, U107 74F04, U108 74LS74A, U302 74LS32, U900 74F00, X1 28.63636MHz

Commit message: Rename bus with correct syntax
Parts:
- added J101: Conn_01x03_Male, symbol Connector:Conn_01x03_Male
Connections:
- net A17: now also U101.76 (A17)
- net A18: now also U101.77 (A18)
- net A19: now also J101.3 (Pin_3)
- net A23: now also J101.1 (Pin_1)
- net DRD13: now reaches U101.1 (DRD13)
- net DRD4: now reaches U101.10 (DRD4)
- net DRD3: now reaches U101.11 (DRD3)
- net DRD2: now reaches U101.12 (DRD2)
- net DRD1: now reaches U101.13 (DRD1)
- net DRD0: now reaches U101.14 (DRD0)
- net DRD12: now reaches U101.2 (DRD12)
- net DRD11: now reaches U101.3 (DRD11)
- net DRD10: now reaches U101.4 (DRD10)
- net DRD9: now reaches U101.5 (DRD9)
- net at U101.59 (A19): now also J101.2 (Pin_2)
- net DRD8: now reaches U101.6 (DRD8)
- net A1: now reaches U101.60 (A1)
- net A2: now reaches U101.61 (A2)
- net A3: now reaches U101.62 (A3)
- net A4: now reaches U101.63 (A4)
- net A5: now reaches U101.64 (A5)
- net A6: now reaches U101.65 (A6)
- net A7: now reaches U101.66 (A7)
- net A8: now reaches U101.67 (A8)
- net A9: now reaches U101.68 (A9)
- net A10: now reaches U101.69 (A10)
- net DRD7: now reaches U101.7 (DRD7)
- net A11: now reaches U101.70 (A11)
- net A12: now reaches U101.71 (A12)
- net A13: now reaches U101.72 (A13)
- net A14: now reaches U101.73 (A14)
- net A15: now reaches U101.74 (A15)
- net A16: now reaches U101.75 (A16)
- net DRD6: now reaches U101.8 (DRD6)
- net DRD15: now reaches U101.83 (DRD15)
- net DRD14: now reaches U101.84 (DRD14)
- net DRD5: now reaches U101.9 (DRD5)
Other:
- note added: "normal\n\nspecial"
- moved on the sheet: C107, C918, U108C, U900E

Commit message: Some ERC things
Connections:
- net __RAS0 renamed _RAS0
Changed lines of the file:
@@
-EESchema Schematic File Version 5
+EESchema Schematic File Version 4
 LIBS:amiga2000-cache
 EELAYER 29 0
@@
 _RAS1
 Text GLabel 10350 5850 2    50   Input ~ 0
-__RAS0
+_RAS0
 Text GLabel 10350 5750 2    50   Input ~ 0
 _CASU

Commit message: Implemented various rev 6.2 fixes from forums and my own board
Connections:
- net _LDS: now reaches U101.52 (_LDS), U102.10 (_LDS)
- net _UDS: now reaches U101.53 (_UDS), U102.11 (_UDS)
- net R_W: now reaches U101.22 (R/W), U102.12 (R/W)
- net _AS: now reaches U101.24 (_AS), U102.13 (_AS)
Changed lines of the file:
@@
 Wire Bus Line
 	7600 4350 7600 5950
+Text GLabel 2100 8850 0    50   Input ~ 0
+_LDS
+Text GLabel 2200 8950 0    50   Input ~ 0
+_UDS
+Text GLabel 2300 9050 0    50   Input ~ 0
+R_W
+Text GLabel 2400 9150 0    50   Input ~ 0
+_AS
 $EndSCHEMATC

Commit message: Review done
Parts:
- added C107: 0.1uF, symbol Device:C
- added unit 7 of U107
- U107: value 74F04 -> 74LS74A
- renumbered C107 to C108
Connections:
- net +5V: now also C107.1, U107.14 (VCC)
- net GND: now also C107.2, U107.7 (GND)
Other:
- moved on the sheet: C108, C918, U108C, U900E
Changed lines of the file:
@@
 U 1 1 6B4C7698
 P 1400 3200
-F 0 "J900" H 1400 3303 50  0000 C CNN
+F 0 "J900" H 1400 3100 50  0000 C CNN
 F 1 "Jumper_2_Bridged" H 1400 3304 50  0001 C CNN
 F 2 "" H 1400 3200 50  0001 C CNN
@@
 P 10800 2000
 F 0 "U107" H 10800 2317 50  0000 C CNN
-F 1 "74F04" H 10800 2226 50  0000 C CNN
+F 1 "74LS74A" H 10800 2226 50  0000 C CNN
 F 2 "" H 10800 2000 50  0001 C CNN
-F 3 "http://www.ti.com/lit/gpn/sn74LS04" H 10800 2000 50  0001 C CNN
+F 3 "74xx/74hc_hct74.pdf" H 10800 2000 50  0001 C CNN
 	1    10800 2000
 	1    0    0    -1
@@
 P 10800 2500
 F 0 "U107" H 10800 2817 50  0000 C CNN
-F 1 "74F04" H 10800 2726 50  0000 C CNN
+F 1 "74LS74A" H 10800 2726 50  0000 C CNN
 F 2 "" H 10800 2500 50  0001 C CNN
-F 3 "http://www.ti.com/lit/gpn/sn74LS04" H 10800 2500 50  0001 C CNN
+F 3 "74xx/74hc_hct74.pdf" H 10800 2500 50  0001 C CNN
 	5    10800 2500
 	1    0    0    -1
@@
 P 12400 2900
 F 0 "U107" H 12400 3217 50  0000 C CNN
-F 1 "74F04" H 12400 3126 50  0000 C CNN
+F 1 "74LS74A" H 12400 3126 50  0000 C CNN
 F 2 "" H 12400 2900 50  0001 C CNN
-F 3 "http://www.ti.com/lit/gpn/sn74LS04" H 12400 2900 50  0001 C CNN
+F 3 "74xx/74hc_hct74.pdf" H 12400 2900 50  0001 C CNN
 	2    12400 2900
 	1    0    0    -1
@@
 P 12400 3450
 F 0 "U107" H 12400 3767 50  0000 C CNN
-F 1 "74F04" H 12400 3676 50  0000 C CNN
+F 1 "74LS74A" H 12400 3676 50  0000 C CNN
 F 2 "" H 12400 3450 50  0001 C CNN
-F 3 "http://www.ti.com/lit/gpn/sn74LS04" H 12400 3450 50  0001 C CNN
+F 3 "74xx/74hc_hct74.pdf" H 12400 3450 50  0001 C CNN
 	6    12400 3450
 	1    0    0    -1
@@
 P 12400 4000
 F 0 "U107" H 12400 4317 50  0000 C CNN
-F 1 "74F04" H 12400 4226 50  0000 C CNN
+F 1 "74LS74A" H 12400 4226 50  0000 C CNN
 F 2 "" H 12400 4000 50  0001 C CNN
-F 3 "http://www.ti.com/lit/gpn/sn74LS04" H 12400 4000 50  0001 C CNN
+F 3 "74xx/74hc_hct74.pdf" H 12400 4000 50  0001 C CNN
 	3    12400 4000
 	1    0    0    -1
@@
 P 12400 4500
 F 0 "U107" H 12400 4817 50  0000 C CNN
-F 1 "74F04" H 12400 4726 50  0000 C CNN
+F 1 "74LS74A" H 12400 4726 50  0000 C CNN
 F 2 "" H 12400 4500 50  0001 C CNN
-F 3 "http://www.ti.com/lit/gpn/sn74LS04" H 12400 4500 50  0001 C CNN
+F 3 "74xx/74hc_hct74.pdf" H 12400 4500 50  0001 C CNN
 	4    12400 4500
 	1    0    0    -1
@@
 L 74xx:74LS00 U900
 U 5 1 6B7B9312
-P 2800 6550
-F 0 "U900" H 2570 6596 50  0000 R CNN
-F 1 "74F00" H 2570 6505 50  0000 R CNN
-F 2 "" H 2800 6550 50  0001 C CNN
-F 3 "http://www.ti.com/lit/gpn/sn74ls00" H 2800 6550 50  0001 C CNN
-	5    2800 6550
+P 12350 7050
+F 0 "U900" H 12120 7096 50  0000 R CNN
+F 1 "74F00" H 12120 7005 50  0000 R CNN
+F 2 "" H 12350 7050 50  0001 C CNN
+F 3 "http://www.ti.com/lit/gpn/sn74ls00" H 12350 7050 50  0001 C CNN
+	5    12350 7050
 	-1   0    0    -1
 $EndComp
@@
 L 74xx:74LS74 U108
 U 3 1 6B7BBA8F
-P 4000 6550
-F 0 "U108" H 4230 6596 50  0000 L CNN
-F 1 "74LS74A" H 4230 6505 50  0000 L CNN
-F 2 "" H 4000 6550 50  0001 C CNN
-F 3 "74xx/74hc_hct74.pdf" H 4000 6550 50  0001 C CNN
-	3    4000 6550
+P 13550 7050
+F 0 "U108" H 13780 7096 50  0000 L CNN
+F 1 "74LS74A" H 13780 7005 50  0000 L CNN
+F 2 "" H 13550 7050 50  0001 C CNN
+F 3 "74xx/74hc_hct74.pdf" H 13550 7050 50  0001 C CNN
+	3    13550 7050
 	1    0    0    -1
 $EndComp
@@
 L Device:C C918
 U 1 1 6B7BD2B6
-P 3400 6550
-F 0 "C918" H 3515 6596 50  0000 L CNN
-F 1 "0.1uF" H 3515 6505 50  0000 L CNN
-F 2 "" H 3438 6400 50  0001 C CNN
-F 3 "~" H 3400 6550 50  0001 C CNN
-	1    3400 6550
-	1    0    0    -1
-$EndComp
-$Comp
-L Device:C C107
+P 12950 7050
+F 0 "C918" H 13065 7096 50  0000 L CNN
+F 1 "0.1uF" H 13065 7005 50  0000 L CNN
+F 2 "" H 12988 6900 50  0001 C CNN
+F 3 "~" H 12950 7050 50  0001 C CNN
+	1    12950 7050
+	1    0    0    -1
+$EndComp
+$Comp
+L Device:C C108
 U 1 1 6B7BD59D
-P 4650 6500
-F 0 "C107" H 4765 6546 50  0000 L CNN
-F 1 "0.1uF" H 4765 6455 50  0000 L CNN
-F 2 "" H 4688 6350 50  0001 C CNN
-F 3 "~" H 4650 6500 50  0001 C CNN
-	1    4650 6500
+P 14200 7000
+F 0 "C108" H 14315 7046 50  0000 L CNN
+F 1 "0.1uF" H 14315 6955 50  0000 L CNN
+F 2 "" H 14238 6850 50  0001 C CNN
+F 3 "~" H 14200 7000 50  0001 C CNN
+	1    14200 7000
 	1    0    0    -1
 $EndComp
@@
 L power:+5V #PWR0168
 U 1 1 6B7BE40D
-P 2800 5900
-F 0 "#PWR0168" H 2800 5750 50  0001 C CNN
-F 1 "+5V" H 2815 6073 50  0000 C CNN
-F 2 "" H 2800 5900 50  0001 C CNN
-F 3 "" H 2800 5900 50  0001 C CNN
-	1    2800 5900
+P 12350 6400
+F 0 "#PWR0168" H 12350 6250 50  0001 C CNN
+F 1 "+5V" H 12365 6573 50  0000 C CNN
+F 2 "" H 12350 6400 50  0001 C CNN
+F 3 "" H 12350 6400 50  0001 C CNN
+	1    12350 6400
 	1    0    0    -1
 $EndComp
@@
 L power:GND #PWR0169
 U 1 1 6B7BE899
-P 2800 7200
-F 0 "#PWR0169" H 2800 6950 50  0001 C CNN
-F 1 "GND" H 2805 7027 50  0000 C CNN
-F 2 "" H 2800 7200 50  0001 C CNN
-F 3 "" H 2800 7200 50  0001 C CNN
-	1    2800 7200
-	1    0    0    -1
-$EndComp
-Wire Wire Line
-	2800 5900 2800 6000
-Wire Wire Line
-	2800 6000 3400 6000
-Wire Wire Line
-	4650 6000 4650 6350
-Connection ~ 2800 6000
-Wire Wire Line
-	2800 6000 2800 6050
-Wire Wire Line
-	4000 6150 4000 6000
-Connection ~ 4000 6000
-Wire Wire Line
-	4000 6000 4650 6000
-Wire Wire Line
-	3400 6000 3400 6400
-Connection ~ 3400 6000
-Wire Wire Line
-	3400 6000 4000 6000
-Wire Wire Line
-	2800 7050 2800 7150
-Wire Wire Line
-	2800 7150 3400 7150
-Wire Wire Line
-	3400 7150 3400 6700
-Connection ~ 2800 7150
-Wire Wire Line
-	2800 7150 2800 7200
-Wire Wire Line
-	3400 7150 4000 7150
-Wire Wire Line
-	4000 7150 4000 6950
-Connection ~ 3400 7150
-Wire Wire Line
-	4000 7150 4650 7150
-Wire Wire Line
-	4650 7150 4650 6650
-Connection ~ 4000 7150
+P 12350 7700
+F 0 "#PWR0169" H 12350 7450 50  0001 C CNN
+F 1 "GND" H 12355 7527 50  0000 C CNN
+F 2 "" H 12350 7700 50  0001 C CNN
+F 3 "" H 12350 7700 50  0001 C CNN
+	1    12350 7700
+	1    0    0    -1
+$EndComp
+Wire Wire Line
+	12350 6400 12350 6500
+Wire Wire Line
+	12350 6500 12950 6500
+Wire Wire Line
+	14200 6500 14200 6850
+Connection ~ 12350 6500
+Wire Wire Line
+	12350 6500 12350 6550
+Wire Wire Line
+	13550 6650 13550 6500
+Connection ~ 13550 6500
+Wire Wire Line
+	13550 6500 14200 6500
+Wire Wire Line
+	12950 6500 12950 6900
+Connection ~ 12950 6500
+Wire Wire Line
+	12950 6500 13550 6500
+Wire Wire Line
+	12350 7550 12350 7650
+Wire Wire Line
+	12350 7650 12950 7650
+Wire Wire Line
+	12950 7650 12950 7200
+Connection ~ 12350 7650
+Wire Wire Line
+	12350 7650 12350 7700
+Wire Wire Line
+	12950 7650 13550 7650
+Wire Wire Line
+	13550 7650 13550 7450
+Connection ~ 12950 7650
+Wire Wire Line
+	13550 7650 14200 7650
+Wire Wire Line
+	14200 7650 14200 7150
+Connection ~ 13550 7650
 $Comp
 L Connector:Conn_01x03_Male J101
@@
 Text GLabel 2400 9150 0    50   Input ~ 0
 _AS
+$Comp
+L 74xx:74LS04 U107
+U 7 1 5D029E31
+P 14750 7050
+F 0 "U107" H 14980 7096 50  0000 L CNN
+F 1 "74LS74A" H 14980 7005 50  0000 L CNN
+F 2 "" H 14750 7050 50  0001 C CNN
+F 3 "74xx/74hc_hct74.pdf" H 14750 7050 50  0001 C CNN
+	7    14750 7050
+	1    0    0    -1
+$EndComp
+$Comp
+L Device:C C107
+U 1 1 5D04624F
+P 15450 7000
+F 0 "C107" H 15565 7046 50  0000 L CNN
+F 1 "0.1uF" H 15565 6955 50  0000 L CNN
+F 2 "" H 15488 6850 50  0001 C CNN
+F 3 "~" H 15450 7000 50  0001 C CNN
+	1    15450 7000
+	1    0    0    -1
+$EndComp
+Connection ~ 14200 6500
+Wire Wire Line
+	15450 6500 15450 6850
+Connection ~ 14200 7650
+Wire Wire Line
+	15450 7650 15450 7150
+Wire Wire Line
+	14200 6500 14750 6500
+Wire Wire Line
+	14200 7650 14750 7650
+Wire Wire Line
+	14750 7550 14750 7650
+Connection ~ 14750 7650
+Wire Wire Line
+	14750 7650 15450 7650
+Wire Wire Line
+	14750 6550 14750 6500
 Wire Bus Line
 	2200 700  2200 1900
@@
 Wire Bus Line
 	7600 4350 7600 5950
+Connection ~ 14750 6500
+Wire Wire Line
+	14750 6500 15450 6500
 $EndSCHEMATC

Commit message: Associate footprints with components
Parts:
- FB101, FB907: footprint (none) -> Inductor_THT:L_Axial_L7.0mm_D3.3mm_P10.16mm_Horizontal_Fastron_MICC
- FB102: footprint (none) -> Inductor_THT:L_Axial_L9.5mm_D4.0mm_P15.24mm_Horizontal_Fastron_SMCC
- J101: footprint (none) -> Connector_PinSocket_2.54mm:PinSocket_1x03_P2.54mm_Vertical
- J102: value Jumper_2_Bridged -> Jumper_2_Open; footprint (none) -> Jumper:SolderJumper-2_P1.3mm_Open_RoundedPad1.0x1.5mm; symbol Jumper:Jumper_2_Bridged -> Jumper:Jumper_2_Open
- J900: footprint (none) -> Connector_PinSocket_2.54mm:PinSocket_2x01_P2.54mm_Vertical
- R101, R105, R106, R109, R110, R114, R115, R916: footprint (none) -> Resistor_THT:R_Axial_DIN0207_L6.3mm_D2.5mm_P10.16mm_Horizontal
- U101: footprint (none) -> Package_LCC:PLCC-84_THT-Socket
- U102: footprint (none) -> Package_DIP:DIP-48_W15.24mm_Socket
- U107, U108, U302, U900: footprint (none) -> Package_DIP:DIP-14_W7.62mm_Socket
Other:
- moved on the sheet: J102
Changed lines of the file:
@@
 F 0 "U102" H 3750 998 50  0000 C CNN
 F 1 "GARY5719" H 3750 907 50  0000 C CNN
-F 2 "" H 3750 950 50  0001 C CNN
+F 2 "Package_DIP:DIP-48_W15.24mm_Socket" H 3750 950 50  0001 C CNN
 F 3 "" H 3750 950 50  0001 C CNN
 	1    3750 800
@@
 F 0 "U102" V 1496 10222 50  0000 R CNN
 F 1 "GARY5719" V 1405 10222 50  0000 R CNN
-F 2 "" H 1450 10750 50  0001 C CNN
+F 2 "Package_DIP:DIP-48_W15.24mm_Socket" H 1450 10750 50  0001 C CNN
 F 3 "" H 1450 10750 50  0001 C CNN
 	3    1450 10600
@@
 F 0 "U101" H 9350 1500 50  0000 C CNN
 F 1 "AGNUS8372" H 9350 2100 50  0000 C CNN
-F 2 "" H 9300 3900 50  0001 C CNN
+F 2 "Package_LCC:PLCC-84_THT-Socket" H 9300 3900 50  0001 C CNN
 F 3 "" H 9300 3900 50  0001 C CNN
 	1    9350 3900
@@
 F 0 "FB102" V 955 1200 50  0000 C CNN
 F 1 "Ferrite_Bead_Small" V 954 1200 50  0001 C CNN
-F 2 "" V 1030 1200 50  0001 C CNN
+F 2 "Inductor_THT:L_Axial_L9.5mm_D4.0mm_P15.24mm_Horizontal_Fastron_SMCC" V 1030 1200 50  0001 C CNN
 F 3 "~" H 1100 1200 50  0001 C CNN
 	1    1100 1200
@@
 F 0 "R105" V 1443 2200 50  0000 C CNN
 F 1 "22" V 1534 2200 50  0000 C CNN
-F 2 "" V 1580 2200 50  0001 C CNN
+F 2 "Resistor_THT:R_Axial_DIN0207_L6.3mm_D2.5mm_P10.16mm_Horizontal" V 1580 2200 50  0001 C CNN
 F 3 "~" H 1650 2200 50  0001 C CNN
 	1    1650 2200
@@
 F 0 "R106" V 1443 2700 50  0000 C CNN
 F 1 "22" V 1534 2700 50  0000 C CNN
-F 2 "" V 1580 2700 50  0001 C CNN
+F 2 "Resistor_THT:R_Axial_DIN0207_L6.3mm_D2.5mm_P10.16mm_Horizontal" V 1580 2700 50  0001 C CNN
 F 3 "~" H 1650 2700 50  0001 C CNN
 	1    1650 2700
@@
 F 0 "J900" H 1400 3100 50  0000 C CNN
 F 1 "Jumper_2_Bridged" H 1400 3304 50  0001 C CNN
-F 2 "" H 1400 3200 50  0001 C CNN
+F 2 "Connector_PinSocket_2.54mm:PinSocket_2x01_P2.54mm_Vertical" H 1400 3200 50  0001 C CNN
 F 3 "~" H 1400 3200 50  0001 C CNN
 	1    1400 3200
@@
 F 0 "R916" H 1820 3396 50  0000 L CNN
 F 1 "4.7k" H 1820 3305 50  0000 L CNN
-F 2 "" V 1680 3350 50  0001 C CNN
+F 2 "Resistor_THT:R_Axial_DIN0207_L6.3mm_D2.5mm_P10.16mm_Horizontal" V 1680 3350 50  0001 C CNN
 F 3 "~" H 1750 3350 50  0001 C CNN
 	1    1750 3350
@@
 F 0 "R115" H 5520 846 50  0000 L CNN
 F 1 "330" H 5520 755 50  0000 L CNN
-F 2 "" V 5380 800 50  0001 C CNN
+F 2 "Resistor_THT:R_Axial_DIN0207_L6.3mm_D2.5mm_P10.16mm_Horizontal" V 5380 800 50  0001 C CNN
 F 3 "~" H 5450 800 50  0001 C CNN
 	1    5450 800
@@
 F 0 "R114" H 6170 846 50  0000 L CNN
 F 1 "330" H 6170 755 50  0000 L CNN
-F 2 "" V 6030 800 50  0001 C CNN
+F 2 "Resistor_THT:R_Axial_DIN0207_L6.3mm_D2.5mm_P10.16mm_Horizontal" V 6030 800 50  0001 C CNN
 F 3 "~" H 6100 800 50  0001 C CNN
 	1    6100 800
@@
 F 0 "U900" H 5050 3425 50  0000 C CNN
 F 1 "74F00" H 5050 3334 50  0000 C CNN
-F 2 "" H 5050 3100 50  0001 C CNN
+F 2 "Package_DIP:DIP-14_W7.62mm_Socket" H 5050 3100 50  0001 C CNN
 F 3 "http://www.ti.com/lit/gpn/sn74ls00" H 5050 3100 50  0001 C CNN
 	3    5050 3100
@@
 F 0 "U900" H 5950 2883 50  0000 C CNN
 F 1 "74F00" H 5950 2974 50  0000 C CNN
-F 2 "" H 5950 3200 50  0001 C CNN
+F 2 "Package_DIP:DIP-14_W7.62mm_Socket" H 5950 3200 50  0001 C CNN
 F 3 "http://www.ti.com/lit/gpn/sn74ls00" H 5950 3200 50  0001 C CNN
 	4    5950 3200
@@
 F 0 "FB101" V 4755 10500 50  0000 C CNN
 F 1 "Ferrite_Bead_Small" H 5000 10455 50  0001 L CNN
-F 2 "" V 4830 10500 50  0001 C CNN
+F 2 "Inductor_THT:L_Axial_L7.0mm_D3.3mm_P10.16mm_Horizontal_Fastron_MICC" V 4830 10500 50  0001 C CNN
 F 3 "~" H 4900 10500 50  0001 C CNN
 	1    4900 10500
@@
 F 0 "R110" H 7920 10846 50  0000 L CNN
 F 1 "330" H 7920 10755 50  0000 L CNN
-F 2 "" V 7780 10800 50  0001 C CNN
+F 2 "Resistor_THT:R_Axial_DIN0207_L6.3mm_D2.5mm_P10.16mm_Horizontal" V 7780 10800 50  0001 C CNN
 F 3 "~" H 7850 10800 50  0001 C CNN
 	1    7850 10800
@@
 F 0 "R109" H 7470 10846 50  0000 L CNN
 F 1 "4.7k" H 7470 10755 50  0000 L CNN
-F 2 "" V 7330 10800 50  0001 C CNN
+F 2 "Resistor_THT:R_Axial_DIN0207_L6.3mm_D2.5mm_P10.16mm_Horizontal" V 7330 10800 50  0001 C CNN
 F 3 "~" H 7400 10800 50  0001 C CNN
 	1    7400 10800
@@
 F 0 "R101" H 10770 10246 50  0000 L CNN
 F 1 "4.7k" H 10770 10155 50  0000 L CNN
-F 2 "" V 10630 10200 50  0001 C CNN
+F 2 "Resistor_THT:R_Axial_DIN0207_L6.3mm_D2.5mm_P10.16mm_Horizontal" V 10630 10200 50  0001 C CNN
 F 3 "~" H 10700 10200 50  0001 C CNN
 	1    10700 10200
@@
 $EndComp
 $Comp
-L Jumper:Jumper_2_Bridged J102
+L Jumper:Jumper_2_Open J102
 U 1 1 6B58316C
 P 11100 10250
 F 0 "J102" V 11100 10308 50  0000 L CNN
-F 1 "Jumper_2_Bridged" V 11145 10308 50  0001 L CNN
-F 2 "" H 11100 10250 50  0001 C CNN
+F 1 "Jumper_2_Open" V 11145 10308 50  0001 L CNN
+F 2 "Jumper:SolderJumper-2_P1.3mm_Open_RoundedPad1.0x1.5mm" H 11100 10250 50  0001 C CNN
 F 3 "~" H 11100 10250 50  0001 C CNN
 	1    11100 10250
@@
 F 0 "U302" H 11700 9125 50  0000 C CNN
 F 1 "74LS32" H 11700 9034 50  0000 C CNN
-F 2 "" H 11700 8800 50  0001 C CNN
+F 2 "Package_DIP:DIP-14_W7.62mm_Socket" H 11700 8800 50  0001 C CNN
 F 3 "http://www.ti.com/lit/gpn/sn74LS32" H 11700 8800 50  0001 C CNN
 	3    11700 8800
@@
 F 0 "U107" H 10800 2317 50  0000 C CNN
 F 1 "74LS74A" H 10800 2226 50  0000 C CNN
-F 2 "" H 10800 2000 50  0001 C CNN
+F 2 "Package_DIP:DIP-14_W7.62mm_Socket" H 10800 2000 50  0001 C CNN
 F 3 "74xx/74hc_hct74.pdf" H 10800 2000 50  0001 C CNN
 	1    10800 2000
@@
 F 0 "U107" H 10800 2817 50  0000 C CNN
 F 1 "74LS74A" H 10800 2726 50  0000 C CNN
-F 2 "" H 10800 2500 50  0001 C CNN
+F 2 "Package_DIP:DIP-14_W7.62mm_Socket" H 10800 2500 50  0001 C CNN
 F 3 "74xx/74hc_hct74.pdf" H 10800 2500 50  0001 C CNN
 	5    10800 2500
@@
 F 0 "U107" H 12400 3217 50  0000 C CNN
 F 1 "74LS74A" H 12400 3126 50  0000 C CNN
-F 2 "" H 12400 2900 50  0001 C CNN
+F 2 "Package_DIP:DIP-14_W7.62mm_Socket" H 12400 2900 50  0001 C CNN
 F 3 "74xx/74hc_hct74.pdf" H 12400 2900 50  0001 C CNN
 	2    12400 2900
@@
 F 0 "U107" H 12400 3767 50  0000 C CNN
 F 1 "74LS74A" H 12400 3676 50  0000 C CNN
-F 2 "" H 12400 3450 50  0001 C CNN
+F 2 "Package_DIP:DIP-14_W7.62mm_Socket" H 12400 3450 50  0001 C CNN
 F 3 "74xx/74hc_hct74.pdf" H 12400 3450 50  0001 C CNN
 	6    12400 3450
@@
 F 0 "U107" H 12400 4317 50  0000 C CNN
 F 1 "74LS74A" H 12400 4226 50  0000 C CNN
-F 2 "" H 12400 4000 50  0001 C CNN
+F 2 "Package_DIP:DIP-14_W7.62mm_Socket" H 12400 4000 50  0001 C CNN
 F 3 "74xx/74hc_hct74.pdf" H 12400 4000 50  0001 C CNN
 	3    12400 4000
@@
 F 0 "U107" H 12400 4817 50  0000 C CNN
 F 1 "74LS74A" H 12400 4726 50  0000 C CNN
-F 2 "" H 12400 4500 50  0001 C CNN
+F 2 "Package_DIP:DIP-14_W7.62mm_Socket" H 12400 4500 50  0001 C CNN
 F 3 "74xx/74hc_hct74.pdf" H 12400 4500 50  0001 C CNN
 	4    12400 4500
@@
 F 0 "FB907" H 14450 4350 50  0000 L CNN
 F 1 "Ferrite_Bead_Small" H 14450 4305 50  0001 L CNN
-F 2 "" V 14280 4350 50  0001 C CNN
+F 2 "Inductor_THT:L_Axial_L7.0mm_D3.3mm_P10.16mm_Horizontal_Fastron_MICC" V 14280 4350 50  0001 C CNN
 F 3 "~" H 14350 4350 50  0001 C CNN
 	1    14350 4350
@@
 F 0 "U900" H 12120 7096 50  0000 R CNN
 F 1 "74F00" H 12120 7005 50  0000 R CNN
-F 2 "" H 12350 7050 50  0001 C CNN
+F 2 "Package_DIP:DIP-14_W7.62mm_Socket" H 12350 7050 50  0001 C CNN
 F 3 "http://www.ti.com/lit/gpn/sn74ls00" H 12350 7050 50  0001 C CNN
 	5    12350 7050
@@
 F 0 "U108" H 13780 7096 50  0000 L CNN
 F 1 "74LS74A" H 13780 7005 50  0000 L CNN
-F 2 "" H 13550 7050 50  0001 C CNN
+F 2 "Package_DIP:DIP-14_W7.62mm_Socket" H 13550 7050 50  0001 C CNN
 F 3 "74xx/74hc_hct74.pdf" H 13550 7050 50  0001 C CNN
 	3    13550 7050
@@
 F 0 "J101" H 6508 6539 50  0000 C CNN
 F 1 "Conn_01x03_Male" H 6508 6540 50  0001 C CNN
-F 2 "" H 6400 6350 50  0001 C CNN
+F 2 "Connector_PinSocket_2.54mm:PinSocket_1x03_P2.54mm_Vertical" H 6400 6350 50  0001 C CNN
 F 3 "~" H 6400 6350 50  0001 C CNN
 	1    6400 6350
@@
 F 0 "U107" H 14980 7096 50  0000 L CNN
 F 1 "74LS74A" H 14980 7005 50  0000 L CNN
-F 2 "" H 14750 7050 50  0001 C CNN
+F 2 "Package_DIP:DIP-14_W7.62mm_Socket" H 14750 7050 50  0001 C CNN
 F 3 "74xx/74hc_hct74.pdf" H 14750 7050 50  0001 C CNN
 	7    14750 7050
@@
 Wire Wire Line
 	14750 6550 14750 6500
+Connection ~ 14750 6500
+Wire Wire Line
+	14750 6500 15450 6500
 Wire Bus Line
 	2200 700  2200 1900
@@
 Wire Bus Line
 	7600 4350 7600 5950
-Connection ~ 14750 6500
-Wire Wire Line
-	14750 6500 15450 6500
 $EndSCHEMATC

Commit message: Associate more components
Parts:
- C415: footprint (none) -> Capacitor_THT:CP_Radial_D8.0mm_P5.00mm
Changed lines of the file:
@@
 F 0 "C415" H 11268 4846 50  0000 L CNN
 F 1 "4.7uF 16V" H 11268 4755 50  0000 L CNN
-F 2 "" H 11188 4650 50  0001 C CNN
+F 2 "Capacitor_THT:CP_Radial_D8.0mm_P5.00mm" H 11188 4650 50  0001 C CNN
 F 3 "~" H 11150 4800 50  0001 C CNN
 	1    11150 4800
