File: chipram.sch (KiCad schematic (older format))
At the start: 0 parts

Commit message: Use correct source rev6. mostly all schematics done for first pass...
Parts:
- added C500: 0.22uF, symbol Device:C
- added C501, C502, C503, C504, C505, C506, C507, C508: 0.33uF, symbol Device:C
- added J500: Jumper_2_Bridged, symbol Jumper:Jumper_2_Bridged
- added R500: 4.7k, symbol Device:R
- added RP500, RP501: 47, Resistor_THT:R_Array_SIP10, symbol Device:R_Pack05_SIP
- added RP502: 22, Resistor_THT:R_Array_SIP10, symbol Device:R_Pack05_SIP
- added RP503: 470, Resistor_THT:R_Array_SIP10, symbol Device:R_Network09
- added U500: 62402, symbol d_eeproms:62402
- added U501, U502, U503, U504, U505, U506, U507, U508: XX4256-15, symbol d_memory:XX4256-15
- added U540, U541: 74F244, symbol 74xx:74LS244
Connections:
- new net: RP500.7 (R4.1), U540.12 (O3a)
- new net: RP500.6 (R3.2), U540.14 (O2a)
- new net: RP500.4 (R2.2), U540.16 (O1a)
- new net: RP500.2 (R1.2), U540.18 (O0a)
- new net: RP500.9 (R5.1), U540.3 (O3b)
- new net: RP501.2 (R1.2), U540.5 (O2b)
- new net: RP501.6 (R3.2), U540.7 (O1b)
- new net: RP501.7 (R4.1), U540.9 (O0b)
- new net: RP502.2 (R1.2), U541.12 (O3a)
- new net: RP502.4 (R2.2), U541.14 (O2a)
- new net: RP501.10 (R5.2), U541.16 (O1a)
- new net: RP501.4 (R2.2), U541.18 (O0a)
- new net: RP502.10 (R5.2), U541.3 (O3b)
- new net: RP502.6 (R3.2), U541.7 (O1b)
- new net: RP501.9 (R5.1), U501.17 (_CAS), U502.17 (_CAS), U505.17 (_CAS), U506.17 (_CAS)
- new net: RP502.9 (R5.1), U501.3 (WE), U502.3 (WE), U503.3 (WE), U504.3 (WE), U505.3 (WE), U506.3 (WE), U507.3 (WE), U508.3 (WE)
- new net: RP502.1 (R1.1), U501.4 (_RAS), U502.4 (_RAS), U503.4 (_RAS), U504.4 (_RAS), U505.4 (_RAS), U506.4 (_RAS), U507.4 (_RAS), U508.4 (_RAS)
- new net: RP502.3 (R2.1), U503.17 (_CAS), U504.17 (_CAS), U507.17 (_CAS), U508.17 (_CAS)
- new net +5V: C500.2, C501.1, C502.1, C503.1, C504.1, C505.1, C506.1, C507.1, C508.1, R500.1, RP503.1 (common), U500.21 (VCC), U500.31 (WORD/_BYTE), U501.20 (GND), U502.20 (GND), U503.20 (GND), U504.20 (GND), U505.20 (GND), U506.20 (GND), U507.20 (GND), U508.20 (GND)
- new net A1: U500.9 (A0)
- new net A10: U500.39 (A9)
- new net A11: U500.38 (A10)
- new net A12: U500.37 (A11)
- new net A13: U500.36 (A12)
- new net A14: U500.35 (A13)
- new net A15: U500.34 (A14)
- new net A16: U500.33 (A15)
- new net A17: U500.32 (A16)
- new net A18: U500.1 (A17)
- new net A2: U500.8 (A1)
- new net A3: U500.7 (A2)
- new net A4: U500.6 (A3)
- new net A5: U500.5 (A4)
- new net A6: U500.4 (A5)
- new net A7: U500.3 (A6)
- new net A8: U500.2 (A7)
- new net A9: U500.40 (A8)
- new net D0: U500.13 (D0)
- new net D1: U500.15 (D1)
- new net D10: U500.18 (D10)
- new net D11: U500.20 (D11)
- new net D12: U500.23 (D12)
- new net D13: U500.25 (D13)
- new net D14: U500.27 (D14)
- new net D15: U500.29 (D15)
- new net D2: U500.17 (D2)
- new net D3: U500.19 (D3)
- new net D4: U500.22 (D4)
- new net D5: U500.24 (D5)
- new net D6: U500.26 (D6)
- new net D7: U500.28 (D7)
- new net D8: U500.14 (D8)
- new net D9: U500.16 (D9)
- new net DRA0: U540.2 (I0a)
- new net DRA1: U540.4 (I1a)
- new net DRA2: U540.6 (I2a)
- new net DRA3: U540.8 (I3a)
- new net DRA4: U540.17 (I3b)
- new net DRA5: U540.15 (I2b)
- new net DRA6: U540.13 (I1b)
- new net DRA7: U540.11 (I0b)
- new net DRA8: U541.2 (I0a)
- new net DRAB0: RP500.1 (R1.1), RP503.10 (R9), U501.6 (A0), U502.6 (A0), U503.6 (A0), U504.6 (A0), U505.6 (A0), U506.6 (A0), U507.6 (A0), U508.6 (A0)
- new net DRAB1: RP500.3 (R2.1), RP503.9 (R8), U501.7 (A1), U502.7 (A1), U503.7 (A1), U504.7 (A1), U505.7 (A1), U506.7 (A1), U507.7 (A1), U508.7 (A1)
- new net DRAB2: RP500.5 (R3.1), RP503.8 (R7), U501.8 (A2), U502.8 (A2), U503.8 (A2), U504.8 (A2), U505.8 (A2), U506.8 (A2), U507.8 (A2), U508.8 (A2)
- new net DRAB3: RP500.8 (R4.2), RP503.7 (R6), U501.9 (A3), U502.9 (A3), U503.9 (A3), U504.9 (A3), U505.9 (A3), U506.9 (A3), U507.9 (A3), U508.9 (A3)
- new net DRAB4: RP500.10 (R5.2), RP503.6 (R5), U501.11 (A4), U502.11 (A4), U503.11 (A4), U504.11 (A4), U505.11 (A4), U506.11 (A4), U507.11 (A4), U508.11 (A4)
- new net DRAB5: RP501.1 (R1.1), RP503.5 (R4), U501.12 (A5), U502.12 (A5), U503.12 (A5), U504.12 (A5), U505.12 (A5), U506.12 (A5), U507.12 (A5), U508.12 (A5)
- new net DRAB6: RP501.5 (R3.1), RP503.4 (R3), U501.13 (A6), U502.13 (A6), U503.13 (A6), U504.13 (A6), U505.13 (A6), U506.13 (A6), U507.13 (A6), U508.13 (A6)
- new net DRAB7: RP501.8 (R4.2), RP503.3 (R2), U501.14 (A7), U502.14 (A7), U503.14 (A7), U504.14 (A7), U505.14 (A7), U506.14 (A7), U507.14 (A7), U508.14 (A7)
- new net DRAB8: RP501.3 (R2.1), RP503.2 (R1), U501.15 (A8), U502.15 (A8), U503.15 (A8), U504.15 (A8), U505.15 (A8), U506.15 (A8), U507.15 (A8), U508.15 (A8)
- new net DRD0: U501.1 (D1), U505.1 (D1)
- new net DRD1: U501.2 (D2), U505.2 (D2)
- new net DRD10: U503.18 (D3), U507.18 (D3)
- new net DRD11: U503.19 (D4), U507.19 (D4)
- new net DRD12: U504.1 (D1), U508.1 (D1)
- new net DRD13: U504.2 (D2), U508.2 (D2)
- new net DRD14: U504.18 (D3), U508.18 (D3)
- new net DRD15: U504.19 (D4), U508.19 (D4)
- new net DRD2: U501.18 (D3), U505.18 (D3)
- new net DRD3: U501.19 (D4), U505.19 (D4)
- new net DRD4: U502.1 (D1), U506.1 (D1)
- new net DRD5: U502.2 (D2), U506.2 (D2)
- new net DRD6: U502.18 (D3), U506.18 (D3)
- new net DRD7: U502.19 (D4), U506.19 (D4)
- new net DRD8: U503.1 (D1), U507.1 (D1)
- new net DRD9: U503.2 (D2), U507.2 (D2)
- new net GND: C500.1, C501.2, C502.2, C503.2, C504.2, C505.2, C506.2, C507.2, C508.2, J500.2 (B), U500.11 (GND), U500.30 (GND), U501.10 (VCC), U501.16 (_OE), U502.10 (VCC), U502.16 (_OE), U503.10 (VCC), U503.16 (_OE), U504.10 (VCC), U504.16 (_OE), U505.10 (VCC), U505.16 (_OE), U506.10 (VCC), U506.16 (_OE), U507.10 (VCC), U507.16 (_OE), U508.10 (VCC), U508.16 (_OE), U541.11 (I0b), U541.15 (I2b)
- new net _CASL: U541.4 (I1a)
- new net _CASU: U541.6 (I2a)
- new net _EXRAM: J500.1 (A), R500.2
- new net _RAS0: U541.8 (I3a)
- new net _RAS1: U541.13 (I1b)
- new net _ROMEN: U500.12 (_OE)
- new net _WE: U541.17 (I3b)
- no-connect marks 0 -> 4

Commit message: Some fixes
Changed lines of the file:
@@
 Connection ~ 11750 3900
 Connection ~ 6800 3900
-Text GLabel 6800 3900 1    50   Input ~ 0
-DRAB(0:8)
 Text Label 6900 6200 0    50   ~ 0
 DRAB0
@@
 Wire Bus Line
 	15750 6800 15750 9800
-Wire Bus Line
-	3750 1850 5850 1850
-Wire Bus Line
-	3750 3250 5850 3250
-Wire Bus Line
-	5850 1850 5850 3250
-Wire Bus Line
-	1250 1200 1250 3150
-Wire Bus Line
-	4300 8500 4300 10000
-Wire Bus Line
-	11750 3900 11750 9100
-Wire Bus Line
-	2000 8100 2000 9800
-Wire Bus Line
-	13800 3900 13800 9100
-Wire Bus Line
-	9300 3900 9300 9100
-Wire Bus Line
-	6800 3900 6800 9100
-Wire Bus Line
-	7650 6800 15750 6800
-Wire Bus Line
-	7350 9800 15750 9800
 Text GLabel 7350 9800 0    50   Input ~ 0
 DRD(0:15)
+Wire Bus Line
+	3750 1850 5850 1850
+Wire Bus Line
+	3750 3250 5850 3250
+Wire Bus Line
+	5850 1850 5850 3250
+Wire Bus Line
+	1250 1200 1250 3150
+Wire Bus Line
+	4300 8500 4300 10000
+Wire Bus Line
+	11750 3900 11750 9100
+Wire Bus Line
+	2000 8100 2000 9800
+Wire Bus Line
+	13800 3900 13800 9100
+Wire Bus Line
+	9300 3900 9300 9100
+Wire Bus Line
+	6800 3900 6800 9100
+Wire Bus Line
+	7650 6800 15750 6800
+Wire Bus Line
+	7350 9800 15750 9800
 $EndSCHEMATC
