File: processor.sch (KiCad schematic (older format))
At the start: 19 parts, among them U100 MC68000, U103 74F245, U104 74LS373, U105 74F245, U106 74LS373, U303 74F08

Commit message: Update footprints
Parts:
- C1, C100, C103, C104, C105, C106: footprint (none) -> Capacitor_THT:C_Rect_L11.0mm_W2.8mm_P10.00mm_MKT
Changed lines of the file:
@@
 F 0 "C100" H 4115 7296 50  0000 L CNN
 F 1 "0.1uF" H 4115 7205 50  0000 L CNN
-F 2 "" H 4038 7100 50  0001 C CNN
+F 2 "Capacitor_THT:C_Rect_L11.0mm_W2.8mm_P10.00mm_MKT" H 4038 7100 50  0001 C CNN
 F 3 "~" H 4000 7250 50  0001 C CNN
 	1    4000 7250
@@
 F 0 "C103" H 4665 7296 50  0000 L CNN
 F 1 "0.1uF" H 4665 7205 50  0000 L CNN
-F 2 "" H 4588 7100 50  0001 C CNN
+F 2 "Capacitor_THT:C_Rect_L11.0mm_W2.8mm_P10.00mm_MKT" H 4588 7100 50  0001 C CNN
 F 3 "~" H 4550 7250 50  0001 C CNN
 	1    4550 7250
@@
 F 0 "C104" H 5215 7296 50  0000 L CNN
 F 1 "0.1uF" H 5215 7205 50  0000 L CNN
-F 2 "" H 5138 7100 50  0001 C CNN
+F 2 "Capacitor_THT:C_Rect_L11.0mm_W2.8mm_P10.00mm_MKT" H 5138 7100 50  0001 C CNN
 F 3 "~" H 5100 7250 50  0001 C CNN
 	1    5100 7250
@@
 F 0 "C105" H 5765 7296 50  0000 L CNN
 F 1 "0.1uF" H 5765 7205 50  0000 L CNN
-F 2 "" H 5688 7100 50  0001 C CNN
+F 2 "Capacitor_THT:C_Rect_L11.0mm_W2.8mm_P10.00mm_MKT" H 5688 7100 50  0001 C CNN
 F 3 "~" H 5650 7250 50  0001 C CNN
 	1    5650 7250
@@
 F 0 "C106" H 6315 7296 50  0000 L CNN
 F 1 "0.1uF" H 6315 7205 50  0000 L CNN
-F 2 "" H 6238 7100 50  0001 C CNN
+F 2 "Capacitor_THT:C_Rect_L11.0mm_W2.8mm_P10.00mm_MKT" H 6238 7100 50  0001 C CNN
 F 3 "~" H 6200 7250 50  0001 C CNN
 	1    6200 7250
@@
 F 0 "C1" H 965 3696 50  0000 L CNN
 F 1 "270pF" H 965 3605 50  0000 L CNN
-F 2 "" H 888 3500 50  0001 C CNN
+F 2 "Capacitor_THT:C_Rect_L11.0mm_W2.8mm_P10.00mm_MKT" H 888 3500 50  0001 C CNN
 F 3 "~" H 850 3650 50  0001 C CNN
 	1    850  3650

Commit message: Make caps footprint smaller
Parts:
- C1, C100, C103, C104, C105, C106: footprint Capacitor_THT:C_Rect_L11.0mm_W2.8mm_P10.00mm_MKT -> Capacitor_THT:C_Rect_L11.5mm_W2.0mm_P10.00mm_MKT
Changed lines of the file:
@@
 F 0 "C100" H 4115 7296 50  0000 L CNN
 F 1 "0.1uF" H 4115 7205 50  0000 L CNN
-F 2 "Capacitor_THT:C_Rect_L11.0mm_W2.8mm_P10.00mm_MKT" H 4038 7100 50  0001 C CNN
+F 2 "Capacitor_THT:C_Rect_L11.5mm_W2.0mm_P10.00mm_MKT" H 4038 7100 50  0001 C CNN
 F 3 "~" H 4000 7250 50  0001 C CNN
 	1    4000 7250
@@
 F 0 "C103" H 4665 7296 50  0000 L CNN
 F 1 "0.1uF" H 4665 7205 50  0000 L CNN
-F 2 "Capacitor_THT:C_Rect_L11.0mm_W2.8mm_P10.00mm_MKT" H 4588 7100 50  0001 C CNN
+F 2 "Capacitor_THT:C_Rect_L11.5mm_W2.0mm_P10.00mm_MKT" H 4588 7100 50  0001 C CNN
 F 3 "~" H 4550 7250 50  0001 C CNN
 	1    4550 7250
@@
 F 0 "C104" H 5215 7296 50  0000 L CNN
 F 1 "0.1uF" H 5215 7205 50  0000 L CNN
-F 2 "Capacitor_THT:C_Rect_L11.0mm_W2.8mm_P10.00mm_MKT" H 5138 7100 50  0001 C CNN
+F 2 "Capacitor_THT:C_Rect_L11.5mm_W2.0mm_P10.00mm_MKT" H 5138 7100 50  0001 C CNN
 F 3 "~" H 5100 7250 50  0001 C CNN
 	1    5100 7250
@@
 F 0 "C105" H 5765 7296 50  0000 L CNN
 F 1 "0.1uF" H 5765 7205 50  0000 L CNN
-F 2 "Capacitor_THT:C_Rect_L11.0mm_W2.8mm_P10.00mm_MKT" H 5688 7100 50  0001 C CNN
+F 2 "Capacitor_THT:C_Rect_L11.5mm_W2.0mm_P10.00mm_MKT" H 5688 7100 50  0001 C CNN
 F 3 "~" H 5650 7250 50  0001 C CNN
 	1    5650 7250
@@
 F 0 "C106" H 6315 7296 50  0000 L CNN
 F 1 "0.1uF" H 6315 7205 50  0000 L CNN
-F 2 "Capacitor_THT:C_Rect_L11.0mm_W2.8mm_P10.00mm_MKT" H 6238 7100 50  0001 C CNN
+F 2 "Capacitor_THT:C_Rect_L11.5mm_W2.0mm_P10.00mm_MKT" H 6238 7100 50  0001 C CNN
 F 3 "~" H 6200 7250 50  0001 C CNN
 	1    6200 7250
@@
 F 0 "C1" H 965 3696 50  0000 L CNN
 F 1 "270pF" H 965 3605 50  0000 L CNN
-F 2 "Capacitor_THT:C_Rect_L11.0mm_W2.8mm_P10.00mm_MKT" H 888 3500 50  0001 C CNN
+F 2 "Capacitor_THT:C_Rect_L11.5mm_W2.0mm_P10.00mm_MKT" H 888 3500 50  0001 C CNN
 F 3 "~" H 850 3650 50  0001 C CNN
 	1    850  3650

Commit message: Switch footprints for suitable modern replacements
Parts:
- C1, C100, C103, C104, C105, C106: footprint Capacitor_THT:C_Rect_L11.5mm_W2.0mm_P10.00mm_MKT -> Capacitor_THT:C_Rect_L11.5mm_W2.6mm_P10.00mm_MKT
Changed lines of the file:
@@
 F 0 "C100" H 4115 7296 50  0000 L CNN
 F 1 "0.1uF" H 4115 7205 50  0000 L CNN
-F 2 "Capacitor_THT:C_Rect_L11.5mm_W2.0mm_P10.00mm_MKT" H 4038 7100 50  0001 C CNN
+F 2 "Capacitor_THT:C_Rect_L11.5mm_W2.6mm_P10.00mm_MKT" H 4038 7100 50  0001 C CNN
 F 3 "~" H 4000 7250 50  0001 C CNN
 	1    4000 7250
@@
 F 0 "C103" H 4665 7296 50  0000 L CNN
 F 1 "0.1uF" H 4665 7205 50  0000 L CNN
-F 2 "Capacitor_THT:C_Rect_L11.5mm_W2.0mm_P10.00mm_MKT" H 4588 7100 50  0001 C CNN
+F 2 "Capacitor_THT:C_Rect_L11.5mm_W2.6mm_P10.00mm_MKT" H 4588 7100 50  0001 C CNN
 F 3 "~" H 4550 7250 50  0001 C CNN
 	1    4550 7250
@@
 F 0 "C104" H 5215 7296 50  0000 L CNN
 F 1 "0.1uF" H 5215 7205 50  0000 L CNN
-F 2 "Capacitor_THT:C_Rect_L11.5mm_W2.0mm_P10.00mm_MKT" H 5138 7100 50  0001 C CNN
+F 2 "Capacitor_THT:C_Rect_L11.5mm_W2.6mm_P10.00mm_MKT" H 5138 7100 50  0001 C CNN
 F 3 "~" H 5100 7250 50  0001 C CNN
 	1    5100 7250
@@
 F 0 "C105" H 5765 7296 50  0000 L CNN
 F 1 "0.1uF" H 5765 7205 50  0000 L CNN
-F 2 "Capacitor_THT:C_Rect_L11.5mm_W2.0mm_P10.00mm_MKT" H 5688 7100 50  0001 C CNN
+F 2 "Capacitor_THT:C_Rect_L11.5mm_W2.6mm_P10.00mm_MKT" H 5688 7100 50  0001 C CNN
 F 3 "~" H 5650 7250 50  0001 C CNN
 	1    5650 7250
@@
 F 0 "C106" H 6315 7296 50  0000 L CNN
 F 1 "0.1uF" H 6315 7205 50  0000 L CNN
-F 2 "Capacitor_THT:C_Rect_L11.5mm_W2.0mm_P10.00mm_MKT" H 6238 7100 50  0001 C CNN
+F 2 "Capacitor_THT:C_Rect_L11.5mm_W2.6mm_P10.00mm_MKT" H 6238 7100 50  0001 C CNN
 F 3 "~" H 6200 7250 50  0001 C CNN
 	1    6200 7250
@@
 F 0 "C1" H 965 3696 50  0000 L CNN
 F 1 "270pF" H 965 3605 50  0000 L CNN
-F 2 "Capacitor_THT:C_Rect_L11.5mm_W2.0mm_P10.00mm_MKT" H 888 3500 50  0001 C CNN
+F 2 "Capacitor_THT:C_Rect_L11.5mm_W2.6mm_P10.00mm_MKT" H 888 3500 50  0001 C CNN
 F 3 "~" H 850 3650 50  0001 C CNN
 	1    850  3650

Commit message: Some footprints updates; Add all Mouser references
Parts:
- C1: RefOrder (none) -> 581-SA101A271KAA
- C100, C103, C104, C105, C106: RefOrder (none) -> 581-SA105C104KARC
- R1: RefOrder (none) -> 603-CFR-25JT-52-68R
- R1000, R111, R917: RefOrder (none) -> 603-CFR-25JT-52-330R
- R104: RefOrder (none) -> 603-CFR-25JR-524K7
- RP100, RP101: value 4.7K -> 4.7k; RefOrder (none) -> 858-L101S472LF
- U103, U105: RefOrder (none) -> 595-SN74F245N
- U104, U106: RefOrder (none) -> 595-SN74LS373N
- U303: RefOrder (none) -> 595-SN74F08N
Changed lines of the file:
@@
 F 2 "Package_DIP:DIP-20_W7.62mm_Socket" H 7600 1850 50  0001 C CNN
 F 3 "http://www.mouser.com/ds/2/308/fairchild%20semiconductor_74f245-1116738.pdf" H 7600 1850 50  0001 C CNN
+F 4 "595-SN74F245N" H 7600 1850 50  0001 C CNN "RefOrder"
 	1    7600 1850
 	1    0    0    -1
@@
 F 2 "Package_DIP:DIP-20_W7.62mm_Socket" H 7600 4950 50  0001 C CNN
 F 3 "http://www.mouser.com/ds/2/308/fairchild%20semiconductor_74f245-1116738.pdf" H 7600 4950 50  0001 C CNN
+F 4 "595-SN74F245N" H 7600 4950 50  0001 C CNN "RefOrder"
 	1    7600 4950
 	1    0    0    -1
@@
 F 2 "Package_DIP:DIP-20_W7.62mm_Socket" H 10100 1850 50  0001 C CNN
 F 3 "http://www.ti.com/lit/gpn/sn74LS373" H 10100 1850 50  0001 C CNN
+F 4 "595-SN74LS373N" H 10100 1850 50  0001 C CNN "RefOrder"
 	1    10100 1850
 	1    0    0    -1
@@
 F 2 "Package_DIP:DIP-20_W7.62mm_Socket" H 10100 4950 50  0001 C CNN
 F 3 "http://www.ti.com/lit/gpn/sn74LS373" H 10100 4950 50  0001 C CNN
+F 4 "595-SN74LS373N" H 10100 4950 50  0001 C CNN "RefOrder"
 	1    10100 4950
 	1    0    0    -1
@@
 F 2 "Package_DIP:DIP-14_W7.62mm_Socket" H 1500 1550 50  0001 C CNN
 F 3 "http://www.ti.com/lit/ds/symlink/sn74f08.pdf" H 1500 1550 50  0001 C CNN
+F 4 "595-SN74F08N" H 1500 1550 50  0001 C CNN "RefOrder"
 	4    1500 1550
 	1    0    0    -1
@@
 P 2450 1200
 F 0 "RP100" H 1970 1246 50  0000 R CNN
-F 1 "4.7K" H 1970 1155 50  0000 R CNN
+F 1 "4.7k" H 1970 1155 50  0000 R CNN
 F 2 "Resistor_THT:R_Array_SIP10" V 3025 1200 50  0001 C CNN
 F 3 "http://www.vishay.com/docs/31509/csc.pdf" H 2450 1200 50  0001 C CNN
+F 4 "858-L101S472LF" H 2450 1200 50  0001 C CNN "RefOrder"
 	1    2450 1200
 	-1   0    0    -1
@@
 F 2 "Resistor_THT:R_Axial_DIN0207_L6.3mm_D2.5mm_P10.16mm_Horizontal" V 930 1150 50  0001 C CNN
 F 3 "~" H 1000 1150 50  0001 C CNN
+F 4 "603-CFR-25JR-524K7" H 1000 1150 50  0001 C CNN "RefOrder"
 	1    1000 1150
 	1    0    0    -1
@@
 F 2 "Resistor_THT:R_Axial_DIN0207_L6.3mm_D2.5mm_P10.16mm_Horizontal" V 3680 4050 50  0001 C CNN
 F 3 "~" H 3750 4050 50  0001 C CNN
+F 4 "603-CFR-25JT-52-330R" H 3750 4050 50  0001 C CNN "RefOrder"
 	1    3750 4050
 	1    0    0    -1
@@
 F 2 "Capacitor_THT:C_Rect_L11.5mm_W2.6mm_P10.00mm_MKT" H 4038 7100 50  0001 C CNN
 F 3 "~" H 4000 7250 50  0001 C CNN
+F 4 "581-SA105C104KARC" H 4000 7250 50  0001 C CNN "RefOrder"
 	1    4000 7250
 	1    0    0    -1
@@
 F 2 "Capacitor_THT:C_Rect_L11.5mm_W2.6mm_P10.00mm_MKT" H 4588 7100 50  0001 C CNN
 F 3 "~" H 4550 7250 50  0001 C CNN
+F 4 "581-SA105C104KARC" H 4550 7250 50  0001 C CNN "RefOrder"
 	1    4550 7250
 	1    0    0    -1
@@
 F 2 "Capacitor_THT:C_Rect_L11.5mm_W2.6mm_P10.00mm_MKT" H 5138 7100 50  0001 C CNN
 F 3 "~" H 5100 7250 50  0001 C CNN
+F 4 "581-SA105C104KARC" H 5100 7250 50  0001 C CNN "RefOrder"
 	1    5100 7250
 	1    0    0    -1
@@
 F 2 "Capacitor_THT:C_Rect_L11.5mm_W2.6mm_P10.00mm_MKT" H 5688 7100 50  0001 C CNN
 F 3 "~" H 5650 7250 50  0001 C CNN
+F 4 "581-SA105C104KARC" H 5650 7250 50  0001 C CNN "RefOrder"
 	1    5650 7250
 	1    0    0    -1
@@
 F 2 "Capacitor_THT:C_Rect_L11.5mm_W2.6mm_P10.00mm_MKT" H 6238 7100 50  0001 C CNN
 F 3 "~" H 6200 7250 50  0001 C CNN
+F 4 "581-SA105C104KARC" H 6200 7250 50  0001 C CNN "RefOrder"
 	1    6200 7250
 	1    0    0    -1
@@
 P 2750 7200
 F 0 "RP101" H 2271 7154 50  0000 R CNN
-F 1 "4.7K" H 2271 7245 50  0000 R CNN
+F 1 "4.7k" H 2271 7245 50  0000 R CNN
 F 2 "Resistor_THT:R_Array_SIP10" V 3325 7200 50  0001 C CNN
 F 3 "http://www.vishay.com/docs/31509/csc.pdf" H 2750 7200 50  0001 C CNN
+F 4 "858-L101S472LF" H 2750 7200 50  0001 C CNN "RefOrder"
 	1    2750 7200
 	1    0    0    1
@@
 F 2 "Resistor_THT:R_Axial_DIN0207_L6.3mm_D2.5mm_P10.16mm_Horizontal" V 3180 4050 50  0001 C CNN
 F 3 "~" H 3250 4050 50  0001 C CNN
+F 4 "603-CFR-25JT-52-330R" H 3250 4050 50  0001 C CNN "RefOrder"
 	1    3250 4050
 	1    0    0    -1
@@
 F 2 "Resistor_THT:R_Axial_DIN0207_L6.3mm_D2.5mm_P10.16mm_Horizontal" V 3430 3750 50  0001 C CNN
 F 3 "~" H 3500 3750 50  0001 C CNN
+F 4 "603-CFR-25JT-52-330R" H 3500 3750 50  0001 C CNN "RefOrder"
 	1    3500 3750
 	1    0    0    -1
@@
 F 2 "Resistor_THT:R_Axial_DIN0207_L6.3mm_D2.5mm_P10.16mm_Horizontal" V 780 3950 50  0001 C CNN
 F 3 "~" H 850 3950 50  0001 C CNN
+F 4 "603-CFR-25JT-52-68R" H 850 3950 50  0001 C CNN "RefOrder"
 	1    850  3950
 	1    0    0    -1
@@
 F 2 "Capacitor_THT:C_Rect_L11.5mm_W2.6mm_P10.00mm_MKT" H 888 3500 50  0001 C CNN
 F 3 "~" H 850 3650 50  0001 C CNN
+F 4 "581-SA101A271KAA" H 850 3650 50  0001 C CNN "RefOrder"
 	1    850  3650
 	1    0    0    -1
