File: coprocessor slot.sch (KiCad schematic (older format))
At the start: 0 parts

Commit message: All done; now to review
Parts:
- added C600, C601, C602, C603, C604, C605: 0.1uF, symbol Device:C
- added CN600: CO-PROCESSOR_SLOT, symbol amiga_customs:CO-PROCESSOR_SLOT
- added RP900: 3.2k, Resistor_THT:R_Array_SIP10, symbol Device:R_Network09
- added RP901: 3.3k, Resistor_THT:R_Array_SIP10, symbol Device:R_Network09
- added RP903, RP908: 1k, Resistor_THT:R_Array_SIP6, symbol Device:R_Network05
- added U600, U601, U603, U604: 74LS245, symbol 74xx:74LS245
- added U602, U605: 74ALS245, symbol 74xx:74LS245
Connections:
- new net: RP908.5 (R4), U605.18 (B0)
- new net: RP908.6 (R5), U605.2 (A0)
- new net +12V: CN600.~ (9)
- new net +5V: C600.1, C601.1, C602.1, C603.1, C604.1, C605.2, CN600.~ (9), RP900.1 (common), RP901.1 (common), RP903.1 (common), RP908.1 (common), U600.20 (VCC), U601.20 (VCC), U602.20 (VCC), U603.20 (VCC), U604.20 (VCC), U605.20 (VCC)
- new net -5V: CN600.~ (9)
- new net 28M: CN600.~ (9)
- new net A1: CN600.~ (9), U600.8 (A6)
- new net A10: CN600.~ (9), U601.4 (A2)
- new net A11: CN600.~ (9), U601.5 (A3)
- new net A12: CN600.~ (9), U601.6 (A4)
- new net A13: CN600.~ (9), U601.7 (A5)
- new net A14: CN600.~ (9), U601.8 (A6)
- new net A15: CN600.~ (9), U601.9 (A7)
- new net A16: CN600.~ (9), U602.2 (A0)
- new net A17: CN600.~ (9), U602.3 (A1)
- new net A18: CN600.~ (9), U602.4 (A2)
- new net A19: CN600.~ (9), U602.5 (A3)
- new net A2: CN600.~ (9), U600.7 (A5)
- new net A20: CN600.~ (9), U602.6 (A4)
- new net A21: CN600.~ (9), U602.7 (A5)
- new net A22: CN600.~ (9), U602.8 (A6)
- new net A23: CN600.~ (9), U602.9 (A7)
- new net A3: CN600.~ (9), U600.6 (A4)
- new net A4: CN600.~ (9), U600.5 (A3)
- new net A5: CN600.~ (9), U600.4 (A2)
- new net A6: CN600.~ (9), U600.3 (A1)
- new net A7: CN600.~ (9), U600.2 (A0)
- new net A8: CN600.~ (9), U601.2 (A0)
- new net A9: CN600.~ (9), U601.3 (A1)
- new net BA1: U600.12 (B6)
- new net BA10: U601.16 (B2)
- new net BA11: U601.15 (B3)
- new net BA12: U601.14 (B4)
- new net BA13: U601.13 (B5)
- new net BA14: U601.12 (B6)
- new net BA15: U601.11 (B7)
- new net BA16: U602.18 (B0)
- new net BA17: U602.17 (B1)
- new net BA18: U602.16 (B2)
- new net BA19: U602.15 (B3)
- new net BA2: U600.13 (B5)
- new net BA20: U602.14 (B4)
- new net BA21: U602.13 (B5)
- new net BA22: U602.12 (B6)
- new net BA23: U602.11 (B7)
- new net BA3: U600.14 (B4)
- new net BA4: U600.15 (B3)
- new net BA5: U600.16 (B2)
- new net BA6: U600.17 (B1)
- new net BA7: U600.18 (B0)
- new net BA8: U601.18 (B0)
- new net BA9: U601.17 (B1)
- new net BD0: U603.18 (B0)
- new net BD1: U603.17 (B1)
- new net BD10: U604.13 (B5)
- new net BD11: U604.14 (B4)
- new net BD12: U604.15 (B3)
- new net BD13: U604.16 (B2)
- new net BD14: U604.17 (B1)
- new net BD15: U604.18 (B0)
- new net BD2: U603.16 (B2)
- new net BD3: U603.15 (B3)
- new net BD4: U603.14 (B4)
- new net BD5: U603.13 (B5)
- new net BD6: U603.12 (B6)
- new net BD7: U603.11 (B7)
- new net BD8: U604.11 (B7)
- new net BD9: U604.12 (B6)
- new net BFC0: RP908.2 (R1), U605.15 (B3)
- new net BFC1: RP908.3 (R2), U605.16 (B2)
- new net BFC2: RP908.4 (R3), U605.17 (B1)
- new net D0: CN600.~ (9), RP900.9 (R8), U603.2 (A0)
- new net D1: CN600.~ (9), RP900.8 (R7), U603.3 (A1)
- new net D10: CN600.~ (9), RP901.4 (R3), U604.7 (A5)
- new net D11: CN600.~ (9), RP901.5 (R4), U604.6 (A4)
- new net D12: CN600.~ (9), RP901.6 (R5), U604.5 (A3)
- new net D13: CN600.~ (9), RP901.7 (R6), U604.4 (A2)
- new net D14: CN600.~ (9), RP901.8 (R7), U604.3 (A1)
- new net D15: CN600.~ (9), RP901.9 (R8), U604.2 (A0)
- new net D2: CN600.~ (9), RP900.7 (R6), U603.4 (A2)
- new net D3: CN600.~ (9), RP900.5 (R4), U603.5 (A3)
- new net D4: CN600.~ (9), RP900.3 (R2), U603.6 (A4)
- new net D5: CN600.~ (9), RP900.2 (R1), U603.7 (A5)
- new net D6: CN600.~ (9), RP900.4 (R3), U603.8 (A6)
- new net D7: CN600.~ (9), RP900.6 (R5), U603.9 (A7)
- new net D8: CN600.~ (9), RP901.2 (R1), U604.9 (A7)
- new net D9: CN600.~ (9), RP901.3 (R2), U604.8 (A6)
- new net DMAOUT: U600.1 (A->B), U601.1 (A->B), U602.1 (A->B), U605.1 (A->B)
- new net E: CN600.~ (9)
- new net FC0: CN600.~ (9), U605.5 (A3)
- new net FC1: CN600.~ (9), U605.4 (A2)
- new net FC2: CN600.~ (9), U605.3 (A1)
- new net GND: C600.2, C601.2, C602.2, C603.2, C604.2, C605.1, CN600.~ (9), U600.10 (GND), U600.19 (CE), U601.10 (GND), U601.19 (CE), U602.10 (GND), U602.19 (CE), U603.10 (GND), U604.10 (GND), U605.10 (GND), U605.19 (CE)
- new net READ: RP903.3 (R2), U605.14 (B4)
- new net R_W: CN600.~ (9), U605.6 (A4)
- new net V7M: CN600.~ (9)
- new net VCDAC: CN600.~ (9)
- new net XRDY: CN600.~ (9)
- new net _AS: CN600.~ (9), U605.9 (A7)
- new net _BAS: RP903.6 (R5), U605.11 (B7)
- new net _BEER: CN600.~ (9)
- new net _BGACK: CN600.~ (9)
- new net _BLDS: RP903.4 (R3), U605.13 (B5)
- new net _BOSS: CN600.~ (9)
- new net _BUDS: RP903.5 (R4), U605.12 (B6)
- new net _CBG: CN600.~ (9)
- new net _CBR: CN600.~ (9)
- new net _COPCFG: CN600.~ (9)
- new net _D2P: U603.1 (A->B), U604.1 (A->B)
- new net _DBOE: U603.19 (CE), U604.19 (CE)
- new net _DTACK: CN600.~ (9)
- new net _HLT: CN600.~ (9)
- new net _INT2: CN600.~ (9)
- new net _INT6: CN600.~ (9)
- new net _IPL0: CN600.~ (9)
- new net _IPL1: CN600.~ (9)
- new net _IPL2: CN600.~ (9)
- new net _LDS: CN600.~ (9), U605.7 (A5)
- new net _OVR: CN600.~ (9)
- new net _RST: CN600.~ (9)
- new net _UDS: CN600.~ (9), U605.8 (A6)
- new net _VC1: CN600.~ (9)
- new net _VC3: CN600.~ (9)
- new net _VMA: CN600.~ (9)
- new net _VPA: CN600.~ (9)
- no-connect marks 0 -> 5
