File: coprocessor slot.sch (KiCad schematic (older format))
At the start: 17 parts, among them CN600 CO-PROCESSOR_SLOT, U600 74LS245, U601 74LS245, U602 74ALS245, U603 74LS245, U604 74LS245, U605 74ALS245

Commit message: Update footprints
Parts:
- C600, C601, C602, C603, C604, C605: footprint (none) -> Capacitor_THT:C_Rect_L11.0mm_W2.8mm_P10.00mm_MKT
- CN600: footprint (none) -> d_amiga:COPRO
Changed lines of the file:
@@
 F 0 "CN600" H 5975 1175 50  0000 C CNN
 F 1 "CO-PROCESSOR_SLOT" H 5975 1084 50  0000 C CNN
-F 2 "" H 5950 1050 50  0001 C CNN
+F 2 "d_amiga:COPRO" H 5950 1050 50  0001 C CNN
 F 3 "" H 5950 1050 50  0001 C CNN
 	1    5950 1000
@@
 F 0 "C602" H 9565 5496 50  0000 L CNN
 F 1 "0.1uF" H 9565 5405 50  0000 L CNN
-F 2 "" H 9488 5300 50  0001 C CNN
+F 2 "Capacitor_THT:C_Rect_L11.0mm_W2.8mm_P10.00mm_MKT" H 9488 5300 50  0001 C CNN
 F 3 "~" H 9450 5450 50  0001 C CNN
 	1    9450 5450
@@
 F 0 "C601" H 9565 3496 50  0000 L CNN
 F 1 "0.1uF" H 9565 3405 50  0000 L CNN
-F 2 "" H 9488 3300 50  0001 C CNN
+F 2 "Capacitor_THT:C_Rect_L11.0mm_W2.8mm_P10.00mm_MKT" H 9488 3300 50  0001 C CNN
 F 3 "~" H 9450 3450 50  0001 C CNN
 	1    9450 3450
@@
 F 0 "C600" H 9515 1546 50  0000 L CNN
 F 1 "0.1uF" H 9515 1455 50  0000 L CNN
-F 2 "" H 9438 1350 50  0001 C CNN
+F 2 "Capacitor_THT:C_Rect_L11.0mm_W2.8mm_P10.00mm_MKT" H 9438 1350 50  0001 C CNN
 F 3 "~" H 9400 1500 50  0001 C CNN
 	1    9400 1500
@@
 F 0 "C603" H 16015 7996 50  0000 L CNN
 F 1 "0.1uF" H 16015 7905 50  0000 L CNN
-F 2 "" H 15938 7800 50  0001 C CNN
+F 2 "Capacitor_THT:C_Rect_L11.0mm_W2.8mm_P10.00mm_MKT" H 15938 7800 50  0001 C CNN
 F 3 "~" H 15900 7950 50  0001 C CNN
 	1    15900 7950
@@
 F 0 "C604" H 16015 10046 50  0000 L CNN
 F 1 "0.1uF" H 16015 9955 50  0000 L CNN
-F 2 "" H 15938 9850 50  0001 C CNN
+F 2 "Capacitor_THT:C_Rect_L11.0mm_W2.8mm_P10.00mm_MKT" H 15938 9850 50  0001 C CNN
 F 3 "~" H 15900 10000 50  0001 C CNN
 	1    15900 10000
@@
 F 0 "C605" H 9215 12896 50  0000 L CNN
 F 1 "0.1uF" H 9215 12805 50  0000 L CNN
-F 2 "" H 9138 12700 50  0001 C CNN
+F 2 "Capacitor_THT:C_Rect_L11.0mm_W2.8mm_P10.00mm_MKT" H 9138 12700 50  0001 C CNN
 F 3 "~" H 9100 12850 50  0001 C CNN
 	1    9100 12850

Commit message: Make caps footprint smaller
Parts:
- C600, C601, C602, C603, C604, C605: footprint Capacitor_THT:C_Rect_L11.0mm_W2.8mm_P10.00mm_MKT -> Capacitor_THT:C_Rect_L11.5mm_W2.0mm_P10.00mm_MKT
Changed lines of the file:
@@
 F 0 "C602" H 9565 5496 50  0000 L CNN
 F 1 "0.1uF" H 9565 5405 50  0000 L CNN
-F 2 "Capacitor_THT:C_Rect_L11.0mm_W2.8mm_P10.00mm_MKT" H 9488 5300 50  0001 C CNN
+F 2 "Capacitor_THT:C_Rect_L11.5mm_W2.0mm_P10.00mm_MKT" H 9488 5300 50  0001 C CNN
 F 3 "~" H 9450 5450 50  0001 C CNN
 	1    9450 5450
@@
 F 0 "C601" H 9565 3496 50  0000 L CNN
 F 1 "0.1uF" H 9565 3405 50  0000 L CNN
-F 2 "Capacitor_THT:C_Rect_L11.0mm_W2.8mm_P10.00mm_MKT" H 9488 3300 50  0001 C CNN
+F 2 "Capacitor_THT:C_Rect_L11.5mm_W2.0mm_P10.00mm_MKT" H 9488 3300 50  0001 C CNN
 F 3 "~" H 9450 3450 50  0001 C CNN
 	1    9450 3450
@@
 F 0 "C600" H 9515 1546 50  0000 L CNN
 F 1 "0.1uF" H 9515 1455 50  0000 L CNN
-F 2 "Capacitor_THT:C_Rect_L11.0mm_W2.8mm_P10.00mm_MKT" H 9438 1350 50  0001 C CNN
+F 2 "Capacitor_THT:C_Rect_L11.5mm_W2.0mm_P10.00mm_MKT" H 9438 1350 50  0001 C CNN
 F 3 "~" H 9400 1500 50  0001 C CNN
 	1    9400 1500
@@
 F 0 "C603" H 16015 7996 50  0000 L CNN
 F 1 "0.1uF" H 16015 7905 50  0000 L CNN
-F 2 "Capacitor_THT:C_Rect_L11.0mm_W2.8mm_P10.00mm_MKT" H 15938 7800 50  0001 C CNN
+F 2 "Capacitor_THT:C_Rect_L11.5mm_W2.0mm_P10.00mm_MKT" H 15938 7800 50  0001 C CNN
 F 3 "~" H 15900 7950 50  0001 C CNN
 	1    15900 7950
@@
 F 0 "C604" H 16015 10046 50  0000 L CNN
 F 1 "0.1uF" H 16015 9955 50  0000 L CNN
-F 2 "Capacitor_THT:C_Rect_L11.0mm_W2.8mm_P10.00mm_MKT" H 15938 9850 50  0001 C CNN
+F 2 "Capacitor_THT:C_Rect_L11.5mm_W2.0mm_P10.00mm_MKT" H 15938 9850 50  0001 C CNN
 F 3 "~" H 15900 10000 50  0001 C CNN
 	1    15900 10000
@@
 F 0 "C605" H 9215 12896 50  0000 L CNN
 F 1 "0.1uF" H 9215 12805 50  0000 L CNN
-F 2 "Capacitor_THT:C_Rect_L11.0mm_W2.8mm_P10.00mm_MKT" H 9138 12700 50  0001 C CNN
+F 2 "Capacitor_THT:C_Rect_L11.5mm_W2.0mm_P10.00mm_MKT" H 9138 12700 50  0001 C CNN
 F 3 "~" H 9100 12850 50  0001 C CNN
 	1    9100 12850
