File: coprocessor slot.sch (KiCad schematic (older format))
At the start: 17 parts, among them CN600 CO-PROCESSOR_SLOT, U600 74LS245, U601 74LS245, U602 74ALS245, U603 74LS245, U604 74LS245, U605 74ALS245

Commit message: Switch footprints for suitable modern replacements
Parts:
- C600, C601, C602, C603, C604, C605: footprint Capacitor_THT:C_Rect_L11.5mm_W2.0mm_P10.00mm_MKT -> Capacitor_THT:C_Rect_L11.5mm_W2.6mm_P10.00mm_MKT
Changed lines of the file:
@@
 F 0 "C602" H 9565 5496 50  0000 L CNN
 F 1 "0.1uF" H 9565 5405 50  0000 L CNN
-F 2 "Capacitor_THT:C_Rect_L11.5mm_W2.0mm_P10.00mm_MKT" H 9488 5300 50  0001 C CNN
+F 2 "Capacitor_THT:C_Rect_L11.5mm_W2.6mm_P10.00mm_MKT" H 9488 5300 50  0001 C CNN
 F 3 "~" H 9450 5450 50  0001 C CNN
 	1    9450 5450
@@
 F 0 "C601" H 9565 3496 50  0000 L CNN
 F 1 "0.1uF" H 9565 3405 50  0000 L CNN
-F 2 "Capacitor_THT:C_Rect_L11.5mm_W2.0mm_P10.00mm_MKT" H 9488 3300 50  0001 C CNN
+F 2 "Capacitor_THT:C_Rect_L11.5mm_W2.6mm_P10.00mm_MKT" H 9488 3300 50  0001 C CNN
 F 3 "~" H 9450 3450 50  0001 C CNN
 	1    9450 3450
@@
 F 0 "C600" H 9515 1546 50  0000 L CNN
 F 1 "0.1uF" H 9515 1455 50  0000 L CNN
-F 2 "Capacitor_THT:C_Rect_L11.5mm_W2.0mm_P10.00mm_MKT" H 9438 1350 50  0001 C CNN
+F 2 "Capacitor_THT:C_Rect_L11.5mm_W2.6mm_P10.00mm_MKT" H 9438 1350 50  0001 C CNN
 F 3 "~" H 9400 1500 50  0001 C CNN
 	1    9400 1500
@@
 F 0 "C603" H 16015 7996 50  0000 L CNN
 F 1 "0.1uF" H 16015 7905 50  0000 L CNN
-F 2 "Capacitor_THT:C_Rect_L11.5mm_W2.0mm_P10.00mm_MKT" H 15938 7800 50  0001 C CNN
+F 2 "Capacitor_THT:C_Rect_L11.5mm_W2.6mm_P10.00mm_MKT" H 15938 7800 50  0001 C CNN
 F 3 "~" H 15900 7950 50  0001 C CNN
 	1    15900 7950
@@
 F 0 "C604" H 16015 10046 50  0000 L CNN
 F 1 "0.1uF" H 16015 9955 50  0000 L CNN
-F 2 "Capacitor_THT:C_Rect_L11.5mm_W2.0mm_P10.00mm_MKT" H 15938 9850 50  0001 C CNN
+F 2 "Capacitor_THT:C_Rect_L11.5mm_W2.6mm_P10.00mm_MKT" H 15938 9850 50  0001 C CNN
 F 3 "~" H 15900 10000 50  0001 C CNN
 	1    15900 10000
@@
 F 0 "C605" H 9215 12896 50  0000 L CNN
 F 1 "0.1uF" H 9215 12805 50  0000 L CNN
-F 2 "Capacitor_THT:C_Rect_L11.5mm_W2.0mm_P10.00mm_MKT" H 9138 12700 50  0001 C CNN
+F 2 "Capacitor_THT:C_Rect_L11.5mm_W2.6mm_P10.00mm_MKT" H 9138 12700 50  0001 C CNN
 F 3 "~" H 9100 12850 50  0001 C CNN
 	1    9100 12850

Commit message: Some footprints updates; Add all Mouser references
Parts:
- C600, C601, C602, C603, C604, C605: RefOrder (none) -> 581-SA105C104KARC
- RP903, RP908: RefOrder (none) -> 652-4606M-1LF-1K
- RPF603, RPF604: RefOrder (none) -> 652-4610X-1LF-3.3K
- U600, U601, U603, U604: RefOrder (none) -> 595-SN74LS245N
- U602, U605: RefOrder (none) -> 595-SN74ALS245AN
Changed lines of the file:
@@
 F 2 "Package_DIP:DIP-20_W7.62mm_Socket" H 11000 1500 50  0001 C CNN
 F 3 "http://www.ti.com/lit/gpn/sn74LS245" H 11000 1500 50  0001 C CNN
+F 4 "595-SN74LS245N" H 11000 1500 50  0001 C CNN "RefOrder"
 	1    11000 1500
 	1    0    0    -1
@@
 F 2 "Package_DIP:DIP-20_W7.62mm_Socket" H 11000 3500 50  0001 C CNN
 F 3 "http://www.ti.com/lit/gpn/sn74LS245" H 11000 3500 50  0001 C CNN
+F 4 "595-SN74LS245N" H 11000 3500 50  0001 C CNN "RefOrder"
 	1    11000 3500
 	1    0    0    -1
@@
 F 2 "Package_DIP:DIP-20_W7.62mm_Socket" H 11000 5500 50  0001 C CNN
 F 3 "http://www.ti.com/lit/ds/symlink/sn74als245a.pdf" H 11000 5500 50  0001 C CNN
+F 4 "595-SN74ALS245AN" H 11000 5500 50  0001 C CNN "RefOrder"
 	1    11000 5500
 	1    0    0    -1
@@
 F 2 "Package_DIP:DIP-20_W7.62mm_Socket" H 12500 8000 50  0001 C CNN
 F 3 "http://www.ti.com/lit/gpn/sn74LS245" H 12500 8000 50  0001 C CNN
+F 4 "595-SN74LS245N" H 12500 8000 50  0001 C CNN "RefOrder"
 	1    12500 8000
 	1    0    0    -1
@@
 F 2 "Package_DIP:DIP-20_W7.62mm_Socket" H 12500 10000 50  0001 C CNN
 F 3 "http://www.ti.com/lit/gpn/sn74LS245" H 12500 10000 50  0001 C CNN
+F 4 "595-SN74LS245N" H 12500 10000 50  0001 C CNN "RefOrder"
 	1    12500 10000
 	1    0    0    -1
@@
 F 2 "Package_DIP:DIP-20_W7.62mm_Socket" H 11000 12500 50  0001 C CNN
 F 3 "http://www.ti.com/lit/ds/symlink/sn74als245a.pdf" H 11000 12500 50  0001 C CNN
+F 4 "595-SN74ALS245AN" H 11000 12500 50  0001 C CNN "RefOrder"
 	1    11000 12500
 	1    0    0    1
@@
 F 2 "Capacitor_THT:C_Rect_L11.5mm_W2.6mm_P10.00mm_MKT" H 9488 5300 50  0001 C CNN
 F 3 "~" H 9450 5450 50  0001 C CNN
+F 4 "581-SA105C104KARC" H 9450 5450 50  0001 C CNN "RefOrder"
 	1    9450 5450
 	1    0    0    -1
@@
 F 2 "Capacitor_THT:C_Rect_L11.5mm_W2.6mm_P10.00mm_MKT" H 9488 3300 50  0001 C CNN
 F 3 "~" H 9450 3450 50  0001 C CNN
+F 4 "581-SA105C104KARC" H 9450 3450 50  0001 C CNN "RefOrder"
 	1    9450 3450
 	1    0    0    -1
@@
 F 2 "Capacitor_THT:C_Rect_L11.5mm_W2.6mm_P10.00mm_MKT" H 9438 1350 50  0001 C CNN
 F 3 "~" H 9400 1500 50  0001 C CNN
+F 4 "581-SA105C104KARC" H 9400 1500 50  0001 C CNN "RefOrder"
 	1    9400 1500
 	1    0    0    -1
@@
 F 2 "Resistor_THT:R_Array_SIP6" V 13425 11550 50  0001 C CNN
 F 3 "http://www.vishay.com/docs/31509/csc.pdf" H 13050 11550 50  0001 C CNN
+F 4 "652-4606M-1LF-1K" H 13050 11550 50  0001 C CNN "RefOrder"
 	1    13050 11550
 	-1   0    0    -1
@@
 F 2 "Resistor_THT:R_Array_SIP6" V 14725 11550 50  0001 C CNN
 F 3 "http://www.vishay.com/docs/31509/csc.pdf" H 14350 11550 50  0001 C CNN
+F 4 "652-4606M-1LF-1K" H 14350 11550 50  0001 C CNN "RefOrder"
 	1    14350 11550
 	-1   0    0    -1
@@
 F 2 "Capacitor_THT:C_Rect_L11.5mm_W2.6mm_P10.00mm_MKT" H 15938 7800 50  0001 C CNN
 F 3 "~" H 15900 7950 50  0001 C CNN
+F 4 "581-SA105C104KARC" H 15900 7950 50  0001 C CNN "RefOrder"
 	1    15900 7950
 	1    0    0    -1
@@
 F 2 "Capacitor_THT:C_Rect_L11.5mm_W2.6mm_P10.00mm_MKT" H 15938 9850 50  0001 C CNN
 F 3 "~" H 15900 10000 50  0001 C CNN
+F 4 "581-SA105C104KARC" H 15900 10000 50  0001 C CNN "RefOrder"
 	1    15900 10000
 	1    0    0    -1
@@
 F 2 "Capacitor_THT:C_Rect_L11.5mm_W2.6mm_P10.00mm_MKT" H 9138 12700 50  0001 C CNN
 F 3 "~" H 9100 12850 50  0001 C CNN
+F 4 "581-SA105C104KARC" H 9100 12850 50  0001 C CNN "RefOrder"
 	1    9100 12850
 	1    0    0    -1
@@
 F 2 "Resistor_THT:R_Array_SIP10" V 11175 9800 50  0001 C CNN
 F 3 "http://www.vishay.com/docs/31509/csc.pdf" H 10600 9800 50  0001 C CNN
+F 4 "652-4610X-1LF-3.3K" H 10600 9800 50  0001 C CNN "RefOrder"
 	1    10600 9800
 	0    -1   1    0
@@
 F 2 "Resistor_THT:R_Array_SIP10" V 11175 7850 50  0001 C CNN
 F 3 "http://www.vishay.com/docs/31509/csc.pdf" H 10600 7850 50  0001 C CNN
+F 4 "652-4610X-1LF-3.3K" H 10600 7850 50  0001 C CNN "RefOrder"
 	1    10600 7850
 	0    -1   1    0
