File: zorro.sch (KiCad schematic (older format))
At the start: 0 parts

Commit message: Use correct source rev6. mostly all schematics done for first pass...
Parts:
- added C416, C417, C418, C419: 220uF 16V, symbol Device:CP_Small
- added C606: 0.1uF, symbol Device:C
- added C617, C619, C620, C621, C622, C623, C624, C625, C626, C627, C628, C629, C630, C631, C632, C633, C635, C637, C639, C641, C645, C647, C649, C650, C651, C652, C654, C655, C657, C658, C659, C660, C661, C662, C663, C664, C665, C666, C667, C668, C669, C670, C671, C672, C673, C674, C678: 1000pF, symbol Device:C_Small
- added C902, C917: XXpF, symbol Device:C
- added CN601, CN602, CN603, CN604, CN605: zorro_socket, symbol amiga_customs:zorro_socket
- added CN606: Conn_01x04_Male, symbol Connector:Conn_01x04_Male
- added J1, J2: Conn_01x03_Male, symbol Connector:Conn_01x03_Male
- added R311, R312, R601, R603, R604, R605: 1k, symbol Device:R
- added R901: Xk, symbol Device:R
- added RP601, RP602, RP603, RP605: 1k, Resistor_THT:R_Array_SIP10, symbol Device:R_Network09
- added RP604: 470, Resistor_THT:R_Array_SIP10, symbol Device:R_Network09
- added RP607: 1k, Resistor_THT:R_Array_SIP6, symbol Device:R_Network05
- added U606: 74LS32, symbol 74xx:74LS32
Connections:
- new net: CN604.11 (/CFGOUTn), RP607.2 (R1), U606.2
- new net: CN604.12 (/CFGINn), U606.1, U606.11
- new net: CN601.97 (/FCS), CN602.97 (/FCS), CN603.97 (/FCS), CN604.97 (/FCS), CN605.97 (/FCS), J2.1 (Pin_1), J2.2 (Pin_2), J2.3 (Pin_3)
- new net: CN601.98 (/DS1), CN602.98 (/DS1), CN603.98 (/DS1), CN604.98 (/DS1), CN605.98 (/DS1), J1.1 (Pin_1), J1.2 (Pin_2), J1.3 (Pin_3)
- new net: CN603.11 (/CFGOUTn), RP607.6 (R5), U606.5
- new net: CN603.12 (/CFGINn), U606.3, U606.4
- new net: CN602.11 (/CFGOUTn), RP607.5 (R4), U606.10
- new net: CN602.12 (/CFGINn), U606.6, U606.9
- new net: CN601.12 (/CFGINn), U606.8
- new net: CN605.11 (/CFGOUTn), RP607.3 (R2), U606.13
- new net: C617.1, RP601.10 (R9)
- new net: C619.1, RP601.9 (R8)
- new net: C620.1, RP601.8 (R7)
- new net: C621.1, RP601.7 (R6)
- new net: C622.1, RP601.6 (R5)
- new net: C623.1, RP601.5 (R4)
- new net: C624.1, RP601.4 (R3)
- new net: C625.1, RP601.3 (R2)
- new net: C626.1, RP601.2 (R1)
- new net: C627.1, RP602.10 (R9)
- new net: C628.1, RP602.9 (R8)
- new net: C629.1, RP602.8 (R7)
- new net: C630.1, RP602.7 (R6)
- new net: C631.1, RP602.6 (R5)
- new net: C632.1, RP602.5 (R4)
- new net: C633.1, RP602.4 (R3)
- new net: C635.1, RP602.3 (R2)
- new net: C637.1, RP602.2 (R1)
- new net: C639.1, RP603.10 (R9)
- new net: C641.1, RP603.9 (R8)
- new net: C645.1, RP603.8 (R7)
- new net: C647.1, RP603.7 (R6)
- new net: C649.1, RP603.6 (R5)
- new net: C650.1, RP603.5 (R4)
- new net: C651.1, RP603.4 (R3)
- new net: C652.1, RP603.3 (R2)
- new net: C654.1, RP603.2 (R1)
- new net: C655.1, RP604.10 (R9)
- new net: C657.1, RP604.9 (R8)
- new net: C659.1, RP604.7 (R6)
- new net: C661.1, RP604.5 (R4)
- new net: C662.1, RP604.4 (R3)
- new net: C660.1, RP604.6 (R5)
- new net: C658.1, RP604.8 (R7)
- new net: C663.1, RP604.3 (R2)
- new net: C664.1, RP604.2 (R1)
- new net: C665.1, R604.2
- new net: C666.1, R605.2
- new net: C667.1, RP605.10 (R9)
- new net: C668.1, RP605.9 (R8)
- new net: C669.1, RP605.8 (R7)
- new net: C670.1, RP605.7 (R6)
- new net: C671.1, RP605.6 (R5)
- new net: C672.1, RP605.5 (R4)
- new net: C673.1, RP605.4 (R3)
- new net: C674.1, RP605.3 (R2)
- new net: C678.1, RP605.2 (R1)
- new net +12V: CN601.10 (+12V), CN602.10 (+12V), CN603.10 (+12V), CN604.10 (+12V), CN605.10 (+12V)
- new net +5V: C416.1, C417.1, C418.1, C419.1, C606.1, CN601.5 (+5V), CN601.6 (+5V), CN602.5 (+5V), CN602.6 (+5V), CN603.5 (+5V), CN603.6 (+5V), CN604.5 (+5V), CN604.6 (+5V), CN605.5 (+5V), CN605.6 (+5V), R311.1, R312.1, R601.1, R603.1, U606.14 (VCC)
- new net -12V: CN601.20 (-12V), CN602.20 (-12V), CN603.20 (-12V), CN604.20 (-12V), CN605.20 (-12V)
- new net -5V: CN601.8 (-5V), CN602.8 (-5V), CN603.8 (-5V), CN604.8 (-5V), CN605.8 (-5V)
- new net BA1: C624.2, CN601.29 (A1), CN602.29 (A1), CN603.29 (A1), CN604.29 (A1), CN605.29 (A1)
- new net BA10: C629.2, CN601.34 (A10), CN602.34 (A10), CN603.34 (A10), CN604.34 (A10), CN605.34 (A10)
- new net BA11: C631.2, CN601.36 (A11), CN602.36 (A11), CN603.36 (A11), CN604.36 (A11), CN605.36 (A11)
- new net BA12: C632.2, CN601.38 (A12), CN602.38 (A12), CN603.38 (A12), CN604.38 (A12), CN605.38 (A12)
- new net BA13: C633.2, CN601.39 (A13), CN602.39 (A13), CN603.39 (A13), CN604.39 (A13), CN605.39 (A13)
- new net BA14: C635.2, CN601.41 (A14), CN602.41 (A14), CN603.41 (A14), CN604.41 (A14), CN605.41 (A14)
- new net BA15: C637.2, CN601.43 (A15), CN602.43 (A15), CN603.43 (A15), CN604.43 (A15), CN605.43 (A15)
- new net BA16: C639.2, CN601.45 (A16), CN602.45 (A16), CN603.45 (A16), CN604.45 (A16), CN605.45 (A16)
- new net BA17: C641.2, CN601.47 (A17), CN602.47 (A17), CN603.47 (A17), CN604.47 (A17), CN605.47 (A17)
- new net BA18: C645.2, CN601.52 (A18), CN602.52 (A18), CN603.52 (A18), CN604.52 (A18), CN605.52 (A18)
- new net BA19: C647.2, CN601.54 (A19), CN602.54 (A19), CN603.54 (A19), CN604.54 (A19), CN605.54 (A19)
- new net BA2: C622.2, CN601.27 (A2), CN602.27 (A2), CN603.27 (A2), CN604.27 (A2), CN605.27 (A2)
- new net BA20: C649.2, CN601.56 (A20), CN602.56 (A20), CN603.56 (A20), CN604.56 (A20), CN605.56 (A20)
- new net BA21: C651.2, CN601.58 (A21), CN602.58 (A21), CN603.58 (A21), CN604.58 (A21), CN605.58 (A21)
- new net BA22: C650.2, CN601.57 (A22), CN602.57 (A22), CN603.57 (A22), CN604.57 (A22), CN605.57 (A22)
- new net BA23: C652.2, CN601.59 (A23), CN602.59 (A23), CN603.59 (A23), CN604.59 (A23), CN605.59 (A23)
- new net BA3: C621.2, CN601.26 (A3), CN602.26 (A3), CN603.26 (A3), CN604.26 (A3), CN605.26 (A3)
- new net BA4: C620.2, CN601.24 (A4), CN602.24 (A4), CN603.24 (A4), CN604.24 (A4), CN605.24 (A4)
- new net BA5: C617.2, CN601.21 (A5), CN602.21 (A5), CN603.21 (A5), CN604.21 (A5), CN605.21 (A5)
- new net BA6: C619.2, CN601.23 (A6), CN602.23 (A6), CN603.23 (A6), CN604.23 (A6), CN605.23 (A6)
- new net BA7: C623.2, CN601.28 (A7), CN602.28 (A7), CN603.28 (A7), CN604.28 (A7), CN605.28 (A7)
- new net BA8: C625.2, CN601.30 (A8), CN602.30 (A8), CN603.30 (A8), CN604.30 (A8), CN605.30 (A8)
- new net BA9: C627.2, CN601.32 (A9), CN602.32 (A9), CN603.32 (A9), CN604.32 (A9), CN605.32 (A9)
- new net BD0: C664.2, CN601.75 (D0), CN602.75 (D0), CN603.75 (D0), CN604.75 (D0), CN605.75 (D0)
- new net BD1: C666.2, CN601.77 (D1), CN602.77 (D1), CN603.77 (D1), CN604.77 (D1), CN605.77 (D1)
- new net BD10: C665.2, CN601.76 (D10), CN602.76 (D10), CN603.76 (D10), CN604.76 (D10), CN605.76 (D10)
- new net BD11: C661.2, CN601.71 (D11), CN602.71 (D11), CN603.71 (D11), CN604.71 (D11), CN605.71 (D11)
- new net BD12: C659.2, CN601.69 (D12), CN602.69 (D12), CN603.69 (D12), CN604.69 (D12), CN605.69 (D12)
- new net BD13: C657.2, CN601.67 (D13), CN602.67 (D13), CN603.67 (D13), CN604.67 (D13), CN605.67 (D13)
- new net BD14: C655.2, CN601.65 (D14), CN602.65 (D14), CN603.65 (D14), CN604.65 (D14), CN605.65 (D14)
- new net BD15: C654.2, CN601.63 (D15), CN602.63 (D15), CN603.63 (D15), CN604.63 (D15), CN605.63 (D15)
- new net BD2: C668.2, CN601.79 (D2), CN602.79 (D2), CN603.79 (D2), CN604.79 (D2), CN605.79 (D2)
- new net BD3: C670.2, CN601.81 (D3), CN602.81 (D3), CN603.81 (D3), CN604.81 (D3), CN605.81 (D3)
- new net BD4: C672.2, CN601.83 (D4), CN602.83 (D4), CN603.83 (D4), CN604.83 (D4), CN605.83 (D4)
- new net BD5: C674.2, CN601.86 (D5), CN602.86 (D5), CN603.86 (D5), CN604.86 (D5), CN605.86 (D5)
- new net BD6: C673.2, CN601.84 (D6), CN602.84 (D6), CN603.84 (D6), CN604.84 (D6), CN605.84 (D6)
- new net BD7: C671.2, CN601.82 (D7), CN602.82 (D7), CN603.82 (D7), CN604.82 (D7), CN605.82 (D7)
- new net BD8: C669.2, CN601.80 (D8), CN602.80 (D8), CN603.80 (D8), CN604.80 (D8), CN605.80 (D8)
- new net BD9: C667.2, CN601.78 (D9), CN602.78 (D9), CN603.78 (D9), CN604.78 (D9), CN605.78 (D9)
- new net BFC0: C626.2, CN601.31 (FC0), CN602.31 (FC0), CN603.31 (FC0), CN604.31 (FC0), CN605.31 (FC0)
- new net BFC1: C628.2, CN601.33 (FC1), CN602.33 (FC1), CN603.33 (FC1), CN604.33 (FC1), CN605.33 (FC1)
- new net BFC2: C630.2, CN601.35 (FC2), CN602.35 (FC2), CN603.35 (FC2), CN604.35 (FC2), CN605.35 (FC2)
- new net DOE: CN601.93 (DOE), CN602.93 (DOE), CN603.93 (DOE), CN604.93 (DOE), CN605.93 (DOE), R601.2
- new net E: CN601.50 (ECLK), CN602.50 (ECLK), CN603.50 (ECLK), CN604.50 (ECLK), CN605.50 (ECLK)
- new net E7M: CN601.92 (E7M), CN602.92 (E7M), CN603.92 (E7M), CN604.92 (E7M), CN605.92 (E7M)
- new net ECDAC: CN601.15 (CDAC), CN602.15 (CDAC), CN603.15 (CDAC), CN604.15 (CDAC), CN605.15 (CDAC)
- new net GND: C416.2, C417.2, C418.2, C419.2, C606.2, C902.2, C917.2, CN601.1 (GND), CN601.100 (GND), CN601.13 (GND), CN601.2 (GND), CN601.25 (GND), CN601.3 (GND), CN601.37 (GND), CN601.4 (GND), CN601.49 (GND), CN601.61 (GND), CN601.73 (GND), CN601.85 (GND), CN601.87 (GND), CN601.88 (GND), CN601.89 (GND), CN601.90 (GND), CN601.91 (SenseZ3), CN601.99 (GND), CN602.1 (GND), CN602.100 (GND), CN602.13 (GND), CN602.2 (GND), CN602.25 (GND), CN602.3 (GND), CN602.37 (GND), CN602.4 (GND), CN602.49 (GND), CN602.61 (GND), CN602.73 (GND), CN602.85 (GND), CN602.87 (GND), CN602.88 (GND), CN602.89 (GND), CN602.90 (GND), CN602.91 (SenseZ3), CN602.99 (GND), CN603.1 (GND), CN603.100 (GND), CN603.13 (GND), CN603.2 (GND), CN603.25 (GND), CN603.3 (GND), CN603.37 (GND), CN603.4 (GND), CN603.49 (GND), CN603.61 (GND), CN603.73 (GND), CN603.85 (GND), CN603.87 (GND), CN603.88 (GND), CN603.89 (GND), CN603.90 (GND), CN603.91 (SenseZ3), CN603.99 (GND), CN604.1 (GND), CN604.100 (GND), CN604.13 (GND), CN604.2 (GND), CN604.25 (GND), CN604.3 (GND), CN604.37 (GND), CN604.4 (GND), CN604.49 (GND), CN604.61 (GND), CN604.73 (GND), CN604.85 (GND), CN604.87 (GND), CN604.88 (GND), CN604.89 (GND), CN604.90 (GND), CN604.91 (SenseZ3), CN604.99 (GND), CN605.1 (GND), CN605.100 (GND), CN605.13 (GND), CN605.2 (GND), CN605.25 (GND), CN605.3 (GND), CN605.37 (GND), CN605.4 (GND), CN605.49 (GND), CN605.61 (GND), CN605.73 (GND), CN605.85 (GND), CN605.87 (GND), CN605.88 (GND), CN605.89 (GND), CN605.90 (GND), CN605.91 (SenseZ3), CN605.99 (GND), CN606.4 (Pin_4), R604.1, R605.1, R901.2, RP601.1 (common), RP602.1 (common), RP603.1 (common), RP604.1 (common), RP605.1 (common), RP607.1 (common), U606.7 (GND)
- new net OVR: CN601.17 (/CINH_/OVR), CN602.17 (/CINH_/OVR), CN603.17 (/CINH_/OVR), CN604.17 (/CINH_/OVR), CN605.17 (/CINH_/OVR)
- new net READ: C658.2, CN601.68 (READ), CN602.68 (READ), CN603.68 (READ), CN604.68 (READ), CN605.68 (READ)
- new net XRDY: CN601.18 (/MTCR_XRDY), CN602.18 (/MTCR_XRDY), CN603.18 (/MTCR_XRDY), CN604.18 (/MTCR_XRDY), CN605.18 (/MTCR_XRDY)
- new net _BAS: C663.2, CN601.74 (/CCS_/AS), CN602.74 (/CCS_/AS), CN603.74 (/CCS_/AS), CN604.74 (/CCS_/AS), CN605.74 (/CCS_/AS)
- new net _BEER: CN601.46 (/BERR), CN602.46 (/BERR), CN603.46 (/BERR), CN604.46 (/BERR), CN605.46 (/BERR)
- new net _BG1: CN605.64 (/BGn)
- new net _BG2: CN604.64 (/BGn)
- new net _BG3: CN603.64 (/BGn)
- new net _BG4: CN602.64 (/BGn)
- new net _BG5: CN601.64 (/BGn)
- new net _BGACK: CN601.62 (/BGACK), CN602.62 (/BGACK), CN603.62 (/BGACK), CN604.62 (/BGACK), CN605.62 (/BGACK)
- new net _BLDS: C660.2, CN601.70 (/LDS), CN602.70 (/LDS), CN603.70 (/LDS), CN604.70 (/LDS), CN605.70 (/LDS)
- new net _BR1: CN605.60 (/BRn)
- new net _BR2: CN604.60 (/BRn)
- new net _BR3: CN603.60 (/BRn)
- new net _BR4: CN602.60 (/BRn)
- new net _BR5: CN601.60 (/BRn)
- new net _BUDS: C662.2, CN601.72 (/UDS), CN602.72 (/UDS), CN603.72 (/UDS), CN604.72 (/UDS), CN605.72 (/UDS)
- new net _BUSRST: CN601.94 (/IORST), CN602.94 (/IORST), CN603.94 (/IORST), CN604.94 (/IORST), CN605.94 (/IORST), R603.2
- new net _COPCFG: CN605.12 (/CFGINn), RP607.4 (R3), U606.12
- new net _DTACK: CN601.66 (/DTACK), CN602.66 (/DTACK), CN603.66 (/DTACK), CN604.66 (/DTACK), CN605.66 (/DTACK)
- new net _EC1: C917.1, CN601.16 (/C1), CN602.16 (/C1), CN603.16 (/C1), CN604.16 (/C1), CN605.16 (/C1), R901.1
- new net _EC3: C902.1, CN601.14 (/C3), CN602.14 (/C3), CN603.14 (/C3), CN604.14 (/C3), CN605.14 (/C3)
- new net _EINT1: CN601.96 (/EINT1), CN602.96 (/EINT1), CN603.96 (/EINT1), CN604.96 (/EINT1), CN605.96 (/EINT1)
- new net _EINT4: CN601.44 (/EINT4), CN602.44 (/EINT4), CN603.44 (/EINT4), CN604.44 (/EINT4), CN605.44 (/EINT4)
- new net _EINT5: CN601.42 (/EINT5), CN602.42 (/EINT5), CN603.42 (/EINT5), CN604.42 (/EINT5), CN605.42 (/EINT5)
- new net _EINT7: CN601.40 (/EINT7), CN602.40 (/EINT7), CN603.40 (/EINT7), CN604.40 (/EINT7), CN605.40 (/EINT7)
- new net _GBG: C678.2, CN601.95 (/BCLR), CN602.95 (/BCLR), CN603.95 (/BCLR), CN604.95 (/BCLR), CN605.95 (/BCLR)
- new net _HLT: CN601.55 (/HLT), CN602.55 (/HLT), CN603.55 (/HLT), CN604.55 (/HLT), CN605.55 (/HLT)
- new net _INT2: CN601.19 (/INT2), CN602.19 (/INT2), CN603.19 (/INT2), CN604.19 (/INT2), CN605.19 (/INT2), R312.2
- new net _INT6: CN601.22 (/INT6), CN602.22 (/INT6), CN603.22 (/INT6), CN604.22 (/INT6), CN605.22 (/INT6), R311.2
- new net _IPL0: CN606.3 (Pin_3)
- new net _IPL1: CN606.2 (Pin_2)
- new net _IPL2: CN606.1 (Pin_1)
- new net _OWN: CN601.7 (/OWN), CN602.7 (/OWN), CN603.7 (/OWN), CN604.7 (/OWN), CN605.7 (/OWN)
- new net _RST: CN601.53 (/RST), CN602.53 (/RST), CN603.53 (/RST), CN604.53 (/RST), CN605.53 (/RST)
- new net _SLAVE1: CN605.9 (/SLAVEn)
- new net _SLAVE2: CN604.9 (/SLAVEn)
- new net _SLAVE3: CN603.9 (/SLAVEn)
- new net _SLAVE4: CN602.9 (/SLAVEn)
- new net _SLAVE5: CN601.9 (/SLAVEn)
- new net _VMA: CN601.51 (/DS0), CN602.51 (/DS0), CN603.51 (/DS0), CN604.51 (/DS0), CN605.51 (/DS0)
- new net _VPA: CN601.48 (/MTACK), CN602.48 (/MTACK), CN603.48 (/MTACK), CN604.48 (/MTACK), CN605.48 (/MTACK)
