File: zorro.sch (KiCad schematic (older format))
At the start: 77 parts, among them CN601 zorro_socket, CN602 zorro_socket, CN603 zorro_socket, CN604 zorro_socket, CN605 zorro_socket, CN606 Conn_01x04_Male, J1 Conn_01x03_Male, J2 Conn_01x03_Male, U606 74LS32

Commit message: Update footprints
Parts:
- C606, C617, C619, C620, C621, C622, C623, C624, C625, C626, C627, C628, C629, C630, C631, C632, C633, C635, C637, C639, C641, C645, C647, C649, C650, C651, C652, C654, C655, C657, C658, C659, C660, C661, C662, C663, C664, C665, C666, C667, C668, C669, C670, C671, C672, C673, C674, C678, C902, C917: footprint (none) -> Capacitor_THT:C_Rect_L11.0mm_W2.8mm_P10.00mm_MKT
- CN601, CN602, CN603, CN604, CN605: footprint (none) -> d_amiga:Zorro

Commit message: More placement
Parts:
- CN606: footprint Connector_PinSocket_2.54mm:PinSocket_1x04_P2.54mm_Vertical -> Connector_PinHeader_2.54mm:PinHeader_1x04_P2.54mm_Vertical
- J1, J2: footprint Connector_PinSocket_2.54mm:PinSocket_1x03_P2.54mm_Vertical -> Connector_PinHeader_2.54mm:PinHeader_1x03_P2.54mm_Vertical
Changed lines of the file:
@@
 F 0 "J1" V 16800 13250 50  0000 R CNN
 F 1 "Conn_01x03_Male" V 16963 13012 50  0001 R CNN
-F 2 "Connector_PinSocket_2.54mm:PinSocket_1x03_P2.54mm_Vertical" H 16900 13200 50  0001 C CNN
+F 2 "Connector_PinHeader_2.54mm:PinHeader_1x03_P2.54mm_Vertical" H 16900 13200 50  0001 C CNN
 F 3 "~" H 16900 13200 50  0001 C CNN
 	1    16900 13200
@@
 F 0 "J2" V 17150 13150 50  0000 R CNN
 F 1 "Conn_01x03_Male" V 17313 12912 50  0001 R CNN
-F 2 "Connector_PinSocket_2.54mm:PinSocket_1x03_P2.54mm_Vertical" H 17250 13100 50  0001 C CNN
+F 2 "Connector_PinHeader_2.54mm:PinHeader_1x03_P2.54mm_Vertical" H 17250 13100 50  0001 C CNN
 F 3 "~" H 17250 13100 50  0001 C CNN
 	1    17250 13100
@@
 F 0 "CN606" H 3922 6978 50  0000 R CNN
 F 1 "Conn_01x04_Male" H 4058 7240 50  0001 C CNN
-F 2 "Connector_PinSocket_2.54mm:PinSocket_1x04_P2.54mm_Vertical" H 3950 7050 50  0001 C CNN
+F 2 "Connector_PinHeader_2.54mm:PinHeader_1x04_P2.54mm_Vertical" H 3950 7050 50  0001 C CNN
 F 3 "~" H 3950 7050 50  0001 C CNN
 	1    3950 7050

Commit message: Make caps footprint smaller
Parts:
- C606, C617, C619, C620, C621, C622, C623, C624, C625, C626, C627, C628, C629, C630, C631, C632, C633, C635, C637, C639, C641, C645, C647, C649, C650, C651, C652, C654, C655, C657, C658, C659, C660, C661, C662, C663, C664, C665, C666, C667, C668, C669, C670, C671, C672, C673, C674, C678, C902, C917: footprint Capacitor_THT:C_Rect_L11.0mm_W2.8mm_P10.00mm_MKT -> Capacitor_THT:C_Rect_L11.5mm_W2.0mm_P10.00mm_MKT

Commit message: Add DoNotPopulate field for components which shouldn't be fitted
Parts:
- C902, C917, J1, J2, R901: DoNotPopulate (none) -> yes
Changed lines of the file:
@@
 F 2 "Connector_PinHeader_2.54mm:PinHeader_1x03_P2.54mm_Vertical" H 16900 13200 50  0001 C CNN
 F 3 "~" H 16900 13200 50  0001 C CNN
+F 4 "yes" H 16900 13200 50  0001 C CNN "DoNotPopulate"
 	1    16900 13200
 	0    -1   -1   0
@@
 F 2 "Connector_PinHeader_2.54mm:PinHeader_1x03_P2.54mm_Vertical" H 17250 13100 50  0001 C CNN
 F 3 "~" H 17250 13100 50  0001 C CNN
+F 4 "yes" H 17250 13100 50  0001 C CNN "DoNotPopulate"
 	1    17250 13100
 	0    -1   -1   0
@@
 F 2 "Resistor_THT:R_Axial_DIN0207_L6.3mm_D2.5mm_P10.16mm_Horizontal" V 21680 5250 50  0001 C CNN
 F 3 "~" H 21750 5250 50  0001 C CNN
+F 4 "yes" H 21750 5250 50  0001 C CNN "DoNotPopulate"
 	1    21750 5250
 	1    0    0    -1
@@
 F 2 "Capacitor_THT:C_Rect_L11.5mm_W2.0mm_P10.00mm_MKT" H 22188 5100 50  0001 C CNN
 F 3 "~" H 22150 5250 50  0001 C CNN
+F 4 "yes" H 22150 5250 50  0001 C CNN "DoNotPopulate"
 	1    22150 5250
 	1    0    0    -1
@@
 F 2 "Capacitor_THT:C_Rect_L11.5mm_W2.0mm_P10.00mm_MKT" H 22588 5100 50  0001 C CNN
 F 3 "~" H 22550 5250 50  0001 C CNN
+F 4 "yes" H 22550 5250 50  0001 C CNN "DoNotPopulate"
 	1    22550 5250
 	1    0    0    -1

Commit message: Switch footprints for suitable modern replacements
Parts:
- C416, C417, C418, C419: footprint Capacitor_THT:C_Axial_L12.0mm_D7.5mm_P20.00mm_Horizontal -> Capacitor_THT:C_Axial_L12.0mm_D8.5mm_P15.00mm_Horizontal
- C606, C617, C619, C620, C621, C622, C623, C624, C625, C626, C627, C628, C629, C630, C631, C632, C633, C635, C637, C639, C641, C645, C647, C649, C650, C651, C652, C654, C655, C657, C658, C659, C660, C661, C662, C663, C664, C665, C666, C667, C668, C669, C670, C671, C672, C673, C674, C678: footprint Capacitor_THT:C_Rect_L11.5mm_W2.0mm_P10.00mm_MKT -> Capacitor_THT:C_Rect_L11.5mm_W2.6mm_P10.00mm_MKT

Commit message: Some footprints updates; Add all Mouser references
Parts:
- C416, C417, C418, C419: RefOrder (none) -> 667-ECA-1CM221B
- C606: RefOrder (none) -> 581-SA105C104KARC
- C617, C619, C620, C621, C622, C623, C624, C625, C626, C627, C628, C629, C630, C631, C632, C633, C635, C637, C639, C641, C645, C647, C649, C650, C651, C652, C654, C655, C657, C658, C659, C660, C661, C662, C663, C664, C665, C666, C667, C668, C669, C670, C671, C672, C673, C674, C678: RefOrder (none) -> 581-SA105C102KAR
- R311, R312, R601, R603, R604, R605: RefOrder (none) -> 603-CFR-25JR-521K
- RP600: RefOrder (none) -> 652-4608X-101-103FLF
- RP601, RP602, RP603, RP605: RefOrder (none) -> 652-4610X-1LF-1K
- RP604: RefOrder (none) -> 652-4610X-1LF-470
- RP607: RefOrder (none) -> 652-4606M-1LF-1K
- U606: RefOrder (none) -> 595-SN74LS32N

Commit message: Got the components, reduce some footprints
Parts:
- C416, C417, C418, C419: footprint Capacitor_THT:C_Axial_L12.0mm_D8.5mm_P15.00mm_Horizontal -> Capacitor_THT:C_Axial_L19.0mm_D8.0mm_P25.00mm_Horizontal; RefOrder 667-ECA-1CM221B -> 75-516D227M025MM6AE3
Changed lines of the file:
@@
 F 0 "C416" V 7925 3150 50  0000 C CNN
 F 1 "220uF 16V" V 7834 3150 50  0000 C CNN
-F 2 "Capacitor_THT:C_Axial_L12.0mm_D8.5mm_P15.00mm_Horizontal" H 7700 3150 50  0001 C CNN
+F 2 "Capacitor_THT:C_Axial_L19.0mm_D8.0mm_P25.00mm_Horizontal" H 7700 3150 50  0001 C CNN
 F 3 "~" H 7700 3150 50  0001 C CNN
-F 4 "667-ECA-1CM221B" H 7700 3150 50  0001 C CNN "RefOrder"
+F 4 "75-516D227M025MM6AE3" H 7700 3150 50  0001 C CNN "RefOrder"
 	1    7700 3150
 	0    -1   -1   0
@@
 F 0 "C417" V 10025 3150 50  0000 C CNN
 F 1 "220uF 16V" V 9934 3150 50  0000 C CNN
-F 2 "Capacitor_THT:C_Axial_L12.0mm_D8.5mm_P15.00mm_Horizontal" H 9800 3150 50  0001 C CNN
+F 2 "Capacitor_THT:C_Axial_L19.0mm_D8.0mm_P25.00mm_Horizontal" H 9800 3150 50  0001 C CNN
 F 3 "~" H 9800 3150 50  0001 C CNN
-F 4 "667-ECA-1CM221B" H 9800 3150 50  0001 C CNN "RefOrder"
+F 4 "75-516D227M025MM6AE3" H 9800 3150 50  0001 C CNN "RefOrder"
 	1    9800 3150
 	0    -1   -1   0
@@
 F 0 "C418" V 12125 3150 50  0000 C CNN
 F 1 "220uF 16V" V 12034 3150 50  0000 C CNN
-F 2 "Capacitor_THT:C_Axial_L12.0mm_D8.5mm_P15.00mm_Horizontal" H 11900 3150 50  0001 C CNN
+F 2 "Capacitor_THT:C_Axial_L19.0mm_D8.0mm_P25.00mm_Horizontal" H 11900 3150 50  0001 C CNN
 F 3 "~" H 11900 3150 50  0001 C CNN
-F 4 "667-ECA-1CM221B" H 11900 3150 50  0001 C CNN "RefOrder"
+F 4 "75-516D227M025MM6AE3" H 11900 3150 50  0001 C CNN "RefOrder"
 	1    11900 3150
 	0    -1   -1   0
@@
 F 0 "C419" V 14275 3150 50  0000 C CNN
 F 1 "220uF 16V" V 14184 3150 50  0000 C CNN
-F 2 "Capacitor_THT:C_Axial_L12.0mm_D8.5mm_P15.00mm_Horizontal" H 14050 3150 50  0001 C CNN
+F 2 "Capacitor_THT:C_Axial_L19.0mm_D8.0mm_P25.00mm_Horizontal" H 14050 3150 50  0001 C CNN
 F 3 "~" H 14050 3150 50  0001 C CNN
-F 4 "667-ECA-1CM221B" H 14050 3150 50  0001 C CNN "RefOrder"
+F 4 "75-516D227M025MM6AE3" H 14050 3150 50  0001 C CNN "RefOrder"
 	1    14050 3150
 	0    -1   -1   0

Commit message: Some footprint changes; Tidy pcb
Parts:
- C617, C619, C620, C621, C622, C623, C624, C625, C626, C627, C628, C629, C630, C631, C632, C633, C635, C637, C639, C641, C645, C647, C649, C650, C651, C652, C654, C655, C657, C658, C659, C660, C661, C662, C663, C664, C665, C666, C667, C668, C669, C670, C671, C672, C673, C674, C678: footprint Capacitor_THT:C_Rect_L11.5mm_W2.6mm_P10.00mm_MKT -> Capacitor_THT:C_Rect_L11.5mm_W2.0mm_P10.00mm_MKT
