File: expansion logic.sch (KiCad schematic (older format))
At the start: 30 parts, among them U302 74LS32, U800 BUSTER5721, U801 MSM6242, U802 74LS138, U803 74LS08, U804 74LS148, Y800 32768Hz

Commit message: REV 6.2 fixes applied
Parts:
- added R2: 1k, symbol Device:R
Connections:
- net +5V: now also R2.1
- net _BAS: now also R2.2
Other:
- note added: "REV 6.2 fix\np36 to +5 via 1k"
Changed lines of the file:
@@
 Text GLabel 2000 4100 0    50   Input ~ 0
 _BRST
-Text GLabel 2000 4000 0    50   Input ~ 0
+Text GLabel 850  4000 0    50   Input ~ 0
 _BAS
 $Comp
@@
 	0    1    1    0
 $EndComp
+Wire Wire Line
+	850  4000 1050 4000
 Wire Bus Line
 	7050 3250 7050 3500
@@
 Wire Bus Line
 	3350 7550 3350 7900
+$Comp
+L Device:R R2
+U 1 1 5D3BFFB3
+P 1050 3850
+F 0 "R2" H 1120 3896 50  0000 L CNN
+F 1 "1k" H 1120 3805 50  0000 L CNN
+F 2 "" V 980 3850 50  0001 C CNN
+F 3 "~" H 1050 3850 50  0001 C CNN
+	1    1050 3850
+	1    0    0    -1
+$EndComp
+Connection ~ 1050 4000
+Wire Wire Line
+	1050 4000 2000 4000
+$Comp
+L power:+5V #PWR0265
+U 1 1 5D3C02DA
+P 1050 3700
+F 0 "#PWR0265" H 1050 3550 50  0001 C CNN
+F 1 "+5V" H 1065 3873 50  0000 C CNN
+F 2 "" H 1050 3700 50  0001 C CNN
+F 3 "" H 1050 3700 50  0001 C CNN
+	1    1050 3700
+	1    0    0    -1
+$EndComp
+Text Notes 650  3450 0    50   ~ 0
+REV 6.2 fix\np36 to +5 via 1k
 $EndSCHEMATC

Commit message: more done
Parts:
- C920: Notes (none) -> To check on PCB
Changed lines of the file:
@@
 F 2 "" H 3838 4750 50  0001 C CNN
 F 3 "~" H 3800 4900 50  0001 C CNN
+F 4 "To check on PCB" H 3800 4750 50  0000 C CNN "Notes"
 	1    3800 4900
 	1    0    0    -1

Commit message: Associate footprints with components
Parts:
- BT800: footprint (none) -> Connector_PinSocket_2.54mm:PinSocket_2x01_P2.54mm_Vertical
- R2, R800, R801, R803, R804, R806, R807, R904, R905: footprint (none) -> Resistor_THT:R_Axial_DIN0207_L6.3mm_D2.5mm_P10.16mm_Horizontal
- U302, U803: footprint (none) -> Package_DIP:DIP-14_W7.62mm_Socket
- U800: footprint (none) -> Package_DIP:DIP-48_W15.24mm_Socket
- U801: footprint (none) -> Package_DIP:DIP-18_W7.62mm_Socket
- U802, U804: footprint (none) -> Package_DIP:DIP-16_W7.62mm_Socket
- VC800: footprint (none) -> Capacitor_THT:C_Rect_L7.0mm_W6.5mm_P5.00mm
- Y800: footprint (none) -> Crystal:Crystal_DS10_D1.0mm_L4.3mm_Horizontal
Changed lines of the file:
@@
 F 0 "U800" H 2500 1425 50  0000 C CNN
 F 1 "BUSTER5721" H 2500 1334 50  0000 C CNN
-F 2 "" H 2500 1300 50  0001 C CNN
+F 2 "Package_DIP:DIP-48_W15.24mm_Socket" H 2500 1300 50  0001 C CNN
 F 3 "http://obligement.free.fr/articles/chipsetamiga.php#buster" H 2500 1300 50  0001 C CNN
 	1    2500 1300
@@
 F 0 "R904" V 3043 2200 50  0000 C CNN
 F 1 "47" V 3134 2200 50  0000 C CNN
-F 2 "" V 3180 2200 50  0001 C CNN
+F 2 "Resistor_THT:R_Axial_DIN0207_L6.3mm_D2.5mm_P10.16mm_Horizontal" V 3180 2200 50  0001 C CNN
 F 3 "~" H 3250 2200 50  0001 C CNN
 	1    3250 2200
@@
 F 0 "R806" H 3430 3304 50  0000 R CNN
 F 1 "4.7k" H 3430 3395 50  0000 R CNN
-F 2 "" V 3430 3350 50  0001 C CNN
+F 2 "Resistor_THT:R_Axial_DIN0207_L6.3mm_D2.5mm_P10.16mm_Horizontal" V 3430 3350 50  0001 C CNN
 F 3 "~" H 3500 3350 50  0001 C CNN
 	1    3500 3350
@@
 F 0 "R807" H 3780 3304 50  0000 R CNN
 F 1 "4.7k" H 3780 3395 50  0000 R CNN
-F 2 "" V 3780 3350 50  0001 C CNN
+F 2 "Resistor_THT:R_Axial_DIN0207_L6.3mm_D2.5mm_P10.16mm_Horizontal" V 3780 3350 50  0001 C CNN
 F 3 "~" H 3850 3350 50  0001 C CNN
 	1    3850 3350
@@
 F 0 "R905" V 3507 4550 50  0000 C CNN
 F 1 "47" V 3416 4550 50  0000 C CNN
-F 2 "" V 3230 4550 50  0001 C CNN
+F 2 "Resistor_THT:R_Axial_DIN0207_L6.3mm_D2.5mm_P10.16mm_Horizontal" V 3230 4550 50  0001 C CNN
 F 3 "~" H 3300 4550 50  0001 C CNN
 	1    3300 4550
@@
 F 0 "U302" H 1150 5325 50  0000 C CNN
 F 1 "74LS32" H 1150 5234 50  0000 C CNN
-F 2 "" H 1150 5000 50  0001 C CNN
+F 2 "Package_DIP:DIP-14_W7.62mm_Socket" H 1150 5000 50  0001 C CNN
 F 3 "http://www.ti.com/lit/gpn/sn74LS32" H 1150 5000 50  0001 C CNN
 	4    1150 5000
@@
 F 0 "R800" V 1907 4850 50  0000 C CNN
 F 1 "1k" V 1816 4850 50  0000 C CNN
-F 2 "" V 1630 4850 50  0001 C CNN
+F 2 "Resistor_THT:R_Axial_DIN0207_L6.3mm_D2.5mm_P10.16mm_Horizontal" V 1630 4850 50  0001 C CNN
 F 3 "~" H 1700 4850 50  0001 C CNN
 	1    1700 4850
@@
 F 0 "U801" H 4450 7225 50  0000 C CNN
 F 1 "MSM6242" H 4450 7134 50  0000 C CNN
-F 2 "" H 4450 7100 50  0001 C CNN
+F 2 "Package_DIP:DIP-18_W7.62mm_Socket" H 4450 7100 50  0001 C CNN
 F 3 "https://pdf1.alldatasheet.com/datasheet-pdf/view/11259/OKI/MSM6242B.html" H 4450 7100 50  0001 C CNN
 	1    4450 7100
@@
 F 0 "Y800" H 4450 9918 50  0000 C CNN
 F 1 "32768Hz" H 4450 9827 50  0000 C CNN
-F 2 "" H 4450 9650 50  0001 C CNN
+F 2 "Crystal:Crystal_DS10_D1.0mm_L4.3mm_Horizontal" H 4450 9650 50  0001 C CNN
 F 3 "~" H 4450 9650 50  0001 C CNN
 	1    4450 9650
@@
 F 0 "VC800" H 5065 9996 50  0000 L CNN
 F 1 "22-47pF" H 5065 9905 50  0000 L CNN
-F 2 "" H 4950 9950 50  0001 C CNN
+F 2 "Capacitor_THT:C_Rect_L7.0mm_W6.5mm_P5.00mm" H 4950 9950 50  0001 C CNN
 F 3 "~" H 4950 9950 50  0001 C CNN
 	1    4950 9950
@@
 F 0 "R804" H 5270 6846 50  0000 L CNN
 F 1 "10k" H 5270 6755 50  0000 L CNN
-F 2 "" V 5130 6800 50  0001 C CNN
+F 2 "Resistor_THT:R_Axial_DIN0207_L6.3mm_D2.5mm_P10.16mm_Horizontal" V 5130 6800 50  0001 C CNN
 F 3 "~" H 5200 6800 50  0001 C CNN
 	1    5200 6800
@@
 F 0 "R801" H 6370 6846 50  0000 L CNN
 F 1 "470" H 6370 6755 50  0000 L CNN
-F 2 "" V 6230 6800 50  0001 C CNN
+F 2 "Resistor_THT:R_Axial_DIN0207_L6.3mm_D2.5mm_P10.16mm_Horizontal" V 6230 6800 50  0001 C CNN
 F 3 "~" H 6300 6800 50  0001 C CNN
 	1    6300 6800
@@
 F 0 "R803" H 6370 7846 50  0000 L CNN
 F 1 "470" H 6370 7755 50  0000 L CNN
-F 2 "" V 6230 7800 50  0001 C CNN
+F 2 "Resistor_THT:R_Axial_DIN0207_L6.3mm_D2.5mm_P10.16mm_Horizontal" V 6230 7800 50  0001 C CNN
 F 3 "~" H 6300 7800 50  0001 C CNN
 	1    6300 7800
@@
 F 0 "BT800" H 6408 8446 50  0000 L CNN
 F 1 "3/60DK Ni-Cd 3.6V 60mAH" H 6408 8355 50  0000 L CNN
-F 2 "" V 6300 8460 50  0001 C CNN
+F 2 "Connector_PinSocket_2.54mm:PinSocket_2x01_P2.54mm_Vertical" V 6300 8460 50  0001 C CNN
 F 3 "~" V 6300 8460 50  0001 C CNN
 	1    6300 8400
@@
 F 0 "U802" H 8000 2419 50  0000 C CNN
 F 1 "74LS138" H 8000 2510 50  0000 C CNN
-F 2 "" H 8000 3300 50  0001 C CNN
+F 2 "Package_DIP:DIP-16_W7.62mm_Socket" H 8000 3300 50  0001 C CNN
 F 3 "http://www.ti.com/lit/gpn/sn74LS138" H 8000 3300 50  0001 C CNN
 	1    8000 3300
@@
 F 0 "U804" H 12800 4231 50  0000 C CNN
 F 1 "74LS148" H 12800 4140 50  0000 C CNN
-F 2 "" H 12800 3350 50  0001 C CNN
+F 2 "Package_DIP:DIP-16_W7.62mm_Socket" H 12800 3350 50  0001 C CNN
 F 3 "http://www.ti.com/lit/gpn/sn74LS148" H 12800 3350 50  0001 C CNN
 	1    12800 3350
@@
 F 0 "U803" H 10300 2775 50  0000 C CNN
 F 1 "74LS08" H 10300 2684 50  0000 C CNN
-F 2 "" H 10300 2450 50  0001 C CNN
+F 2 "Package_DIP:DIP-14_W7.62mm_Socket" H 10300 2450 50  0001 C CNN
 F 3 "http://www.ti.com/lit/gpn/sn74LS08" H 10300 2450 50  0001 C CNN
 	1    10300 2450
@@
 F 0 "U803" H 10300 3325 50  0000 C CNN
 F 1 "74LS08" H 10300 3234 50  0000 C CNN
-F 2 "" H 10300 3000 50  0001 C CNN
+F 2 "Package_DIP:DIP-14_W7.62mm_Socket" H 10300 3000 50  0001 C CNN
 F 3 "http://www.ti.com/lit/gpn/sn74LS08" H 10300 3000 50  0001 C CNN
 	2    10300 3000
@@
 F 0 "U803" H 10300 3875 50  0000 C CNN
 F 1 "74LS08" H 10300 3784 50  0000 C CNN
-F 2 "" H 10300 3550 50  0001 C CNN
+F 2 "Package_DIP:DIP-14_W7.62mm_Socket" H 10300 3550 50  0001 C CNN
 F 3 "http://www.ti.com/lit/gpn/sn74LS08" H 10300 3550 50  0001 C CNN
 	3    10300 3550
@@
 F 0 "U803" H 10300 4425 50  0000 C CNN
 F 1 "74LS08" H 10300 4334 50  0000 C CNN
-F 2 "" H 10300 4100 50  0001 C CNN
+F 2 "Package_DIP:DIP-14_W7.62mm_Socket" H 10300 4100 50  0001 C CNN
 F 3 "http://www.ti.com/lit/gpn/sn74LS08" H 10300 4100 50  0001 C CNN
 	4    10300 4100
@@
 F 0 "U803" H 10530 5646 50  0000 L CNN
 F 1 "74LS08" H 10530 5555 50  0000 L CNN
-F 2 "" H 10300 5600 50  0001 C CNN
+F 2 "Package_DIP:DIP-14_W7.62mm_Socket" H 10300 5600 50  0001 C CNN
 F 3 "http://www.ti.com/lit/gpn/sn74LS08" H 10300 5600 50  0001 C CNN
 	5    10300 5600
@@
 F 0 "R2" H 1120 3896 50  0000 L CNN
 F 1 "1k" H 1120 3805 50  0000 L CNN
-F 2 "" V 980 3850 50  0001 C CNN
+F 2 "Resistor_THT:R_Axial_DIN0207_L6.3mm_D2.5mm_P10.16mm_Horizontal" V 980 3850 50  0001 C CNN
 F 3 "~" H 1050 3850 50  0001 C CNN
 	1    1050 3850

Commit message: Associate more components
Parts:
- C811: footprint (none) -> Capacitor_THT:CP_Radial_D8.0mm_P5.00mm
Changed lines of the file:
@@
 F 0 "C811" H 5468 8596 50  0000 L CNN
 F 1 "4.7uF 16V" H 5468 8505 50  0000 L CNN
-F 2 "" H 5388 8400 50  0001 C CNN
+F 2 "Capacitor_THT:CP_Radial_D8.0mm_P5.00mm" H 5388 8400 50  0001 C CNN
 F 3 "~" H 5350 8550 50  0001 C CNN
 	1    5350 8550

Commit message: Update footprints
Parts:
- C800, C802, C803, C804, C810, C812, C904, C920: footprint (none) -> Capacitor_THT:C_Rect_L11.0mm_W2.8mm_P10.00mm_MKT
Changed lines of the file:
@@
 F 0 "C920" H 3915 4946 50  0000 L CNN
 F 1 "100pF" H 3915 4855 50  0000 L CNN
-F 2 "" H 3838 4750 50  0001 C CNN
+F 2 "Capacitor_THT:C_Rect_L11.0mm_W2.8mm_P10.00mm_MKT" H 3838 4750 50  0001 C CNN
 F 3 "~" H 3800 4900 50  0001 C CNN
 F 4 "To check on PCB" H 3800 4750 50  0000 C CNN "Notes"
@@
 F 0 "C904" H 4465 4946 50  0000 L CNN
 F 1 "100pF" H 4465 4855 50  0000 L CNN
-F 2 "" H 4388 4750 50  0001 C CNN
+F 2 "Capacitor_THT:C_Rect_L11.0mm_W2.8mm_P10.00mm_MKT" H 4388 4750 50  0001 C CNN
 F 3 "~" H 4350 4900 50  0001 C CNN
 	1    4350 4900
@@
 F 0 "C800" V 2248 5500 50  0000 C CNN
 F 1 "0.1uF" V 2339 5500 50  0000 C CNN
-F 2 "" H 2538 5350 50  0001 C CNN
+F 2 "Capacitor_THT:C_Rect_L11.0mm_W2.8mm_P10.00mm_MKT" H 2538 5350 50  0001 C CNN
 F 3 "~" H 2500 5500 50  0001 C CNN
 	1    2500 5500
@@
 F 0 "C810" H 4115 9996 50  0000 L CNN
 F 1 "20pF" H 4115 9905 50  0000 L CNN
-F 2 "" H 4038 9800 50  0001 C CNN
+F 2 "Capacitor_THT:C_Rect_L11.0mm_W2.8mm_P10.00mm_MKT" H 4038 9800 50  0001 C CNN
 F 3 "~" H 4000 9950 50  0001 C CNN
 	1    4000 9950
@@
 F 0 "C812" H 5965 8396 50  0000 L CNN
 F 1 "0.1uF" H 5965 8305 50  0000 L CNN
-F 2 "" H 5888 8200 50  0001 C CNN
+F 2 "Capacitor_THT:C_Rect_L11.0mm_W2.8mm_P10.00mm_MKT" H 5888 8200 50  0001 C CNN
 F 3 "~" H 5850 8350 50  0001 C CNN
 	1    5850 8350
@@
 F 0 "C803" H 11215 5596 50  0000 L CNN
 F 1 "0.1uF" H 11215 5505 50  0000 L CNN
-F 2 "" H 11138 5400 50  0001 C CNN
+F 2 "Capacitor_THT:C_Rect_L11.0mm_W2.8mm_P10.00mm_MKT" H 11138 5400 50  0001 C CNN
 F 3 "~" H 11100 5550 50  0001 C CNN
 	1    11100 5550
@@
 F 0 "C804" H 14865 3346 50  0000 L CNN
 F 1 "0.1uF" H 14865 3255 50  0000 L CNN
-F 2 "" H 14788 3150 50  0001 C CNN
+F 2 "Capacitor_THT:C_Rect_L11.0mm_W2.8mm_P10.00mm_MKT" H 14788 3150 50  0001 C CNN
 F 3 "~" H 14750 3300 50  0001 C CNN
 	1    14750 3300
@@
 F 0 "C802" H 5415 3496 50  0000 L CNN
 F 1 "0.1uF" H 5415 3405 50  0000 L CNN
-F 2 "" H 5338 3300 50  0001 C CNN
+F 2 "Capacitor_THT:C_Rect_L11.0mm_W2.8mm_P10.00mm_MKT" H 5338 3300 50  0001 C CNN
 F 3 "~" H 5300 3450 50  0001 C CNN
 	1    5300 3450

Commit message: Make caps footprint smaller
Parts:
- C800, C802, C803, C804, C810, C812, C904, C920: footprint Capacitor_THT:C_Rect_L11.0mm_W2.8mm_P10.00mm_MKT -> Capacitor_THT:C_Rect_L11.5mm_W2.0mm_P10.00mm_MKT
Changed lines of the file:
@@
 F 0 "C920" H 3915 4946 50  0000 L CNN
 F 1 "100pF" H 3915 4855 50  0000 L CNN
-F 2 "Capacitor_THT:C_Rect_L11.0mm_W2.8mm_P10.00mm_MKT" H 3838 4750 50  0001 C CNN
+F 2 "Capacitor_THT:C_Rect_L11.5mm_W2.0mm_P10.00mm_MKT" H 3838 4750 50  0001 C CNN
 F 3 "~" H 3800 4900 50  0001 C CNN
 F 4 "To check on PCB" H 3800 4750 50  0000 C CNN "Notes"
@@
 F 0 "C904" H 4465 4946 50  0000 L CNN
 F 1 "100pF" H 4465 4855 50  0000 L CNN
-F 2 "Capacitor_THT:C_Rect_L11.0mm_W2.8mm_P10.00mm_MKT" H 4388 4750 50  0001 C CNN
+F 2 "Capacitor_THT:C_Rect_L11.5mm_W2.0mm_P10.00mm_MKT" H 4388 4750 50  0001 C CNN
 F 3 "~" H 4350 4900 50  0001 C CNN
 	1    4350 4900
@@
 F 0 "C800" V 2248 5500 50  0000 C CNN
 F 1 "0.1uF" V 2339 5500 50  0000 C CNN
-F 2 "Capacitor_THT:C_Rect_L11.0mm_W2.8mm_P10.00mm_MKT" H 2538 5350 50  0001 C CNN
+F 2 "Capacitor_THT:C_Rect_L11.5mm_W2.0mm_P10.00mm_MKT" H 2538 5350 50  0001 C CNN
 F 3 "~" H 2500 5500 50  0001 C CNN
 	1    2500 5500
@@
 F 0 "C810" H 4115 9996 50  0000 L CNN
 F 1 "20pF" H 4115 9905 50  0000 L CNN
-F 2 "Capacitor_THT:C_Rect_L11.0mm_W2.8mm_P10.00mm_MKT" H 4038 9800 50  0001 C CNN
+F 2 "Capacitor_THT:C_Rect_L11.5mm_W2.0mm_P10.00mm_MKT" H 4038 9800 50  0001 C CNN
 F 3 "~" H 4000 9950 50  0001 C CNN
 	1    4000 9950
@@
 F 0 "C812" H 5965 8396 50  0000 L CNN
 F 1 "0.1uF" H 5965 8305 50  0000 L CNN
-F 2 "Capacitor_THT:C_Rect_L11.0mm_W2.8mm_P10.00mm_MKT" H 5888 8200 50  0001 C CNN
+F 2 "Capacitor_THT:C_Rect_L11.5mm_W2.0mm_P10.00mm_MKT" H 5888 8200 50  0001 C CNN
 F 3 "~" H 5850 8350 50  0001 C CNN
 	1    5850 8350
@@
 F 0 "C803" H 11215 5596 50  0000 L CNN
 F 1 "0.1uF" H 11215 5505 50  0000 L CNN
-F 2 "Capacitor_THT:C_Rect_L11.0mm_W2.8mm_P10.00mm_MKT" H 11138 5400 50  0001 C CNN
+F 2 "Capacitor_THT:C_Rect_L11.5mm_W2.0mm_P10.00mm_MKT" H 11138 5400 50  0001 C CNN
 F 3 "~" H 11100 5550 50  0001 C CNN
 	1    11100 5550
@@
 F 0 "C804" H 14865 3346 50  0000 L CNN
 F 1 "0.1uF" H 14865 3255 50  0000 L CNN
-F 2 "Capacitor_THT:C_Rect_L11.0mm_W2.8mm_P10.00mm_MKT" H 14788 3150 50  0001 C CNN
+F 2 "Capacitor_THT:C_Rect_L11.5mm_W2.0mm_P10.00mm_MKT" H 14788 3150 50  0001 C CNN
 F 3 "~" H 14750 3300 50  0001 C CNN
 	1    14750 3300
@@
 F 0 "C802" H 5415 3496 50  0000 L CNN
 F 1 "0.1uF" H 5415 3405 50  0000 L CNN
-F 2 "Capacitor_THT:C_Rect_L11.0mm_W2.8mm_P10.00mm_MKT" H 5338 3300 50  0001 C CNN
+F 2 "Capacitor_THT:C_Rect_L11.5mm_W2.0mm_P10.00mm_MKT" H 5338 3300 50  0001 C CNN
 F 3 "~" H 5300 3450 50  0001 C CNN
 	1    5300 3450
