File: expansion logic.sch (KiCad schematic (older format))
At the start: 31 parts, among them U302 74LS32, U800 BUSTER5721, U801 MSM6242, U802 74LS138, U803 74LS08, U804 74LS148, Y800 32768Hz

Commit message: It's ok
Parts:
- C920: Notes To check on PCB -> (none)
Changed lines of the file:
@@
 F 2 "Capacitor_THT:C_Rect_L11.5mm_W2.0mm_P10.00mm_MKT" H 3838 4750 50  0001 C CNN
 F 3 "~" H 3800 4900 50  0001 C CNN
-F 4 "To check on PCB" H 3800 4750 50  0000 C CNN "Notes"
 	1    3800 4900
 	1    0    0    -1

Commit message: Switch footprints for suitable modern replacements
Parts:
- C800, C802, C803, C804, C810, C812, C904, C920: footprint Capacitor_THT:C_Rect_L11.5mm_W2.0mm_P10.00mm_MKT -> Capacitor_THT:C_Rect_L11.5mm_W2.6mm_P10.00mm_MKT
- C811: footprint Capacitor_THT:CP_Radial_D8.0mm_P5.00mm -> Capacitor_THT:CP_Radial_D5.0mm_P2.50mm
- Y800: footprint Crystal:Crystal_DS10_D1.0mm_L4.3mm_Horizontal -> Crystal:Crystal_DS15_D1.5mm_L5.0mm_Horizontal
Changed lines of the file:
@@
 F 0 "C920" H 3915 4946 50  0000 L CNN
 F 1 "100pF" H 3915 4855 50  0000 L CNN
-F 2 "Capacitor_THT:C_Rect_L11.5mm_W2.0mm_P10.00mm_MKT" H 3838 4750 50  0001 C CNN
+F 2 "Capacitor_THT:C_Rect_L11.5mm_W2.6mm_P10.00mm_MKT" H 3838 4750 50  0001 C CNN
 F 3 "~" H 3800 4900 50  0001 C CNN
 	1    3800 4900
@@
 F 0 "C904" H 4465 4946 50  0000 L CNN
 F 1 "100pF" H 4465 4855 50  0000 L CNN
-F 2 "Capacitor_THT:C_Rect_L11.5mm_W2.0mm_P10.00mm_MKT" H 4388 4750 50  0001 C CNN
+F 2 "Capacitor_THT:C_Rect_L11.5mm_W2.6mm_P10.00mm_MKT" H 4388 4750 50  0001 C CNN
 F 3 "~" H 4350 4900 50  0001 C CNN
 	1    4350 4900
@@
 F 0 "C800" V 2248 5500 50  0000 C CNN
 F 1 "0.1uF" V 2339 5500 50  0000 C CNN
-F 2 "Capacitor_THT:C_Rect_L11.5mm_W2.0mm_P10.00mm_MKT" H 2538 5350 50  0001 C CNN
+F 2 "Capacitor_THT:C_Rect_L11.5mm_W2.6mm_P10.00mm_MKT" H 2538 5350 50  0001 C CNN
 F 3 "~" H 2500 5500 50  0001 C CNN
 	1    2500 5500
@@
 F 0 "Y800" H 4450 9918 50  0000 C CNN
 F 1 "32768Hz" H 4450 9827 50  0000 C CNN
-F 2 "Crystal:Crystal_DS10_D1.0mm_L4.3mm_Horizontal" H 4450 9650 50  0001 C CNN
+F 2 "Crystal:Crystal_DS15_D1.5mm_L5.0mm_Horizontal" H 4450 9650 50  0001 C CNN
 F 3 "~" H 4450 9650 50  0001 C CNN
 	1    4450 9650
@@
 F 0 "C810" H 4115 9996 50  0000 L CNN
 F 1 "20pF" H 4115 9905 50  0000 L CNN
-F 2 "Capacitor_THT:C_Rect_L11.5mm_W2.0mm_P10.00mm_MKT" H 4038 9800 50  0001 C CNN
+F 2 "Capacitor_THT:C_Rect_L11.5mm_W2.6mm_P10.00mm_MKT" H 4038 9800 50  0001 C CNN
 F 3 "~" H 4000 9950 50  0001 C CNN
 	1    4000 9950
@@
 F 0 "C811" H 5468 8596 50  0000 L CNN
 F 1 "4.7uF 16V" H 5468 8505 50  0000 L CNN
-F 2 "Capacitor_THT:CP_Radial_D8.0mm_P5.00mm" H 5388 8400 50  0001 C CNN
+F 2 "Capacitor_THT:CP_Radial_D5.0mm_P2.50mm" H 5388 8400 50  0001 C CNN
 F 3 "~" H 5350 8550 50  0001 C CNN
 	1    5350 8550
@@
 F 0 "C812" H 5965 8396 50  0000 L CNN
 F 1 "0.1uF" H 5965 8305 50  0000 L CNN
-F 2 "Capacitor_THT:C_Rect_L11.5mm_W2.0mm_P10.00mm_MKT" H 5888 8200 50  0001 C CNN
+F 2 "Capacitor_THT:C_Rect_L11.5mm_W2.6mm_P10.00mm_MKT" H 5888 8200 50  0001 C CNN
 F 3 "~" H 5850 8350 50  0001 C CNN
 	1    5850 8350
@@
 F 0 "C803" H 11215 5596 50  0000 L CNN
 F 1 "0.1uF" H 11215 5505 50  0000 L CNN
-F 2 "Capacitor_THT:C_Rect_L11.5mm_W2.0mm_P10.00mm_MKT" H 11138 5400 50  0001 C CNN
+F 2 "Capacitor_THT:C_Rect_L11.5mm_W2.6mm_P10.00mm_MKT" H 11138 5400 50  0001 C CNN
 F 3 "~" H 11100 5550 50  0001 C CNN
 	1    11100 5550
@@
 F 0 "C804" H 14865 3346 50  0000 L CNN
 F 1 "0.1uF" H 14865 3255 50  0000 L CNN
-F 2 "Capacitor_THT:C_Rect_L11.5mm_W2.0mm_P10.00mm_MKT" H 14788 3150 50  0001 C CNN
+F 2 "Capacitor_THT:C_Rect_L11.5mm_W2.6mm_P10.00mm_MKT" H 14788 3150 50  0001 C CNN
 F 3 "~" H 14750 3300 50  0001 C CNN
 	1    14750 3300
@@
 F 0 "C802" H 5415 3496 50  0000 L CNN
 F 1 "0.1uF" H 5415 3405 50  0000 L CNN
-F 2 "Capacitor_THT:C_Rect_L11.5mm_W2.0mm_P10.00mm_MKT" H 5338 3300 50  0001 C CNN
+F 2 "Capacitor_THT:C_Rect_L11.5mm_W2.6mm_P10.00mm_MKT" H 5338 3300 50  0001 C CNN
 F 3 "~" H 5300 3450 50  0001 C CNN
 	1    5300 3450

Commit message: Some footprints updates; Add all Mouser references
Parts:
- C800, C802, C803, C804, C812: RefOrder (none) -> 581-SA105C104KARC
- C810: RefOrder (none) -> 581-SA102A200JAR
- C811: RefOrder (none) -> 647-UMA1C4R7MCD2TP
- C904, C920: RefOrder (none) -> 80-C410C101K5G
- D800, D801: RefOrder (none) -> 78-1N4148
- R2, R800: RefOrder (none) -> 603-CFR-25JR-521K
- R801, R803: RefOrder (none) -> 603-CFR-25JT-52-470R
- R804: RefOrder (none) -> 603-CFR-25JR-5210K
- R806, R807: RefOrder (none) -> 603-CFR-25JT-52-4K7
- R904, R905: RefOrder (none) -> 603-CFR-25JT-52-47R
- RP800: RefOrder (none) -> 652-4608X-AP1-102LF
- RP801: RefOrder (none) -> 652-4608X-AP1-472LF
- U302: RefOrder (none) -> 595-SN74LS32N
- U802: RefOrder (none) -> 595-SN74LS138N
- U803: RefOrder (none) -> 595-SN74LS08N
- U804: RefOrder (none) -> 595-SN74LS148N
- Y800: RefOrder (none) -> 695-CFS145-327K-U
Changed lines of the file:
@@
 F 2 "Resistor_THT:R_Axial_DIN0207_L6.3mm_D2.5mm_P10.16mm_Horizontal" V 3180 2200 50  0001 C CNN
 F 3 "~" H 3250 2200 50  0001 C CNN
+F 4 "603-CFR-25JT-52-47R" H 3250 2200 50  0001 C CNN "RefOrder"
 	1    3250 2200
 	0    1    1    0
@@
 F 2 "Resistor_THT:R_Axial_DIN0207_L6.3mm_D2.5mm_P10.16mm_Horizontal" V 3430 3350 50  0001 C CNN
 F 3 "~" H 3500 3350 50  0001 C CNN
+F 4 "603-CFR-25JT-52-4K7" H 3500 3350 50  0001 C CNN "RefOrder"
 	1    3500 3350
 	-1   0    0    1
@@
 F 2 "Resistor_THT:R_Axial_DIN0207_L6.3mm_D2.5mm_P10.16mm_Horizontal" V 3780 3350 50  0001 C CNN
 F 3 "~" H 3850 3350 50  0001 C CNN
+F 4 "603-CFR-25JT-52-4K7" H 3850 3350 50  0001 C CNN "RefOrder"
 	1    3850 3350
 	-1   0    0    1
@@
 F 2 "Resistor_THT:R_Axial_DIN0207_L6.3mm_D2.5mm_P10.16mm_Horizontal" V 3230 4550 50  0001 C CNN
 F 3 "~" H 3300 4550 50  0001 C CNN
+F 4 "603-CFR-25JT-52-47R" H 3300 4550 50  0001 C CNN "RefOrder"
 	1    3300 4550
 	0    -1   -1   0
@@
 F 2 "Capacitor_THT:C_Rect_L11.5mm_W2.6mm_P10.00mm_MKT" H 3838 4750 50  0001 C CNN
 F 3 "~" H 3800 4900 50  0001 C CNN
+F 4 "80-C410C101K5G" H 3800 4900 50  0001 C CNN "RefOrder"
 	1    3800 4900
 	1    0    0    -1
@@
 F 2 "Capacitor_THT:C_Rect_L11.5mm_W2.6mm_P10.00mm_MKT" H 4388 4750 50  0001 C CNN
 F 3 "~" H 4350 4900 50  0001 C CNN
+F 4 "80-C410C101K5G" H 4350 4900 50  0001 C CNN "RefOrder"
 	1    4350 4900
 	1    0    0    -1
@@
 F 2 "Capacitor_THT:C_Rect_L11.5mm_W2.6mm_P10.00mm_MKT" H 2538 5350 50  0001 C CNN
 F 3 "~" H 2500 5500 50  0001 C CNN
+F 4 "581-SA105C104KARC" H 2500 5500 50  0001 C CNN "RefOrder"
 	1    2500 5500
 	0    1    1    0
@@
 F 2 "Package_DIP:DIP-14_W7.62mm_Socket" H 1150 5000 50  0001 C CNN
 F 3 "http://www.ti.com/lit/gpn/sn74LS32" H 1150 5000 50  0001 C CNN
+F 4 "595-SN74LS32N" H 1150 5000 50  0001 C CNN "RefOrder"
 	4    1150 5000
 	-1   0    0    -1
@@
 F 2 "Resistor_THT:R_Axial_DIN0207_L6.3mm_D2.5mm_P10.16mm_Horizontal" V 1630 4850 50  0001 C CNN
 F 3 "~" H 1700 4850 50  0001 C CNN
+F 4 "603-CFR-25JR-521K" H 1700 4850 50  0001 C CNN "RefOrder"
 	1    1700 4850
 	0    -1   -1   0
@@
 F 2 "Resistor_THT:R_Array_SIP8" V 1475 1050 50  0001 C CNN
 F 3 "http://www.vishay.com/docs/31509/csc.pdf" H 1000 1050 50  0001 C CNN
+F 4 "652-4608X-AP1-102LF" H 1000 1050 50  0001 C CNN "RefOrder"
 	1    1000 1050
 	-1   0    0    -1
@@
 F 2 "Crystal:Crystal_DS15_D1.5mm_L5.0mm_Horizontal" H 4450 9650 50  0001 C CNN
 F 3 "~" H 4450 9650 50  0001 C CNN
+F 4 "695-CFS145-327K-U" H 4450 9650 50  0001 C CNN "RefOrder"
 	1    4450 9650
 	1    0    0    -1
@@
 F 2 "Capacitor_THT:C_Rect_L11.5mm_W2.6mm_P10.00mm_MKT" H 4038 9800 50  0001 C CNN
 F 3 "~" H 4000 9950 50  0001 C CNN
+F 4 "581-SA102A200JAR" H 4000 9950 50  0001 C CNN "RefOrder"
 	1    4000 9950
 	1    0    0    -1
@@
 F 2 "Capacitor_THT:CP_Radial_D5.0mm_P2.50mm" H 5388 8400 50  0001 C CNN
 F 3 "~" H 5350 8550 50  0001 C CNN
+F 4 "647-UMA1C4R7MCD2TP" H 5350 8550 50  0001 C CNN "RefOrder"
 	1    5350 8550
 	1    0    0    -1
@@
 F 2 "Capacitor_THT:C_Rect_L11.5mm_W2.6mm_P10.00mm_MKT" H 5888 8200 50  0001 C CNN
 F 3 "~" H 5850 8350 50  0001 C CNN
+F 4 "581-SA105C104KARC" H 5850 8350 50  0001 C CNN "RefOrder"
 	1    5850 8350
 	1    0    0    -1
@@
 F 2 "Resistor_THT:R_Axial_DIN0207_L6.3mm_D2.5mm_P10.16mm_Horizontal" V 5130 6800 50  0001 C CNN
 F 3 "~" H 5200 6800 50  0001 C CNN
+F 4 "603-CFR-25JR-5210K" H 5200 6800 50  0001 C CNN "RefOrder"
 	1    5200 6800
 	1    0    0    -1
@@
 F 2 "Diode_THT:D_DO-35_SOD27_P7.62mm_Horizontal" H 5800 6875 50  0001 C CNN
 F 3 "https://assets.nexperia.com/documents/data-sheet/1N4148_1N4448.pdf" H 5800 7050 50  0001 C CNN
+F 4 "78-1N4148" H 5800 7050 50  0001 C CNN "RefOrder"
 	1    5800 7050
 	1    0    0    -1
@@
 F 2 "Resistor_THT:R_Axial_DIN0207_L6.3mm_D2.5mm_P10.16mm_Horizontal" V 6230 6800 50  0001 C CNN
 F 3 "~" H 6300 6800 50  0001 C CNN
+F 4 "603-CFR-25JT-52-470R" H 6300 6800 50  0001 C CNN "RefOrder"
 	1    6300 6800
 	1    0    0    -1
@@
 F 2 "Diode_THT:D_DO-35_SOD27_P7.62mm_Horizontal" H 6300 7125 50  0001 C CNN
 F 3 "https://assets.nexperia.com/documents/data-sheet/1N4148_1N4448.pdf" H 6300 7300 50  0001 C CNN
+F 4 "78-1N4148" H 6300 7300 50  0001 C CNN "RefOrder"
 	1    6300 7300
 	0    -1   -1   0
@@
 F 2 "Resistor_THT:R_Axial_DIN0207_L6.3mm_D2.5mm_P10.16mm_Horizontal" V 6230 7800 50  0001 C CNN
 F 3 "~" H 6300 7800 50  0001 C CNN
+F 4 "603-CFR-25JT-52-470R" H 6300 7800 50  0001 C CNN "RefOrder"
 	1    6300 7800
 	1    0    0    -1
@@
 F 2 "Package_DIP:DIP-16_W7.62mm_Socket" H 8000 3300 50  0001 C CNN
 F 3 "http://www.ti.com/lit/gpn/sn74LS138" H 8000 3300 50  0001 C CNN
+F 4 "595-SN74LS138N" H 8000 3300 50  0001 C CNN "RefOrder"
 	1    8000 3300
 	1    0    0    1
@@
 F 2 "Package_DIP:DIP-16_W7.62mm_Socket" H 12800 3350 50  0001 C CNN
 F 3 "http://www.ti.com/lit/gpn/sn74LS148" H 12800 3350 50  0001 C CNN
+F 4 "595-SN74LS148N" H 12800 3350 50  0001 C CNN "RefOrder"
 	1    12800 3350
 	1    0    0    -1
@@
 F 2 "Package_DIP:DIP-14_W7.62mm_Socket" H 10300 2450 50  0001 C CNN
 F 3 "http://www.ti.com/lit/gpn/sn74LS08" H 10300 2450 50  0001 C CNN
+F 4 "595-SN74LS08N" H 10300 2450 50  0001 C CNN "RefOrder"
 	1    10300 2450
 	1    0    0    -1
@@
 F 2 "Package_DIP:DIP-14_W7.62mm_Socket" H 10300 3000 50  0001 C CNN
 F 3 "http://www.ti.com/lit/gpn/sn74LS08" H 10300 3000 50  0001 C CNN
+F 4 "595-SN74LS08N" H 10300 3000 50  0001 C CNN "RefOrder"
 	2    10300 3000
 	1    0    0    -1
@@
 F 2 "Package_DIP:DIP-14_W7.62mm_Socket" H 10300 3550 50  0001 C CNN
 F 3 "http://www.ti.com/lit/gpn/sn74LS08" H 10300 3550 50  0001 C CNN
+F 4 "595-SN74LS08N" H 10300 3550 50  0001 C CNN "RefOrder"
 	3    10300 3550
 	1    0    0    -1
@@
 F 2 "Package_DIP:DIP-14_W7.62mm_Socket" H 10300 4100 50  0001 C CNN
 F 3 "http://www.ti.com/lit/gpn/sn74LS08" H 10300 4100 50  0001 C CNN
+F 4 "595-SN74LS08N" H 10300 4100 50  0001 C CNN "RefOrder"
 	4    10300 4100
 	1    0    0    -1
@@
 F 2 "Package_DIP:DIP-14_W7.62mm_Socket" H 10300 5600 50  0001 C CNN
 F 3 "http://www.ti.com/lit/gpn/sn74LS08" H 10300 5600 50  0001 C CNN
+F 4 "595-SN74LS08N" H 10300 5600 50  0001 C CNN "RefOrder"
 	5    10300 5600
 	1    0    0    -1
@@
 F 2 "Capacitor_THT:C_Rect_L11.5mm_W2.6mm_P10.00mm_MKT" H 11138 5400 50  0001 C CNN
 F 3 "~" H 11100 5550 50  0001 C CNN
+F 4 "581-SA105C104KARC" H 11100 5550 50  0001 C CNN "RefOrder"
 	1    11100 5550
 	1    0    0    -1
@@
 F 2 "Resistor_THT:R_Array_SIP8" V 6575 2650 50  0001 C CNN
 F 3 "http://www.vishay.com/docs/31509/csc.pdf" H 6100 2650 50  0001 C CNN
+F 4 "652-4608X-AP1-472LF" H 6100 2650 50  0001 C CNN "RefOrder"
 	1    6100 2650
 	-1   0    0    -1
@@
 F 2 "Capacitor_THT:C_Rect_L11.5mm_W2.6mm_P10.00mm_MKT" H 14788 3150 50  0001 C CNN
 F 3 "~" H 14750 3300 50  0001 C CNN
+F 4 "581-SA105C104KARC" H 14750 3300 50  0001 C CNN "RefOrder"
 	1    14750 3300
 	1    0    0    -1
@@
 F 2 "Capacitor_THT:C_Rect_L11.5mm_W2.6mm_P10.00mm_MKT" H 5338 3300 50  0001 C CNN
 F 3 "~" H 5300 3450 50  0001 C CNN
+F 4 "581-SA105C104KARC" H 5300 3450 50  0001 C CNN "RefOrder"
 	1    5300 3450
 	1    0    0    -1
@@
 F 2 "Resistor_THT:R_Axial_DIN0207_L6.3mm_D2.5mm_P10.16mm_Horizontal" V 980 3850 50  0001 C CNN
 F 3 "~" H 1050 3850 50  0001 C CNN
+F 4 "603-CFR-25JR-521K" H 1050 3850 50  0001 C CNN "RefOrder"
 	1    1050 3850
 	1    0    0    -1
