File: paula.sch (KiCad schematic (older format))
At the start: 79 parts, among them CN200 DB9P RIGHT(1), CN201 DB9P LEFT(0), CN204 RIGHT AUDIO, CN205 LEFT AUDIO, J200 Conn_01x03_Male, Q200 MPF102, Q201 MPF102, Q202 2N3906, U200 PAULA, U202 74LS157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

Commit message: Associate footprints with components
Parts:
- CN200, CN201: footprint (none) -> Connector_Dsub:DSUB-9_Male_Horizontal_P2.77x2.84mm_EdgePinOffset7.70mm_Housed_MountingHolesOffset9.12mm
- EMI230, EMI231, EMI232, EMI233, EMI234, EMI235, EMI236, EMI237, EMI238, EMI239, EMI240, EMI241, EMI242, EMI243, J200: footprint (none) -> Connector_PinSocket_2.54mm:PinSocket_1x03_P2.54mm_Vertical
- F1: footprint (none) -> Fuse:Fuse_Littelfuse-LVR100
- FB215, FB401: footprint (none) -> Inductor_THT:L_Axial_L7.0mm_D3.3mm_P10.16mm_Horizontal_Fastron_MICC
- Q200, Q201: footprint (none) -> Package_TO_SOT_THT:TO-92_Inline
- R200, R202, R204, R205, R206, R207, R208, R209, R210, R213, R214, R230, R231, R232, R233, R234, R240, R241, R242, R243, R244, R900: footprint (none) -> Resistor_THT:R_Axial_DIN0207_L6.3mm_D2.5mm_P10.16mm_Horizontal
- U200: footprint (none) -> Package_DIP:DIP-48_W15.24mm_Socket
- U202: footprint (none) -> Package_DIP:DIP-16_W7.62mm_Socket
- U204: footprint (none) -> Package_DIP:DIP-14_W7.62mm_Socket

Commit message: Associate more components
Parts:
- C222, C223, C224, C243: footprint (none) -> Capacitor_THT:CP_Radial_D8.0mm_P5.00mm
- C225: footprint (none) -> Capacitor_THT:CP_Radial_D10.0mm_P5.00mm
- C233: footprint (none) -> Capacitor_THT:CP_Radial_D10.0mm_P2.50mm
Changed lines of the file:
@@
 F 0 "C225" V 2900 700 50  0000 C CNN
 F 1 "470uF 16v" V 2800 500 50  0000 C CNN
-F 2 "" H 2788 600 50  0001 C CNN
+F 2 "Capacitor_THT:CP_Radial_D10.0mm_P5.00mm" H 2788 600 50  0001 C CNN
 F 3 "~" H 2750 750 50  0001 C CNN
 	1    2750 750
@@
 F 0 "C222" H 11268 7346 50  0000 L CNN
 F 1 "47uF 16V" H 11268 7255 50  0000 L CNN
-F 2 "" H 11188 7150 50  0001 C CNN
+F 2 "Capacitor_THT:CP_Radial_D8.0mm_P5.00mm" H 11188 7150 50  0001 C CNN
 F 3 "~" H 11150 7300 50  0001 C CNN
 	1    11150 7300
@@
 F 0 "C223" H 11268 7846 50  0000 L CNN
 F 1 "47uF 16V" H 11268 7755 50  0000 L CNN
-F 2 "" H 11188 7650 50  0001 C CNN
+F 2 "Capacitor_THT:CP_Radial_D8.0mm_P5.00mm" H 11188 7650 50  0001 C CNN
 F 3 "~" H 11150 7800 50  0001 C CNN
 	1    11150 7800
@@
 F 0 "C243" V 12205 1700 50  0000 C CNN
 F 1 "22uF 16V" V 12114 1700 50  0000 C CNN
-F 2 "" H 11988 1550 50  0001 C CNN
+F 2 "Capacitor_THT:CP_Radial_D8.0mm_P5.00mm" H 11988 1550 50  0001 C CNN
 F 3 "~" H 11950 1700 50  0001 C CNN
 	1    11950 1700
@@
 F 0 "C233" V 12205 3850 50  0000 C CNN
 F 1 "22uF 16V" V 12114 3850 50  0000 C CNN
-F 2 "" H 11988 3700 50  0001 C CNN
+F 2 "Capacitor_THT:CP_Radial_D10.0mm_P2.50mm" H 11988 3700 50  0001 C CNN
 F 3 "~" H 11950 3850 50  0001 C CNN
 	1    11950 3850
@@
 F 0 "C224" H 14568 8996 50  0000 L CNN
 F 1 "4.7uF 16V" H 14568 8905 50  0000 L CNN
-F 2 "" H 14488 8800 50  0001 C CNN
+F 2 "Capacitor_THT:CP_Radial_D8.0mm_P5.00mm" H 14488 8800 50  0001 C CNN
 F 3 "~" H 14450 8950 50  0001 C CNN
 	1    14450 8950

Commit message: Update footprints
Parts:
- C200, C202, C204, C210, C211, C212, C213, C218, C219, C220, C221, C230, C231, C232, C234, C240, C241, C242, C244, C900, C901: footprint (none) -> Capacitor_THT:C_Rect_L11.0mm_W2.8mm_P10.00mm_MKT
Changed lines of the file:
@@
 F 0 "C200" V 2350 950 50  0000 C CNN
 F 1 "0.1uF" V 2650 950 50  0000 C CNN
-F 2 "" H 2538 800 50  0001 C CNN
+F 2 "Capacitor_THT:C_Rect_L11.0mm_W2.8mm_P10.00mm_MKT" H 2538 800 50  0001 C CNN
 F 3 "~" H 2500 950 50  0001 C CNN
 	1    2500 950
@@
 F 0 "C210" H 3915 6046 50  0000 L CNN
 F 1 "0.047uF" H 3915 5955 50  0000 L CNN
-F 2 "" H 3838 5850 50  0001 C CNN
+F 2 "Capacitor_THT:C_Rect_L11.0mm_W2.8mm_P10.00mm_MKT" H 3838 5850 50  0001 C CNN
 F 3 "~" H 3800 6000 50  0001 C CNN
 	1    3800 6000
@@
 F 0 "C211" H 4465 6046 50  0000 L CNN
 F 1 "0.047uF" H 4465 5955 50  0000 L CNN
-F 2 "" H 4388 5850 50  0001 C CNN
+F 2 "Capacitor_THT:C_Rect_L11.0mm_W2.8mm_P10.00mm_MKT" H 4388 5850 50  0001 C CNN
 F 3 "~" H 4350 6000 50  0001 C CNN
 	1    4350 6000
@@
 F 0 "C212" H 5015 6046 50  0000 L CNN
 F 1 "0.047uF" H 5015 5955 50  0000 L CNN
-F 2 "" H 4938 5850 50  0001 C CNN
+F 2 "Capacitor_THT:C_Rect_L11.0mm_W2.8mm_P10.00mm_MKT" H 4938 5850 50  0001 C CNN
 F 3 "~" H 4900 6000 50  0001 C CNN
 	1    4900 6000
@@
 F 0 "C213" H 5565 6046 50  0000 L CNN
 F 1 "0.047uF" H 5565 5955 50  0000 L CNN
-F 2 "" H 5488 5850 50  0001 C CNN
+F 2 "Capacitor_THT:C_Rect_L11.0mm_W2.8mm_P10.00mm_MKT" H 5488 5850 50  0001 C CNN
 F 3 "~" H 5450 6000 50  0001 C CNN
 	1    5450 6000
@@
 F 0 "C218" V 6721 6750 50  0000 C CNN
 F 1 "0.047uF" V 6812 6750 50  0000 C CNN
-F 2 "" H 6950 6750 50  0001 C CNN
+F 2 "Capacitor_THT:C_Rect_L11.0mm_W2.8mm_P10.00mm_MKT" H 6950 6750 50  0001 C CNN
 F 3 "~" H 6950 6750 50  0001 C CNN
 	1    6950 6750
@@
 F 0 "C202" H 3315 8646 50  0000 L CNN
 F 1 "0.1uF" H 3315 8555 50  0000 L CNN
-F 2 "" H 3238 8450 50  0001 C CNN
+F 2 "Capacitor_THT:C_Rect_L11.0mm_W2.8mm_P10.00mm_MKT" H 3238 8450 50  0001 C CNN
 F 3 "~" H 3200 8600 50  0001 C CNN
 	1    3200 8600
@@
 F 0 "C220" H 10715 7346 50  0000 L CNN
 F 1 "0.22uF" H 10715 7255 50  0000 L CNN
-F 2 "" H 10638 7150 50  0001 C CNN
+F 2 "Capacitor_THT:C_Rect_L11.0mm_W2.8mm_P10.00mm_MKT" H 10638 7150 50  0001 C CNN
 F 3 "~" H 10600 7300 50  0001 C CNN
 	1    10600 7300
@@
 F 0 "C221" H 10715 7846 50  0000 L CNN
 F 1 "0.22uF" H 10715 7755 50  0000 L CNN
-F 2 "" H 10638 7650 50  0001 C CNN
+F 2 "Capacitor_THT:C_Rect_L11.0mm_W2.8mm_P10.00mm_MKT" H 10638 7650 50  0001 C CNN
 F 3 "~" H 10600 7800 50  0001 C CNN
 	1    10600 7800
@@
 F 0 "C240" H 6665 1396 50  0000 L CNN
 F 1 "0.1uF" H 6665 1305 50  0000 L CNN
-F 2 "" H 6588 1200 50  0001 C CNN
+F 2 "Capacitor_THT:C_Rect_L11.0mm_W2.8mm_P10.00mm_MKT" H 6588 1200 50  0001 C CNN
 F 3 "~" H 6550 1350 50  0001 C CNN
 	1    6550 1350
@@
 F 0 "C241" H 8465 1196 50  0000 L CNN
 F 1 "6800pF" H 8465 1105 50  0000 L CNN
-F 2 "" H 8388 1000 50  0001 C CNN
+F 2 "Capacitor_THT:C_Rect_L11.0mm_W2.8mm_P10.00mm_MKT" H 8388 1000 50  0001 C CNN
 F 3 "~" H 8350 1150 50  0001 C CNN
 	1    8350 1150
@@
 F 0 "C242" H 9915 1846 50  0000 L CNN
 F 1 "3900pF" H 9915 1755 50  0000 L CNN
-F 2 "" H 9838 1650 50  0001 C CNN
+F 2 "Capacitor_THT:C_Rect_L11.0mm_W2.8mm_P10.00mm_MKT" H 9838 1650 50  0001 C CNN
 F 3 "~" H 9800 1800 50  0001 C CNN
 	1    9800 1800
@@
 F 0 "C244" H 13615 1996 50  0000 L CNN
 F 1 "0.1uF" H 13615 1905 50  0000 L CNN
-F 2 "" H 13538 1800 50  0001 C CNN
+F 2 "Capacitor_THT:C_Rect_L11.0mm_W2.8mm_P10.00mm_MKT" H 13538 1800 50  0001 C CNN
 F 3 "~" H 13500 1950 50  0001 C CNN
 	1    13500 1950
@@
 F 0 "C230" H 6665 3546 50  0000 L CNN
 F 1 "0.1uF" H 6665 3455 50  0000 L CNN
-F 2 "" H 6588 3350 50  0001 C CNN
+F 2 "Capacitor_THT:C_Rect_L11.0mm_W2.8mm_P10.00mm_MKT" H 6588 3350 50  0001 C CNN
 F 3 "~" H 6550 3500 50  0001 C CNN
 	1    6550 3500
@@
 F 0 "C231" H 8465 3346 50  0000 L CNN
 F 1 "6800pF" H 8465 3255 50  0000 L CNN
-F 2 "" H 8388 3150 50  0001 C CNN
+F 2 "Capacitor_THT:C_Rect_L11.0mm_W2.8mm_P10.00mm_MKT" H 8388 3150 50  0001 C CNN
 F 3 "~" H 8350 3300 50  0001 C CNN
 	1    8350 3300
@@
 F 0 "C232" H 9915 3996 50  0000 L CNN
 F 1 "3900pF" H 9915 3905 50  0000 L CNN
-F 2 "" H 9838 3800 50  0001 C CNN
+F 2 "Capacitor_THT:C_Rect_L11.0mm_W2.8mm_P10.00mm_MKT" H 9838 3800 50  0001 C CNN
 F 3 "~" H 9800 3950 50  0001 C CNN
 	1    9800 3950
@@
 F 0 "C234" H 13615 4146 50  0000 L CNN
 F 1 "0.1uF" H 13615 4055 50  0000 L CNN
-F 2 "" H 13538 3950 50  0001 C CNN
+F 2 "Capacitor_THT:C_Rect_L11.0mm_W2.8mm_P10.00mm_MKT" H 13538 3950 50  0001 C CNN
 F 3 "~" H 13500 4100 50  0001 C CNN
 	1    13500 4100
@@
 F 0 "C204" H 7865 5946 50  0000 L CNN
 F 1 "0.01uF" H 7865 5855 50  0000 L CNN
-F 2 "" H 7788 5750 50  0001 C CNN
+F 2 "Capacitor_THT:C_Rect_L11.0mm_W2.8mm_P10.00mm_MKT" H 7788 5750 50  0001 C CNN
 F 3 "~" H 7750 5900 50  0001 C CNN
 	1    7750 5900
@@
 F 0 "C219" H 14015 8996 50  0000 L CNN
 F 1 "0.22uF" H 14015 8905 50  0000 L CNN
-F 2 "" H 13938 8800 50  0001 C CNN
+F 2 "Capacitor_THT:C_Rect_L11.0mm_W2.8mm_P10.00mm_MKT" H 13938 8800 50  0001 C CNN
 F 3 "~" H 13900 8950 50  0001 C CNN
 	1    13900 8950
@@
 F 0 "C900" H 12965 7346 50  0000 L CNN
 F 1 "0.1uF" H 12965 7255 50  0000 L CNN
-F 2 "" H 12888 7150 50  0001 C CNN
+F 2 "Capacitor_THT:C_Rect_L11.0mm_W2.8mm_P10.00mm_MKT" H 12888 7150 50  0001 C CNN
 F 3 "~" H 12850 7300 50  0001 C CNN
 	1    12850 7300
@@
 F 0 "C901" H 12965 7846 50  0000 L CNN
 F 1 "0.1uF" H 12965 7755 50  0000 L CNN
-F 2 "" H 12888 7650 50  0001 C CNN
+F 2 "Capacitor_THT:C_Rect_L11.0mm_W2.8mm_P10.00mm_MKT" H 12888 7650 50  0001 C CNN
 F 3 "~" H 12850 7800 50  0001 C CNN
 	1    12850 7800

Commit message: RCA
Parts:
- CN204, CN205: footprint (none) -> d_amiga:RCA
Changed lines of the file:
@@
 F 0 "CN205" H 14700 1675 50  0000 L CNN
 F 1 "LEFT AUDIO" H 14450 1900 50  0000 L CNN
-F 2 "" H 14600 1700 50  0001 C CNN
+F 2 "d_amiga:RCA" H 14600 1700 50  0001 C CNN
 F 3 " ~" H 14600 1700 50  0001 C CNN
 	1    14600 1700
@@
 F 0 "CN204" H 14700 3825 50  0000 L CNN
 F 1 "RIGHT AUDIO" H 14700 3734 50  0000 L CNN
-F 2 "" H 14600 3850 50  0001 C CNN
+F 2 "d_amiga:RCA" H 14600 3850 50  0001 C CNN
 F 3 " ~" H 14600 3850 50  0001 C CNN
 	1    14600 3850

Commit message: More placement
Parts:
- J200: footprint Connector_PinSocket_2.54mm:PinSocket_1x03_P2.54mm_Vertical -> Connector_PinHeader_2.54mm:PinHeader_1x03_P2.54mm_Vertical
Changed lines of the file:
@@
 F 0 "J200" H 10373 9228 50  0000 R CNN
 F 1 "Conn_01x03_Male" H 10372 9273 50  0001 R CNN
-F 2 "Connector_PinSocket_2.54mm:PinSocket_1x03_P2.54mm_Vertical" H 10400 9250 50  0001 C CNN
+F 2 "Connector_PinHeader_2.54mm:PinHeader_1x03_P2.54mm_Vertical" H 10400 9250 50  0001 C CNN
 F 3 "~" H 10400 9250 50  0001 C CNN
 	1    10400 9250

Commit message: first placement pass is done
Parts:
- C233: footprint Capacitor_THT:CP_Radial_D10.0mm_P2.50mm -> Capacitor_THT:CP_Radial_D6.3mm_P2.50mm
Changed lines of the file:
@@
 F 0 "C233" V 12205 3850 50  0000 C CNN
 F 1 "22uF 16V" V 12114 3850 50  0000 C CNN
-F 2 "Capacitor_THT:CP_Radial_D10.0mm_P2.50mm" H 11988 3700 50  0001 C CNN
+F 2 "Capacitor_THT:CP_Radial_D6.3mm_P2.50mm" H 11988 3700 50  0001 C CNN
 F 3 "~" H 11950 3850 50  0001 C CNN
 	1    11950 3850

Commit message: Make caps footprint smaller
Parts:
- C200, C202, C204, C210, C211, C212, C213, C218, C219, C220, C221, C230, C231, C232, C234, C240, C241, C242, C244, C900, C901: footprint Capacitor_THT:C_Rect_L11.0mm_W2.8mm_P10.00mm_MKT -> Capacitor_THT:C_Rect_L11.5mm_W2.0mm_P10.00mm_MKT
Changed lines of the file:
@@
 F 0 "C200" V 2350 950 50  0000 C CNN
 F 1 "0.1uF" V 2650 950 50  0000 C CNN
-F 2 "Capacitor_THT:C_Rect_L11.0mm_W2.8mm_P10.00mm_MKT" H 2538 800 50  0001 C CNN
+F 2 "Capacitor_THT:C_Rect_L11.5mm_W2.0mm_P10.00mm_MKT" H 2538 800 50  0001 C CNN
 F 3 "~" H 2500 950 50  0001 C CNN
 	1    2500 950
@@
 F 0 "C210" H 3915 6046 50  0000 L CNN
 F 1 "0.047uF" H 3915 5955 50  0000 L CNN
-F 2 "Capacitor_THT:C_Rect_L11.0mm_W2.8mm_P10.00mm_MKT" H 3838 5850 50  0001 C CNN
+F 2 "Capacitor_THT:C_Rect_L11.5mm_W2.0mm_P10.00mm_MKT" H 3838 5850 50  0001 C CNN
 F 3 "~" H 3800 6000 50  0001 C CNN
 	1    3800 6000
@@
 F 0 "C211" H 4465 6046 50  0000 L CNN
 F 1 "0.047uF" H 4465 5955 50  0000 L CNN
-F 2 "Capacitor_THT:C_Rect_L11.0mm_W2.8mm_P10.00mm_MKT" H 4388 5850 50  0001 C CNN
+F 2 "Capacitor_THT:C_Rect_L11.5mm_W2.0mm_P10.00mm_MKT" H 4388 5850 50  0001 C CNN
 F 3 "~" H 4350 6000 50  0001 C CNN
 	1    4350 6000
@@
 F 0 "C212" H 5015 6046 50  0000 L CNN
 F 1 "0.047uF" H 5015 5955 50  0000 L CNN
-F 2 "Capacitor_THT:C_Rect_L11.0mm_W2.8mm_P10.00mm_MKT" H 4938 5850 50  0001 C CNN
+F 2 "Capacitor_THT:C_Rect_L11.5mm_W2.0mm_P10.00mm_MKT" H 4938 5850 50  0001 C CNN
 F 3 "~" H 4900 6000 50  0001 C CNN
 	1    4900 6000
@@
 F 0 "C213" H 5565 6046 50  0000 L CNN
 F 1 "0.047uF" H 5565 5955 50  0000 L CNN
-F 2 "Capacitor_THT:C_Rect_L11.0mm_W2.8mm_P10.00mm_MKT" H 5488 5850 50  0001 C CNN
+F 2 "Capacitor_THT:C_Rect_L11.5mm_W2.0mm_P10.00mm_MKT" H 5488 5850 50  0001 C CNN
 F 3 "~" H 5450 6000 50  0001 C CNN
 	1    5450 6000
@@
 F 0 "C218" V 6721 6750 50  0000 C CNN
 F 1 "0.047uF" V 6812 6750 50  0000 C CNN
-F 2 "Capacitor_THT:C_Rect_L11.0mm_W2.8mm_P10.00mm_MKT" H 6950 6750 50  0001 C CNN
+F 2 "Capacitor_THT:C_Rect_L11.5mm_W2.0mm_P10.00mm_MKT" H 6950 6750 50  0001 C CNN
 F 3 "~" H 6950 6750 50  0001 C CNN
 	1    6950 6750
@@
 F 0 "C202" H 3315 8646 50  0000 L CNN
 F 1 "0.1uF" H 3315 8555 50  0000 L CNN
-F 2 "Capacitor_THT:C_Rect_L11.0mm_W2.8mm_P10.00mm_MKT" H 3238 8450 50  0001 C CNN
+F 2 "Capacitor_THT:C_Rect_L11.5mm_W2.0mm_P10.00mm_MKT" H 3238 8450 50  0001 C CNN
 F 3 "~" H 3200 8600 50  0001 C CNN
 	1    3200 8600
@@
 F 0 "C220" H 10715 7346 50  0000 L CNN
 F 1 "0.22uF" H 10715 7255 50  0000 L CNN
-F 2 "Capacitor_THT:C_Rect_L11.0mm_W2.8mm_P10.00mm_MKT" H 10638 7150 50  0001 C CNN
+F 2 "Capacitor_THT:C_Rect_L11.5mm_W2.0mm_P10.00mm_MKT" H 10638 7150 50  0001 C CNN
 F 3 "~" H 10600 7300 50  0001 C CNN
 	1    10600 7300
@@
 F 0 "C221" H 10715 7846 50  0000 L CNN
 F 1 "0.22uF" H 10715 7755 50  0000 L CNN
-F 2 "Capacitor_THT:C_Rect_L11.0mm_W2.8mm_P10.00mm_MKT" H 10638 7650 50  0001 C CNN
+F 2 "Capacitor_THT:C_Rect_L11.5mm_W2.0mm_P10.00mm_MKT" H 10638 7650 50  0001 C CNN
 F 3 "~" H 10600 7800 50  0001 C CNN
 	1    10600 7800
@@
 F 0 "C240" H 6665 1396 50  0000 L CNN
 F 1 "0.1uF" H 6665 1305 50  0000 L CNN
-F 2 "Capacitor_THT:C_Rect_L11.0mm_W2.8mm_P10.00mm_MKT" H 6588 1200 50  0001 C CNN
+F 2 "Capacitor_THT:C_Rect_L11.5mm_W2.0mm_P10.00mm_MKT" H 6588 1200 50  0001 C CNN
 F 3 "~" H 6550 1350 50  0001 C CNN
 	1    6550 1350
@@
 F 0 "C241" H 8465 1196 50  0000 L CNN
 F 1 "6800pF" H 8465 1105 50  0000 L CNN
-F 2 "Capacitor_THT:C_Rect_L11.0mm_W2.8mm_P10.00mm_MKT" H 8388 1000 50  0001 C CNN
+F 2 "Capacitor_THT:C_Rect_L11.5mm_W2.0mm_P10.00mm_MKT" H 8388 1000 50  0001 C CNN
 F 3 "~" H 8350 1150 50  0001 C CNN
 	1    8350 1150
@@
 F 0 "C242" H 9915 1846 50  0000 L CNN
 F 1 "3900pF" H 9915 1755 50  0000 L CNN
-F 2 "Capacitor_THT:C_Rect_L11.0mm_W2.8mm_P10.00mm_MKT" H 9838 1650 50  0001 C CNN
+F 2 "Capacitor_THT:C_Rect_L11.5mm_W2.0mm_P10.00mm_MKT" H 9838 1650 50  0001 C CNN
 F 3 "~" H 9800 1800 50  0001 C CNN
 	1    9800 1800
@@
 F 0 "C244" H 13615 1996 50  0000 L CNN
 F 1 "0.1uF" H 13615 1905 50  0000 L CNN
-F 2 "Capacitor_THT:C_Rect_L11.0mm_W2.8mm_P10.00mm_MKT" H 13538 1800 50  0001 C CNN
+F 2 "Capacitor_THT:C_Rect_L11.5mm_W2.0mm_P10.00mm_MKT" H 13538 1800 50  0001 C CNN
 F 3 "~" H 13500 1950 50  0001 C CNN
 	1    13500 1950
@@
 F 0 "C230" H 6665 3546 50  0000 L CNN
 F 1 "0.1uF" H 6665 3455 50  0000 L CNN
-F 2 "Capacitor_THT:C_Rect_L11.0mm_W2.8mm_P10.00mm_MKT" H 6588 3350 50  0001 C CNN
+F 2 "Capacitor_THT:C_Rect_L11.5mm_W2.0mm_P10.00mm_MKT" H 6588 3350 50  0001 C CNN
 F 3 "~" H 6550 3500 50  0001 C CNN
 	1    6550 3500
@@
 F 0 "C231" H 8465 3346 50  0000 L CNN
 F 1 "6800pF" H 8465 3255 50  0000 L CNN
-F 2 "Capacitor_THT:C_Rect_L11.0mm_W2.8mm_P10.00mm_MKT" H 8388 3150 50  0001 C CNN
+F 2 "Capacitor_THT:C_Rect_L11.5mm_W2.0mm_P10.00mm_MKT" H 8388 3150 50  0001 C CNN
 F 3 "~" H 8350 3300 50  0001 C CNN
 	1    8350 3300
@@
 F 0 "C232" H 9915 3996 50  0000 L CNN
 F 1 "3900pF" H 9915 3905 50  0000 L CNN
-F 2 "Capacitor_THT:C_Rect_L11.0mm_W2.8mm_P10.00mm_MKT" H 9838 3800 50  0001 C CNN
+F 2 "Capacitor_THT:C_Rect_L11.5mm_W2.0mm_P10.00mm_MKT" H 9838 3800 50  0001 C CNN
 F 3 "~" H 9800 3950 50  0001 C CNN
 	1    9800 3950
@@
 F 0 "C234" H 13615 4146 50  0000 L CNN
 F 1 "0.1uF" H 13615 4055 50  0000 L CNN
-F 2 "Capacitor_THT:C_Rect_L11.0mm_W2.8mm_P10.00mm_MKT" H 13538 3950 50  0001 C CNN
+F 2 "Capacitor_THT:C_Rect_L11.5mm_W2.0mm_P10.00mm_MKT" H 13538 3950 50  0001 C CNN
 F 3 "~" H 13500 4100 50  0001 C CNN
 	1    13500 4100
@@
 F 0 "C204" H 7865 5946 50  0000 L CNN
 F 1 "0.01uF" H 7865 5855 50  0000 L CNN
-F 2 "Capacitor_THT:C_Rect_L11.0mm_W2.8mm_P10.00mm_MKT" H 7788 5750 50  0001 C CNN
+F 2 "Capacitor_THT:C_Rect_L11.5mm_W2.0mm_P10.00mm_MKT" H 7788 5750 50  0001 C CNN
 F 3 "~" H 7750 5900 50  0001 C CNN
 	1    7750 5900
@@
 F 0 "C219" H 14015 8996 50  0000 L CNN
 F 1 "0.22uF" H 14015 8905 50  0000 L CNN
-F 2 "Capacitor_THT:C_Rect_L11.0mm_W2.8mm_P10.00mm_MKT" H 13938 8800 50  0001 C CNN
+F 2 "Capacitor_THT:C_Rect_L11.5mm_W2.0mm_P10.00mm_MKT" H 13938 8800 50  0001 C CNN
 F 3 "~" H 13900 8950 50  0001 C CNN
 	1    13900 8950
@@
 F 0 "C900" H 12965 7346 50  0000 L CNN
 F 1 "0.1uF" H 12965 7255 50  0000 L CNN
-F 2 "Capacitor_THT:C_Rect_L11.0mm_W2.8mm_P10.00mm_MKT" H 12888 7150 50  0001 C CNN
+F 2 "Capacitor_THT:C_Rect_L11.5mm_W2.0mm_P10.00mm_MKT" H 12888 7150 50  0001 C CNN
 F 3 "~" H 12850 7300 50  0001 C CNN
 	1    12850 7300
@@
 F 0 "C901" H 12965 7846 50  0000 L CNN
 F 1 "0.1uF" H 12965 7755 50  0000 L CNN
-F 2 "Capacitor_THT:C_Rect_L11.0mm_W2.8mm_P10.00mm_MKT" H 12888 7650 50  0001 C CNN
+F 2 "Capacitor_THT:C_Rect_L11.5mm_W2.0mm_P10.00mm_MKT" H 12888 7650 50  0001 C CNN
 F 3 "~" H 12850 7800 50  0001 C CNN
 	1    12850 7800

Commit message: All components have been realigned; plus small sizes changes
Parts:
- F1: footprint Fuse:Fuse_Littelfuse-LVR100 -> Capacitor_THT:C_Rect_L11.5mm_W2.0mm_P10.00mm_MKT
Changed lines of the file:
@@
 F 0 "F1" H 7710 7050 50  0000 L CNN
 F 1 "Fuse" H 7710 7005 50  0001 L CNN
-F 2 "Fuse:Fuse_Littelfuse-LVR100" V 7580 7050 50  0001 C CNN
+F 2 "Capacitor_THT:C_Rect_L11.5mm_W2.0mm_P10.00mm_MKT" V 7580 7050 50  0001 C CNN
 F 3 "~" H 7650 7050 50  0001 C CNN
 	1    7650 7050
