File: serial.sch (KiCad schematic (older format))
At the start: 53 parts, among them CN304 Conn_02x13_Odd_Even, CN305 DB25M, CN306 Conn_01x03_Male, Q300 2SC945, Q302 2N3906, U1 PST518B, U301 8520, U302 74LS32, U303 74F08, U304 1488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

Commit message: Make caps footprint smaller
Parts:
- C301, C304, C305, C306, C805, C815, C919: footprint Capacitor_THT:C_Rect_L11.0mm_W2.8mm_P10.00mm_MKT -> Capacitor_THT:C_Rect_L11.5mm_W2.0mm_P10.00mm_MKT
Changed lines of the file:
@@
 F 0 "C301" H 1715 4496 50  0000 L CNN
 F 1 "0.1uF" H 1715 4405 50  0000 L CNN
-F 2 "Capacitor_THT:C_Rect_L11.0mm_W2.8mm_P10.00mm_MKT" H 1638 4300 50  0001 C CNN
+F 2 "Capacitor_THT:C_Rect_L11.5mm_W2.0mm_P10.00mm_MKT" H 1638 4300 50  0001 C CNN
 F 3 "~" H 1600 4450 50  0001 C CNN
 	1    1600 4450
@@
 F 0 "C805" H 1165 2346 50  0000 L CNN
 F 1 "0.1uF" H 1165 2255 50  0000 L CNN
-F 2 "Capacitor_THT:C_Rect_L11.0mm_W2.8mm_P10.00mm_MKT" H 1088 2150 50  0001 C CNN
+F 2 "Capacitor_THT:C_Rect_L11.5mm_W2.0mm_P10.00mm_MKT" H 1088 2150 50  0001 C CNN
 F 3 "~" H 1050 2300 50  0001 C CNN
 	1    1050 2300
@@
 F 0 "C815" H 4165 2296 50  0000 L CNN
 F 1 "0.1uF" H 4165 2205 50  0000 L CNN
-F 2 "Capacitor_THT:C_Rect_L11.0mm_W2.8mm_P10.00mm_MKT" H 4088 2100 50  0001 C CNN
+F 2 "Capacitor_THT:C_Rect_L11.5mm_W2.0mm_P10.00mm_MKT" H 4088 2100 50  0001 C CNN
 F 3 "~" H 4050 2250 50  0001 C CNN
 	1    4050 2250
@@
 F 0 "C919" H 9265 2996 50  0000 L CNN
 F 1 "0.1uF" H 9265 2905 50  0000 L CNN
-F 2 "Capacitor_THT:C_Rect_L11.0mm_W2.8mm_P10.00mm_MKT" H 9188 2800 50  0001 C CNN
+F 2 "Capacitor_THT:C_Rect_L11.5mm_W2.0mm_P10.00mm_MKT" H 9188 2800 50  0001 C CNN
 F 3 "~" H 9150 2950 50  0001 C CNN
 	1    9150 2950
@@
 F 0 "C305" V 6198 7850 50  0000 C CNN
 F 1 "0.01uF" V 6289 7850 50  0000 C CNN
-F 2 "Capacitor_THT:C_Rect_L11.0mm_W2.8mm_P10.00mm_MKT" H 6488 7700 50  0001 C CNN
+F 2 "Capacitor_THT:C_Rect_L11.5mm_W2.0mm_P10.00mm_MKT" H 6488 7700 50  0001 C CNN
 F 3 "~" H 6450 7850 50  0001 C CNN
 	1    6450 7850
@@
 F 0 "C304" H 13965 8396 50  0000 L CNN
 F 1 "100pF" H 13965 8305 50  0000 L CNN
-F 2 "Capacitor_THT:C_Rect_L11.0mm_W2.8mm_P10.00mm_MKT" H 13888 8200 50  0001 C CNN
+F 2 "Capacitor_THT:C_Rect_L11.5mm_W2.0mm_P10.00mm_MKT" H 13888 8200 50  0001 C CNN
 F 3 "~" H 13850 8350 50  0001 C CNN
 	1    13850 8350
@@
 F 0 "C306" V 13248 5450 50  0000 C CNN
 F 1 "100pF" V 13339 5450 50  0000 C CNN
-F 2 "Capacitor_THT:C_Rect_L11.0mm_W2.8mm_P10.00mm_MKT" H 13538 5300 50  0001 C CNN
+F 2 "Capacitor_THT:C_Rect_L11.5mm_W2.0mm_P10.00mm_MKT" H 13538 5300 50  0001 C CNN
 F 3 "~" H 13500 5450 50  0001 C CNN
 	1    13500 5450

Commit message: All components have been realigned; plus small sizes changes
Parts:
- F2: footprint Fuse:Fuse_Littelfuse-LVR100 -> Capacitor_THT:C_Rect_L11.5mm_W2.0mm_P10.00mm_MKT
Changed lines of the file:
@@
 F 0 "F2" H 14910 8900 50  0000 L CNN
 F 1 "Fuse" H 14910 8855 50  0001 L CNN
-F 2 "Fuse:Fuse_Littelfuse-LVR100" V 14780 8900 50  0001 C CNN
+F 2 "Capacitor_THT:C_Rect_L11.5mm_W2.0mm_P10.00mm_MKT" V 14780 8900 50  0001 C CNN
 F 3 "~" H 14850 8900 50  0001 C CNN
 	1    14850 8900
