File: serial.sch (KiCad schematic (older format))
At the start: 53 parts, among them CN304 Conn_02x13_Odd_Even, CN305 DB25M, CN306 Conn_01x03_Male, Q300 2SC945, Q302 2N3906, U1 PST518B, U301 8520, U302 74LS32, U303 74F08, U304 1488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

Commit message: Makes the DRC happy
Parts:
- EMI325, EMI326, EMI327, EMI328, EMI329, EMI330, EMI331, EMI332, EMI333, EMI334: footprint Connector_PinSocket_2.54mm:PinSocket_1x03_P2.54mm_Vertical -> d_amiga:EMI_FILTER
Changed lines of the file:
@@
 F 0 "EMI326" H 11600 5663 50  0000 C CNN
 F 1 "C_Feedthrough" H 11600 5664 50  0001 C CNN
-F 2 "Connector_PinSocket_2.54mm:PinSocket_1x03_P2.54mm_Vertical" V 11600 5450 50  0001 C CNN
+F 2 "d_amiga:EMI_FILTER" V 11600 5450 50  0001 C CNN
 F 3 "~" V 11600 5450 50  0001 C CNN
 	1    11600 5450
@@
 F 0 "EMI327" H 11600 6063 50  0000 C CNN
 F 1 "C_Feedthrough" H 11600 6064 50  0001 C CNN
-F 2 "Connector_PinSocket_2.54mm:PinSocket_1x03_P2.54mm_Vertical" V 11600 5850 50  0001 C CNN
+F 2 "d_amiga:EMI_FILTER" V 11600 5850 50  0001 C CNN
 F 3 "~" V 11600 5850 50  0001 C CNN
 	1    11600 5850
@@
 F 0 "EMI330" H 11600 7513 50  0000 C CNN
 F 1 "C_Feedthrough" H 11600 7514 50  0001 C CNN
-F 2 "Connector_PinSocket_2.54mm:PinSocket_1x03_P2.54mm_Vertical" V 11600 7300 50  0001 C CNN
+F 2 "d_amiga:EMI_FILTER" V 11600 7300 50  0001 C CNN
 F 3 "~" V 11600 7300 50  0001 C CNN
 	1    11600 7300
@@
 F 0 "EMI334" H 15200 8613 50  0000 C CNN
 F 1 "C_Feedthrough" H 15200 8614 50  0001 C CNN
-F 2 "Connector_PinSocket_2.54mm:PinSocket_1x03_P2.54mm_Vertical" V 15200 8400 50  0001 C CNN
+F 2 "d_amiga:EMI_FILTER" V 15200 8400 50  0001 C CNN
 F 3 "~" V 15200 8400 50  0001 C CNN
 	1    15200 8400
@@
 F 0 "EMI333" H 12950 8713 50  0000 C CNN
 F 1 "C_Feedthrough" H 12950 8714 50  0001 C CNN
-F 2 "Connector_PinSocket_2.54mm:PinSocket_1x03_P2.54mm_Vertical" V 12950 8500 50  0001 C CNN
+F 2 "d_amiga:EMI_FILTER" V 12950 8500 50  0001 C CNN
 F 3 "~" V 12950 8500 50  0001 C CNN
 	1    12950 8500
@@
 F 0 "EMI332" H 14600 8613 50  0000 C CNN
 F 1 "C_Feedthrough" H 14600 8614 50  0001 C CNN
-F 2 "Connector_PinSocket_2.54mm:PinSocket_1x03_P2.54mm_Vertical" V 14600 8400 50  0001 C CNN
+F 2 "d_amiga:EMI_FILTER" V 14600 8400 50  0001 C CNN
 F 3 "~" V 14600 8400 50  0001 C CNN
 	1    14600 8400
@@
 F 0 "EMI331" H 11600 8063 50  0000 C CNN
 F 1 "C_Feedthrough" H 11600 8064 50  0001 C CNN
-F 2 "Connector_PinSocket_2.54mm:PinSocket_1x03_P2.54mm_Vertical" V 11600 7850 50  0001 C CNN
+F 2 "d_amiga:EMI_FILTER" V 11600 7850 50  0001 C CNN
 F 3 "~" V 11600 7850 50  0001 C CNN
 	1    11600 7850
@@
 F 0 "EMI325" H 11600 5263 50  0000 C CNN
 F 1 "C_Feedthrough" H 11600 5264 50  0001 C CNN
-F 2 "Connector_PinSocket_2.54mm:PinSocket_1x03_P2.54mm_Vertical" V 11600 5050 50  0001 C CNN
+F 2 "d_amiga:EMI_FILTER" V 11600 5050 50  0001 C CNN
 F 3 "~" V 11600 5050 50  0001 C CNN
 	1    11600 5050
@@
 F 0 "EMI329" H 11600 7113 50  0000 C CNN
 F 1 "C_Feedthrough" H 11600 7114 50  0001 C CNN
-F 2 "Connector_PinSocket_2.54mm:PinSocket_1x03_P2.54mm_Vertical" V 11600 6900 50  0001 C CNN
+F 2 "d_amiga:EMI_FILTER" V 11600 6900 50  0001 C CNN
 F 3 "~" V 11600 6900 50  0001 C CNN
 	1    11600 6900
@@
 F 0 "EMI328" H 11600 6713 50  0000 C CNN
 F 1 "C_Feedthrough" H 11600 6714 50  0001 C CNN
-F 2 "Connector_PinSocket_2.54mm:PinSocket_1x03_P2.54mm_Vertical" V 11600 6500 50  0001 C CNN
+F 2 "d_amiga:EMI_FILTER" V 11600 6500 50  0001 C CNN
 F 3 "~" V 11600 6500 50  0001 C CNN
 	1    11600 6500

Commit message: Switch footprints for suitable modern replacements
Parts:
- C301, C304, C306, C805, C815, C919: footprint Capacitor_THT:C_Rect_L11.5mm_W2.0mm_P10.00mm_MKT -> Capacitor_THT:C_Rect_L11.5mm_W2.6mm_P10.00mm_MKT
- C310, C311, C312, C313, C314, C315, C316, C320, C321: footprint Capacitor_THT:C_Rect_L7.0mm_W2.0mm_P5.00mm -> Capacitor_THT:C_Rect_L7.0mm_W4.5mm_P5.00mm
Changed lines of the file:
@@
 F 0 "C301" H 1715 4496 50  0000 L CNN
 F 1 "0.1uF" H 1715 4405 50  0000 L CNN
-F 2 "Capacitor_THT:C_Rect_L11.5mm_W2.0mm_P10.00mm_MKT" H 1638 4300 50  0001 C CNN
+F 2 "Capacitor_THT:C_Rect_L11.5mm_W2.6mm_P10.00mm_MKT" H 1638 4300 50  0001 C CNN
 F 3 "~" H 1600 4450 50  0001 C CNN
 	1    1600 4450
@@
 F 0 "C805" H 1165 2346 50  0000 L CNN
 F 1 "0.1uF" H 1165 2255 50  0000 L CNN
-F 2 "Capacitor_THT:C_Rect_L11.5mm_W2.0mm_P10.00mm_MKT" H 1088 2150 50  0001 C CNN
+F 2 "Capacitor_THT:C_Rect_L11.5mm_W2.6mm_P10.00mm_MKT" H 1088 2150 50  0001 C CNN
 F 3 "~" H 1050 2300 50  0001 C CNN
 	1    1050 2300
@@
 F 0 "C815" H 4165 2296 50  0000 L CNN
 F 1 "0.1uF" H 4165 2205 50  0000 L CNN
-F 2 "Capacitor_THT:C_Rect_L11.5mm_W2.0mm_P10.00mm_MKT" H 4088 2100 50  0001 C CNN
+F 2 "Capacitor_THT:C_Rect_L11.5mm_W2.6mm_P10.00mm_MKT" H 4088 2100 50  0001 C CNN
 F 3 "~" H 4050 2250 50  0001 C CNN
 	1    4050 2250
@@
 F 0 "C320" H 10115 4196 50  0000 L CNN
 F 1 "470pF" H 10115 4105 50  0000 L CNN
-F 2 "Capacitor_THT:C_Rect_L7.0mm_W2.0mm_P5.00mm" H 10038 4000 50  0001 C CNN
+F 2 "Capacitor_THT:C_Rect_L7.0mm_W4.5mm_P5.00mm" H 10038 4000 50  0001 C CNN
 F 3 "~" H 10000 4150 50  0001 C CNN
 	1    10000 4150
@@
 F 0 "C321" V 11348 3350 50  0000 C CNN
 F 1 "470pF" V 11439 3350 50  0000 C CNN
-F 2 "Capacitor_THT:C_Rect_L7.0mm_W2.0mm_P5.00mm" H 11638 3200 50  0001 C CNN
+F 2 "Capacitor_THT:C_Rect_L7.0mm_W4.5mm_P5.00mm" H 11638 3200 50  0001 C CNN
 F 3 "~" H 11600 3350 50  0001 C CNN
 	1    11600 3350
@@
 F 0 "C919" H 9265 2996 50  0000 L CNN
 F 1 "0.1uF" H 9265 2905 50  0000 L CNN
-F 2 "Capacitor_THT:C_Rect_L11.5mm_W2.0mm_P10.00mm_MKT" H 9188 2800 50  0001 C CNN
+F 2 "Capacitor_THT:C_Rect_L11.5mm_W2.6mm_P10.00mm_MKT" H 9188 2800 50  0001 C CNN
 F 3 "~" H 9150 2950 50  0001 C CNN
 	1    9150 2950
@@
 F 0 "C314" H 7565 4346 50  0000 L CNN
 F 1 "1000pF" H 7565 4255 50  0000 L CNN
-F 2 "Capacitor_THT:C_Rect_L7.0mm_W2.0mm_P5.00mm" H 7488 4150 50  0001 C CNN
+F 2 "Capacitor_THT:C_Rect_L7.0mm_W4.5mm_P5.00mm" H 7488 4150 50  0001 C CNN
 F 3 "~" H 7450 4300 50  0001 C CNN
 	1    7450 4300
@@
 F 0 "C315" H 8015 4646 50  0000 L CNN
 F 1 "1000pF" H 8015 4555 50  0000 L CNN
-F 2 "Capacitor_THT:C_Rect_L7.0mm_W2.0mm_P5.00mm" H 7938 4450 50  0001 C CNN
+F 2 "Capacitor_THT:C_Rect_L7.0mm_W4.5mm_P5.00mm" H 7938 4450 50  0001 C CNN
 F 3 "~" H 7900 4600 50  0001 C CNN
 	1    7900 4600
@@
 F 0 "C316" H 8415 4346 50  0000 L CNN
 F 1 "1000pF" H 8415 4255 50  0000 L CNN
-F 2 "Capacitor_THT:C_Rect_L7.0mm_W2.0mm_P5.00mm" H 8338 4150 50  0001 C CNN
+F 2 "Capacitor_THT:C_Rect_L7.0mm_W4.5mm_P5.00mm" H 8338 4150 50  0001 C CNN
 F 3 "~" H 8300 4300 50  0001 C CNN
 	1    8300 4300
@@
 F 0 "C310" H 7615 8146 50  0000 L CNN
 F 1 "1000pF" H 7615 8055 50  0000 L CNN
-F 2 "Capacitor_THT:C_Rect_L7.0mm_W2.0mm_P5.00mm" H 7538 7950 50  0001 C CNN
+F 2 "Capacitor_THT:C_Rect_L7.0mm_W4.5mm_P5.00mm" H 7538 7950 50  0001 C CNN
 F 3 "~" H 7500 8100 50  0001 C CNN
 	1    7500 8100
@@
 F 0 "C311" H 8115 8146 50  0000 L CNN
 F 1 "1000pF" H 8115 8055 50  0000 L CNN
-F 2 "Capacitor_THT:C_Rect_L7.0mm_W2.0mm_P5.00mm" H 8038 7950 50  0001 C CNN
+F 2 "Capacitor_THT:C_Rect_L7.0mm_W4.5mm_P5.00mm" H 8038 7950 50  0001 C CNN
 F 3 "~" H 8000 8100 50  0001 C CNN
 	1    8000 8100
@@
 F 0 "C312" H 8615 8146 50  0000 L CNN
 F 1 "1000pF" H 8615 8055 50  0000 L CNN
-F 2 "Capacitor_THT:C_Rect_L7.0mm_W2.0mm_P5.00mm" H 8538 7950 50  0001 C CNN
+F 2 "Capacitor_THT:C_Rect_L7.0mm_W4.5mm_P5.00mm" H 8538 7950 50  0001 C CNN
 F 3 "~" H 8500 8100 50  0001 C CNN
 	1    8500 8100
@@
 F 0 "C313" H 9115 8146 50  0000 L CNN
 F 1 "1000pF" H 9115 8055 50  0000 L CNN
-F 2 "Capacitor_THT:C_Rect_L7.0mm_W2.0mm_P5.00mm" H 9038 7950 50  0001 C CNN
+F 2 "Capacitor_THT:C_Rect_L7.0mm_W4.5mm_P5.00mm" H 9038 7950 50  0001 C CNN
 F 3 "~" H 9000 8100 50  0001 C CNN
 	1    9000 8100
@@
 F 0 "C304" H 13965 8396 50  0000 L CNN
 F 1 "100pF" H 13965 8305 50  0000 L CNN
-F 2 "Capacitor_THT:C_Rect_L11.5mm_W2.0mm_P10.00mm_MKT" H 13888 8200 50  0001 C CNN
+F 2 "Capacitor_THT:C_Rect_L11.5mm_W2.6mm_P10.00mm_MKT" H 13888 8200 50  0001 C CNN
 F 3 "~" H 13850 8350 50  0001 C CNN
 	1    13850 8350
@@
 F 0 "C306" V 13248 5450 50  0000 C CNN
 F 1 "100pF" V 13339 5450 50  0000 C CNN
-F 2 "Capacitor_THT:C_Rect_L11.5mm_W2.0mm_P10.00mm_MKT" H 13538 5300 50  0001 C CNN
+F 2 "Capacitor_THT:C_Rect_L11.5mm_W2.6mm_P10.00mm_MKT" H 13538 5300 50  0001 C CNN
 F 3 "~" H 13500 5450 50  0001 C CNN
 	1    13500 5450

Commit message: Some footprints updates; Add all Mouser references
Parts:
- C301, C805, C815, C919: RefOrder (none) -> 581-SA105C104KARC
- C304, C306: RefOrder (none) -> 80-C410C101K5G
- C305: RefOrder (none) -> 581-SA105C103K
- C310, C311, C312, C313, C314, C315, C316: RefOrder (none) -> 810-FG28C0G1H102JNT6
- C317, C318, C813, C814: RefOrder (none) -> 667-ECA-1CM220B
- C320, C321: RefOrder (none) -> 810-FG28C0G1H471JNT0
- D300: RefOrder (none) -> 78-1N4148
- EMI325, EMI326, EMI327, EMI328, EMI329, EMI330, EMI331, EMI332, EMI333, EMI334: value C_Feedthrough -> 330pF (Type F 331); RefOrder (none) -> 81-DSS1NB32A331Q91A
- F2: value Fuse -> 4A; RefOrder (none) -> 576-0251004.MRT1L
- Q302: RefOrder (none) -> 833-2N3906-AP
- R302: RefOrder (none) -> 603-CFR-25JR-521K
- R305, R306, R802: RefOrder (none) -> 603-CFR-25JR-5210K
- R307: RefOrder (none) -> 603-CFR-25JT-52-68R
- R308: RefOrder (none) -> 603-CFR-25JR-52-200R
- R805: RefOrder (none) -> 603-CFR-25JR-5247K
- R902: RefOrder (none) -> 603-CFR-25JT-52-4K7
- RP802: value 1k -> 1k (isolated, pack); RefOrder (none) -> 269-1.0K-RC
- U302: RefOrder (none) -> 595-SN74LS32N
- U303: RefOrder (none) -> 595-SN74F08N
- U304: RefOrder (none) -> 595-MC1488N
- U305: RefOrder (none) -> 595-MC1489N
- U805: RefOrder (none) -> 595-LM339N

Commit message: Got the components, reduce some footprints
Parts:
- C305: footprint Capacitor_THT:C_Rect_L11.5mm_W2.0mm_P10.00mm_MKT -> Capacitor_THT:C_Rect_L11.5mm_W2.6mm_P10.00mm_MKT
- C310, C311, C312, C313, C314, C315, C316, C320, C321: footprint Capacitor_THT:C_Rect_L7.0mm_W4.5mm_P5.00mm -> Capacitor_THT:C_Rect_L7.0mm_W2.0mm_P5.00mm
- C317, C318, C813, C814: footprint Capacitor_THT:CP_Radial_D8.0mm_P5.00mm -> Capacitor_THT:CP_Radial_Tantal_D5.0mm_P5.00mm
Changed lines of the file:
@@
 F 0 "C813" H 2718 1746 50  0000 L CNN
 F 1 "22uF 16V" H 2718 1655 50  0000 L CNN
-F 2 "Capacitor_THT:CP_Radial_D8.0mm_P5.00mm" H 2638 1550 50  0001 C CNN
+F 2 "Capacitor_THT:CP_Radial_Tantal_D5.0mm_P5.00mm" H 2638 1550 50  0001 C CNN
 F 3 "~" H 2600 1700 50  0001 C CNN
 F 4 "667-ECA-1CM220B" H 2600 1700 50  0001 C CNN "RefOrder"
@@
 F 0 "C814" H 4368 1746 50  0000 L CNN
 F 1 "22uF 16V" H 4368 1655 50  0000 L CNN
-F 2 "Capacitor_THT:CP_Radial_D8.0mm_P5.00mm" H 4288 1550 50  0001 C CNN
+F 2 "Capacitor_THT:CP_Radial_Tantal_D5.0mm_P5.00mm" H 4288 1550 50  0001 C CNN
 F 3 "~" H 4250 1700 50  0001 C CNN
 F 4 "667-ECA-1CM220B" H 4250 1700 50  0001 C CNN "RefOrder"
@@
 F 0 "C320" H 10115 4196 50  0000 L CNN
 F 1 "470pF" H 10115 4105 50  0000 L CNN
-F 2 "Capacitor_THT:C_Rect_L7.0mm_W4.5mm_P5.00mm" H 10038 4000 50  0001 C CNN
+F 2 "Capacitor_THT:C_Rect_L7.0mm_W2.0mm_P5.00mm" H 10038 4000 50  0001 C CNN
 F 3 "~" H 10000 4150 50  0001 C CNN
 F 4 "810-FG28C0G1H471JNT0" H 10000 4150 50  0001 C CNN "RefOrder"
@@
 F 0 "C321" V 11348 3350 50  0000 C CNN
 F 1 "470pF" V 11439 3350 50  0000 C CNN
-F 2 "Capacitor_THT:C_Rect_L7.0mm_W4.5mm_P5.00mm" H 11638 3200 50  0001 C CNN
+F 2 "Capacitor_THT:C_Rect_L7.0mm_W2.0mm_P5.00mm" H 11638 3200 50  0001 C CNN
 F 3 "~" H 11600 3350 50  0001 C CNN
 F 4 "810-FG28C0G1H471JNT0" H 11600 3350 50  0001 C CNN "RefOrder"
@@
 F 0 "C305" V 6198 7850 50  0000 C CNN
 F 1 "0.01uF" V 6289 7850 50  0000 C CNN
-F 2 "Capacitor_THT:C_Rect_L11.5mm_W2.0mm_P10.00mm_MKT" H 6488 7700 50  0001 C CNN
+F 2 "Capacitor_THT:C_Rect_L11.5mm_W2.6mm_P10.00mm_MKT" H 6488 7700 50  0001 C CNN
 F 3 "~" H 6450 7850 50  0001 C CNN
 F 4 "581-SA105C103K" H 6450 7850 50  0001 C CNN "RefOrder"
@@
 F 0 "C314" H 7565 4346 50  0000 L CNN
 F 1 "1000pF" H 7565 4255 50  0000 L CNN
-F 2 "Capacitor_THT:C_Rect_L7.0mm_W4.5mm_P5.00mm" H 7488 4150 50  0001 C CNN
+F 2 "Capacitor_THT:C_Rect_L7.0mm_W2.0mm_P5.00mm" H 7488 4150 50  0001 C CNN
 F 3 "~" H 7450 4300 50  0001 C CNN
 F 4 "810-FG28C0G1H102JNT6" H 7450 4300 50  0001 C CNN "RefOrder"
@@
 F 0 "C315" H 8015 4646 50  0000 L CNN
 F 1 "1000pF" H 8015 4555 50  0000 L CNN
-F 2 "Capacitor_THT:C_Rect_L7.0mm_W4.5mm_P5.00mm" H 7938 4450 50  0001 C CNN
+F 2 "Capacitor_THT:C_Rect_L7.0mm_W2.0mm_P5.00mm" H 7938 4450 50  0001 C CNN
 F 3 "~" H 7900 4600 50  0001 C CNN
 F 4 "810-FG28C0G1H102JNT6" H 7900 4600 50  0001 C CNN "RefOrder"
@@
 F 0 "C316" H 8415 4346 50  0000 L CNN
 F 1 "1000pF" H 8415 4255 50  0000 L CNN
-F 2 "Capacitor_THT:C_Rect_L7.0mm_W4.5mm_P5.00mm" H 8338 4150 50  0001 C CNN
+F 2 "Capacitor_THT:C_Rect_L7.0mm_W2.0mm_P5.00mm" H 8338 4150 50  0001 C CNN
 F 3 "~" H 8300 4300 50  0001 C CNN
 F 4 "810-FG28C0G1H102JNT6" H 8300 4300 50  0001 C CNN "RefOrder"
@@
 F 0 "C310" H 7615 8146 50  0000 L CNN
 F 1 "1000pF" H 7615 8055 50  0000 L CNN
-F 2 "Capacitor_THT:C_Rect_L7.0mm_W4.5mm_P5.00mm" H 7538 7950 50  0001 C CNN
+F 2 "Capacitor_THT:C_Rect_L7.0mm_W2.0mm_P5.00mm" H 7538 7950 50  0001 C CNN
 F 3 "~" H 7500 8100 50  0001 C CNN
 F 4 "810-FG28C0G1H102JNT6" H 7500 8100 50  0001 C CNN "RefOrder"
@@
 F 0 "C311" H 8115 8146 50  0000 L CNN
 F 1 "1000pF" H 8115 8055 50  0000 L CNN
-F 2 "Capacitor_THT:C_Rect_L7.0mm_W4.5mm_P5.00mm" H 8038 7950 50  0001 C CNN
+F 2 "Capacitor_THT:C_Rect_L7.0mm_W2.0mm_P5.00mm" H 8038 7950 50  0001 C CNN
 F 3 "~" H 8000 8100 50  0001 C CNN
 F 4 "810-FG28C0G1H102JNT6" H 8000 8100 50  0001 C CNN "RefOrder"
@@
 F 0 "C312" H 8615 8146 50  0000 L CNN
 F 1 "1000pF" H 8615 8055 50  0000 L CNN
-F 2 "Capacitor_THT:C_Rect_L7.0mm_W4.5mm_P5.00mm" H 8538 7950 50  0001 C CNN
+F 2 "Capacitor_THT:C_Rect_L7.0mm_W2.0mm_P5.00mm" H 8538 7950 50  0001 C CNN
 F 3 "~" H 8500 8100 50  0001 C CNN
 F 4 "810-FG28C0G1H102JNT6" H 8500 8100 50  0001 C CNN "RefOrder"
@@
 F 0 "C313" H 9115 8146 50  0000 L CNN
 F 1 "1000pF" H 9115 8055 50  0000 L CNN
-F 2 "Capacitor_THT:C_Rect_L7.0mm_W4.5mm_P5.00mm" H 9038 7950 50  0001 C CNN
+F 2 "Capacitor_THT:C_Rect_L7.0mm_W2.0mm_P5.00mm" H 9038 7950 50  0001 C CNN
 F 3 "~" H 9000 8100 50  0001 C CNN
 F 4 "810-FG28C0G1H102JNT6" H 9000 8100 50  0001 C CNN "RefOrder"
@@
 F 0 "C318" H 12668 8946 50  0000 L CNN
 F 1 "22uF 16V" H 12668 8855 50  0000 L CNN
-F 2 "Capacitor_THT:CP_Radial_D8.0mm_P5.00mm" H 12588 8750 50  0001 C CNN
+F 2 "Capacitor_THT:CP_Radial_Tantal_D5.0mm_P5.00mm" H 12588 8750 50  0001 C CNN
 F 3 "~" H 12550 8900 50  0001 C CNN
 F 4 "667-ECA-1CM220B" H 12550 8900 50  0001 C CNN "RefOrder"
@@
 F 0 "C317" H 13268 4996 50  0000 L CNN
 F 1 "22uF 16V" H 13268 4905 50  0000 L CNN
-F 2 "Capacitor_THT:CP_Radial_D8.0mm_P5.00mm" H 13188 4800 50  0001 C CNN
+F 2 "Capacitor_THT:CP_Radial_Tantal_D5.0mm_P5.00mm" H 13188 4800 50  0001 C CNN
 F 3 "~" H 13150 4950 50  0001 C CNN
 F 4 "667-ECA-1CM220B" H 13150 4950 50  0001 C CNN "RefOrder"
