File: parallel.sch (KiCad schematic (older format))
At the start: 75 parts, among them CN300 KEYBOARD, CN301 DB25F, CN302 DB23F, CN303 Conn_02x17_Odd_Even, J3 ACCEL, J300 Conn_01x03_Male, J301 DF1:, Q301 2N3904, U102 GARY5719, U108 74LS74A, U203 74LS38, U300 CIA8520, U302 74LS32, U303 74F08, U607 74LS08, U900 74F00

Commit message: Makes the DRC happy
Parts:
- EMI300, EMI301, EMI302, EMI303, EMI304, EMI305, EMI306, EMI307, EMI308, EMI309, EMI310, EMI311, EMI312, EMI313, EMI314, EMI315, EMI316, EMI317, EMI318, EMI319, EMI320, EMI321, EMI322, EMI323, EMI324, EMI335, EMI336, EMI337, EMI338, EMI339, EMI340, EMI341: footprint Connector_PinSocket_2.54mm:PinSocket_1x03_P2.54mm_Vertical -> d_amiga:EMI_FILTER
Changed lines of the file:
@@
 F 0 "EMI301" H 7450 4800 50  0000 C CNN
 F 1 "C_Feedthrough" H 7300 4814 50  0001 C CNN
-F 2 "Connector_PinSocket_2.54mm:PinSocket_1x03_P2.54mm_Vertical" V 7300 4600 50  0001 C CNN
+F 2 "d_amiga:EMI_FILTER" V 7300 4600 50  0001 C CNN
 F 3 "~" V 7300 4600 50  0001 C CNN
 	1    7300 4600
@@
 F 0 "EMI310" H 8500 4563 50  0000 C CNN
 F 1 "C_Feedthrough" H 8500 4564 50  0001 C CNN
-F 2 "Connector_PinSocket_2.54mm:PinSocket_1x03_P2.54mm_Vertical" V 8500 4350 50  0001 C CNN
+F 2 "d_amiga:EMI_FILTER" V 8500 4350 50  0001 C CNN
 F 3 "~" V 8500 4350 50  0001 C CNN
 	1    8500 4350
@@
 F 0 "EMI300" H 8500 4163 50  0000 C CNN
 F 1 "C_Feedthrough" H 8500 4164 50  0001 C CNN
-F 2 "Connector_PinSocket_2.54mm:PinSocket_1x03_P2.54mm_Vertical" V 8500 3950 50  0001 C CNN
+F 2 "d_amiga:EMI_FILTER" V 8500 3950 50  0001 C CNN
 F 3 "~" V 8500 3950 50  0001 C CNN
 	1    8500 3950
@@
 F 0 "EMI303" H 7450 5100 50  0000 C CNN
 F 1 "C_Feedthrough" H 7300 5114 50  0001 C CNN
-F 2 "Connector_PinSocket_2.54mm:PinSocket_1x03_P2.54mm_Vertical" V 7300 4900 50  0001 C CNN
+F 2 "d_amiga:EMI_FILTER" V 7300 4900 50  0001 C CNN
 F 3 "~" V 7300 4900 50  0001 C CNN
 	1    7300 4900
@@
 F 0 "EMI305" H 7450 5400 50  0000 C CNN
 F 1 "C_Feedthrough" H 7300 5414 50  0001 C CNN
-F 2 "Connector_PinSocket_2.54mm:PinSocket_1x03_P2.54mm_Vertical" V 7300 5200 50  0001 C CNN
+F 2 "d_amiga:EMI_FILTER" V 7300 5200 50  0001 C CNN
 F 3 "~" V 7300 5200 50  0001 C CNN
 	1    7300 5200
@@
 F 0 "EMI308" H 7950 5850 50  0000 C CNN
 F 1 "C_Feedthrough" H 7800 5864 50  0001 C CNN
-F 2 "Connector_PinSocket_2.54mm:PinSocket_1x03_P2.54mm_Vertical" V 7800 5650 50  0001 C CNN
+F 2 "d_amiga:EMI_FILTER" V 7800 5650 50  0001 C CNN
 F 3 "~" V 7800 5650 50  0001 C CNN
 	1    7800 5650
@@
 F 0 "EMI335" H 7950 6150 50  0000 C CNN
 F 1 "C_Feedthrough" H 7800 6164 50  0001 C CNN
-F 2 "Connector_PinSocket_2.54mm:PinSocket_1x03_P2.54mm_Vertical" V 7800 5950 50  0001 C CNN
+F 2 "d_amiga:EMI_FILTER" V 7800 5950 50  0001 C CNN
 F 3 "~" V 7800 5950 50  0001 C CNN
 	1    7800 5950
@@
 F 0 "EMI337" H 7950 6450 50  0000 C CNN
 F 1 "C_Feedthrough" H 7800 6464 50  0001 C CNN
-F 2 "Connector_PinSocket_2.54mm:PinSocket_1x03_P2.54mm_Vertical" V 7800 6250 50  0001 C CNN
+F 2 "d_amiga:EMI_FILTER" V 7800 6250 50  0001 C CNN
 F 3 "~" V 7800 6250 50  0001 C CNN
 	1    7800 6250
@@
 F 0 "EMI307" H 7450 5700 50  0000 C CNN
 F 1 "C_Feedthrough" H 7300 5714 50  0001 C CNN
-F 2 "Connector_PinSocket_2.54mm:PinSocket_1x03_P2.54mm_Vertical" V 7300 5500 50  0001 C CNN
+F 2 "d_amiga:EMI_FILTER" V 7300 5500 50  0001 C CNN
 F 3 "~" V 7300 5500 50  0001 C CNN
 	1    7300 5500
@@
 F 0 "EMI302" H 7950 4950 50  0000 C CNN
 F 1 "C_Feedthrough" H 7800 4964 50  0001 C CNN
-F 2 "Connector_PinSocket_2.54mm:PinSocket_1x03_P2.54mm_Vertical" V 7800 4750 50  0001 C CNN
+F 2 "d_amiga:EMI_FILTER" V 7800 4750 50  0001 C CNN
 F 3 "~" V 7800 4750 50  0001 C CNN
 	1    7800 4750
@@
 F 0 "EMI304" H 7950 5250 50  0000 C CNN
 F 1 "C_Feedthrough" H 7800 5264 50  0001 C CNN
-F 2 "Connector_PinSocket_2.54mm:PinSocket_1x03_P2.54mm_Vertical" V 7800 5050 50  0001 C CNN
+F 2 "d_amiga:EMI_FILTER" V 7800 5050 50  0001 C CNN
 F 3 "~" V 7800 5050 50  0001 C CNN
 	1    7800 5050
@@
 F 0 "EMI306" H 7950 5550 50  0000 C CNN
 F 1 "C_Feedthrough" H 7800 5564 50  0001 C CNN
-F 2 "Connector_PinSocket_2.54mm:PinSocket_1x03_P2.54mm_Vertical" V 7800 5350 50  0001 C CNN
+F 2 "d_amiga:EMI_FILTER" V 7800 5350 50  0001 C CNN
 F 3 "~" V 7800 5350 50  0001 C CNN
 	1    7800 5350
@@
 F 0 "EMI309" H 7450 6000 50  0000 C CNN
 F 1 "C_Feedthrough" H 7300 6014 50  0001 C CNN
-F 2 "Connector_PinSocket_2.54mm:PinSocket_1x03_P2.54mm_Vertical" V 7300 5800 50  0001 C CNN
+F 2 "d_amiga:EMI_FILTER" V 7300 5800 50  0001 C CNN
 F 3 "~" V 7300 5800 50  0001 C CNN
 	1    7300 5800
@@
 F 0 "EMI336" H 7450 6300 50  0000 C CNN
 F 1 "C_Feedthrough" H 7300 6314 50  0001 C CNN
-F 2 "Connector_PinSocket_2.54mm:PinSocket_1x03_P2.54mm_Vertical" V 7300 6100 50  0001 C CNN
+F 2 "d_amiga:EMI_FILTER" V 7300 6100 50  0001 C CNN
 F 3 "~" V 7300 6100 50  0001 C CNN
 	1    7300 6100
@@
 F 0 "EMI338" H 7450 6600 50  0000 C CNN
 F 1 "C_Feedthrough" H 7300 6614 50  0001 C CNN
-F 2 "Connector_PinSocket_2.54mm:PinSocket_1x03_P2.54mm_Vertical" V 7300 6400 50  0001 C CNN
+F 2 "d_amiga:EMI_FILTER" V 7300 6400 50  0001 C CNN
 F 3 "~" V 7300 6400 50  0001 C CNN
 	1    7300 6400
@@
 F 0 "EMI318" H 14100 800 50  0000 C CNN
 F 1 "C_Feedthrough" H 13900 964 50  0001 C CNN
-F 2 "Connector_PinSocket_2.54mm:PinSocket_1x03_P2.54mm_Vertical" V 13900 750 50  0001 C CNN
+F 2 "d_amiga:EMI_FILTER" V 13900 750 50  0001 C CNN
 F 3 "~" V 13900 750 50  0001 C CNN
 	1    13900 750
@@
 F 0 "EMI319" H 14100 1100 50  0000 C CNN
 F 1 "C_Feedthrough" H 13900 1264 50  0001 C CNN
-F 2 "Connector_PinSocket_2.54mm:PinSocket_1x03_P2.54mm_Vertical" V 13900 1050 50  0001 C CNN
+F 2 "d_amiga:EMI_FILTER" V 13900 1050 50  0001 C CNN
 F 3 "~" V 13900 1050 50  0001 C CNN
 	1    13900 1050
@@
 F 0 "EMI321" H 14100 1550 50  0000 C CNN
 F 1 "C_Feedthrough" H 13900 1714 50  0001 C CNN
-F 2 "Connector_PinSocket_2.54mm:PinSocket_1x03_P2.54mm_Vertical" V 13900 1500 50  0001 C CNN
+F 2 "d_amiga:EMI_FILTER" V 13900 1500 50  0001 C CNN
 F 3 "~" V 13900 1500 50  0001 C CNN
 	1    13900 1500
@@
 F 0 "EMI320" H 14100 1850 50  0000 C CNN
 F 1 "C_Feedthrough" H 13900 2014 50  0001 C CNN
-F 2 "Connector_PinSocket_2.54mm:PinSocket_1x03_P2.54mm_Vertical" V 13900 1800 50  0001 C CNN
+F 2 "d_amiga:EMI_FILTER" V 13900 1800 50  0001 C CNN
 F 3 "~" V 13900 1800 50  0001 C CNN
 	1    13900 1800
@@
 F 0 "EMI323" H 11800 2700 50  0000 C CNN
 F 1 "C_Feedthrough" H 11600 2864 50  0001 C CNN
-F 2 "Connector_PinSocket_2.54mm:PinSocket_1x03_P2.54mm_Vertical" V 11600 2650 50  0001 C CNN
+F 2 "d_amiga:EMI_FILTER" V 11600 2650 50  0001 C CNN
 F 3 "~" V 11600 2650 50  0001 C CNN
 	1    11600 2650
@@
 F 0 "EMI311" H 12000 3650 50  0000 C CNN
 F 1 "C_Feedthrough" H 11800 3814 50  0001 C CNN
-F 2 "Connector_PinSocket_2.54mm:PinSocket_1x03_P2.54mm_Vertical" V 11800 3600 50  0001 C CNN
+F 2 "d_amiga:EMI_FILTER" V 11800 3600 50  0001 C CNN
 F 3 "~" V 11800 3600 50  0001 C CNN
 	1    11800 3600
@@
 F 0 "EMI312" H 12300 3650 50  0000 C CNN
 F 1 "C_Feedthrough" H 12100 3814 50  0001 C CNN
-F 2 "Connector_PinSocket_2.54mm:PinSocket_1x03_P2.54mm_Vertical" V 12100 3600 50  0001 C CNN
+F 2 "d_amiga:EMI_FILTER" V 12100 3600 50  0001 C CNN
 F 3 "~" V 12100 3600 50  0001 C CNN
 	1    12100 3600
@@
 F 0 "EMI322" H 12600 3650 50  0000 C CNN
 F 1 "C_Feedthrough" H 12400 3814 50  0001 C CNN
-F 2 "Connector_PinSocket_2.54mm:PinSocket_1x03_P2.54mm_Vertical" V 12400 3600 50  0001 C CNN
+F 2 "d_amiga:EMI_FILTER" V 12400 3600 50  0001 C CNN
 F 3 "~" V 12400 3600 50  0001 C CNN
 	1    12400 3600
@@
 F 0 "EMI313" H 12900 3600 50  0000 C CNN
 F 1 "C_Feedthrough" H 12700 3764 50  0001 C CNN
-F 2 "Connector_PinSocket_2.54mm:PinSocket_1x03_P2.54mm_Vertical" V 12700 3550 50  0001 C CNN
+F 2 "d_amiga:EMI_FILTER" V 12700 3550 50  0001 C CNN
 F 3 "~" V 12700 3550 50  0001 C CNN
 	1    12700 3550
@@
 F 0 "EMI324" H 13200 3550 50  0000 C CNN
 F 1 "C_Feedthrough" H 13000 3714 50  0001 C CNN
-F 2 "Connector_PinSocket_2.54mm:PinSocket_1x03_P2.54mm_Vertical" V 13000 3500 50  0001 C CNN
+F 2 "d_amiga:EMI_FILTER" V 13000 3500 50  0001 C CNN
 F 3 "~" V 13000 3500 50  0001 C CNN
 	1    13000 3500
@@
 F 0 "EMI339" H 13500 3550 50  0000 C CNN
 F 1 "C_Feedthrough" H 13300 3714 50  0001 C CNN
-F 2 "Connector_PinSocket_2.54mm:PinSocket_1x03_P2.54mm_Vertical" V 13300 3500 50  0001 C CNN
+F 2 "d_amiga:EMI_FILTER" V 13300 3500 50  0001 C CNN
 F 3 "~" V 13300 3500 50  0001 C CNN
 	1    13300 3500
@@
 F 0 "EMI314" H 13800 3450 50  0000 C CNN
 F 1 "C_Feedthrough" H 13600 3614 50  0001 C CNN
-F 2 "Connector_PinSocket_2.54mm:PinSocket_1x03_P2.54mm_Vertical" V 13600 3400 50  0001 C CNN
+F 2 "d_amiga:EMI_FILTER" V 13600 3400 50  0001 C CNN
 F 3 "~" V 13600 3400 50  0001 C CNN
 	1    13600 3400
@@
 F 0 "EMI315" H 14100 3450 50  0000 C CNN
 F 1 "C_Feedthrough" H 13900 3614 50  0001 C CNN
-F 2 "Connector_PinSocket_2.54mm:PinSocket_1x03_P2.54mm_Vertical" V 13900 3400 50  0001 C CNN
+F 2 "d_amiga:EMI_FILTER" V 13900 3400 50  0001 C CNN
 F 3 "~" V 13900 3400 50  0001 C CNN
 	1    13900 3400
@@
 F 0 "EMI316" H 14400 3450 50  0000 C CNN
 F 1 "C_Feedthrough" H 14200 3614 50  0001 C CNN
-F 2 "Connector_PinSocket_2.54mm:PinSocket_1x03_P2.54mm_Vertical" V 14200 3400 50  0001 C CNN
+F 2 "d_amiga:EMI_FILTER" V 14200 3400 50  0001 C CNN
 F 3 "~" V 14200 3400 50  0001 C CNN
 	1    14200 3400
@@
 F 0 "EMI317" H 14700 3450 50  0000 C CNN
 F 1 "C_Feedthrough" H 14500 3614 50  0001 C CNN
-F 2 "Connector_PinSocket_2.54mm:PinSocket_1x03_P2.54mm_Vertical" V 14500 3400 50  0001 C CNN
+F 2 "d_amiga:EMI_FILTER" V 14500 3400 50  0001 C CNN
 F 3 "~" V 14500 3400 50  0001 C CNN
 	1    14500 3400
@@
 F 0 "EMI341" H 15000 3450 50  0000 C CNN
 F 1 "C_Feedthrough" H 14800 3614 50  0001 C CNN
-F 2 "Connector_PinSocket_2.54mm:PinSocket_1x03_P2.54mm_Vertical" V 14800 3400 50  0001 C CNN
+F 2 "d_amiga:EMI_FILTER" V 14800 3400 50  0001 C CNN
 F 3 "~" V 14800 3400 50  0001 C CNN
 	1    14800 3400
@@
 F 0 "EMI340" H 15300 3450 50  0000 C CNN
 F 1 "C_Feedthrough" H 15100 3614 50  0001 C CNN
-F 2 "Connector_PinSocket_2.54mm:PinSocket_1x03_P2.54mm_Vertical" V 15100 3400 50  0001 C CNN
+F 2 "d_amiga:EMI_FILTER" V 15100 3400 50  0001 C CNN
 F 3 "~" V 15100 3400 50  0001 C CNN
 	1    15100 3400
