File: amiga2000.kicad_pcb (KiCad board)
At the start: 2 copper layers, 416.3 x 345.8 mm, 558 parts, among them CN200 DB9P RIGHT(1), CN201 DB9P LEFT(0), CN202 DB23M, CN203 INTERNAL VIDEO SLOT TOP, CN204 RIGHT AUDIO, CN205 LEFT AUDIO, CN206 COMPOSITE, CN207 INTERNAL VIDEO SLOT BOT, CN300 KEYBOARD, CN301 DB25F, CN302 DB23F, CN303 Conn_02x17_Odd_Even, CN304 Conn_02x13_Odd_Even, CN305 DB25M, CN306 Conn_01x03_Male, CN400 POWER_CONN, CN600 CO-PROCESSOR_SLOT, CN601 zorro_socket, CN602 zorro_socket, CN603 zorro_socket, CN604 zorro_socket, CN605 zorro_socket, CN606 Conn_01x04_Male, CN700 IBM_8_BIT_EXPANSION_BUS, CN701 IBM_8_BIT_EXPANSION_BUS, CN702 IBM_8_BIT_EXPANSION_BUS, CN703 IBM_8_BIT_EXPANSION_BUS, CN704 IBM_16_BIT_EXTENDED_BUS, CN705 IBM_16_BIT_EXTENDED_BUS, CN706 IBM_16_BIT_EXTENDED_BUS, CN707 IBM_16_BIT_EXTENDED_BUS, J1 Conn_01x03_Male, J101 Conn_01x03_Male, J102 Jumper_2_Open, J2 Conn_01x03_Male, J200 Conn_01x03_Male, J3 ACCEL, J300 Conn_01x03_Male, J301 DF1:, J500 Jumper_2_Bridged, J900 Jumper_2_Bridged, Q200 MPF102, Q201 MPF102, Q202 2N3906, Q300 2SC945, Q301 2N3904, Q302 2N3906, U1 PST518B, U100 MC68000, U101 AGNUS8372, U102 GARY5719, U103 74F245, U104 74LS373, U105 74F245, U106 74LS373, U107 74LS74A, U108 74LS74A, U200 PAULA, U201 DENISE8373, U202 74LS157, U203 74LS38, U204 LF347, U205 74LS244, U206 74LS244, U300 CIA8520, U301 8520, U302 74LS32, U303 74F08, U304 1488, U305 1489, U500 62402, U501 XX4256-15, U502 XX4256-15, U503 XX4256-15, U504 XX4256-15, U505 XX4256-15, U506 XX4256-15, U507 XX4256-15, U508 XX4256-15, U540 74F244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

Commit message: Define track widths
Other:
- net class GND added: clearance 0.2, trace_width 1, via_dia 0.8, via_drill 0.4
- net class PWR added: clearance 0.2, trace_width 1.25, via_dia 0.8, via_drill 0.4
Changed lines of the file:
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@@
     (uvia_dia 0.3)
     (uvia_drill 0.1)
-    (add_net +12V)
-    (add_net +12V_USER)
-    (add_net +5V)
-    (add_net +5V_USER)
-    (add_net +AUD)
-    (add_net +AV)
-    (add_net -12V)
-    (add_net -12V_USER)
-    (add_net -5V)
-    (add_net -AV)
     (add_net /chipram/DRAB0)
     (add_net /chipram/DRAB1)
@@
     (add_net G2)
     (add_net G3)
-    (add_net GND)
-    (add_net GND_AUDIO)
     (add_net M0H)
     (add_net M0V)
@@
     (add_net _XCLKEN)
   )
+  (net_class GND ""
+    (clearance 0.2)
+    (trace_width 1)
+    (via_dia 0.8)
+    (via_drill 0.4)
+    (uvia_dia 0.3)
+    (uvia_drill 0.1)
+    (add_net GND)
+    (add_net GND_AUDIO)
+  )
+  (net_class PWR ""
+    (clearance 0.2)
+    (trace_width 1.25)
+    (via_dia 0.8)
+    (via_drill 0.4)
+    (uvia_dia 0.3)
+    (uvia_drill 0.1)
+    (add_net +12V)
+    (add_net +12V_USER)
+    (add_net +5V)
+    (add_net +5V_USER)
+    (add_net +AUD)
+    (add_net +AV)
+    (add_net -12V)
+    (add_net -12V_USER)
+    (add_net -5V)
+    (add_net -AV)
+  )
   (module Capacitor_THT:C_Rect_L11.0mm_W2.8mm_P10.00mm_MKT locked (layer F.Cu)

Commit message: Make caps footprint smaller
Parts:
- C1, C100, C101, C102, C103, C104, C105, C106, C107, C108, C110, C200, C201, C202, C203, C204, C205, C206, C210, C211, C212, C213, C215, C216, C217, C218, C219, C220, C221, C230, C231, C232, C234, C240, C241, C242, C244, C259, C260, C261, C300, C301, C302, C303, C304, C305, C306, C322, C323, C401, C407, C409, C411, C413, C414, C500, C501, C502, C503, C504, C505, C506, C507, C508, C540, C541, C600, C601, C602, C603, C604, C605, C606, C607, C617, C619, C620, C621, C622, C623, C624, C625, C626, C627, C628, C629, C630, C631, C632, C633, C635, C637, C639, C641, C645, C647, C649, C650, C651, C652, C654, C655, C657, C658, C659, C660, C661, C662, C663, C664, C665, C666, C667, C668, C669, C670, C671, C672, C673, C674, C678, C700, C702, C703, C704, C705, C711, C713, C714, C716, C717, C719, C720, C722, C726, C728, C730, C732, C734, C736, C738, C740, C742, C744, C746, C748, C750, C752, C754, C756, C758, C760, C762, C764, C766, C768, C770, C776, C778, C780, C782, C784, C786, C787, C789, C790, C791, C793, C794, C796, C800, C802, C803, C804, C805, C810, C812, C815, C900, C901, C902, C903, C904, C905, C906, C907, C908, C909, C910, C913, C914, C915, C916, C917, C918, C919, C920: footprint Capacitor_THT:C_Rect_L11.0mm_W2.8mm_P10.00mm_MKT -> Capacitor_THT:C_Rect_L11.5mm_W2.0mm_P10.00mm_MKT
- moved C713 0.08 mm to (124.8, 75.8)
- moved C711 0.08 mm to (124.8, 73.3)

Commit message: All components have been realigned; plus small sizes changes
Parts:
- F1, F2, F3, F4, F5: footprint Fuse:Fuse_Littelfuse-LVR100 -> Capacitor_THT:C_Rect_L11.5mm_W2.0mm_P10.00mm_MKT
- moved F2 13.4 mm to (238.1, 53.3), turned to 180 degrees
- moved C605 8.82 mm to (201.6, 268.6), turned to 0 degrees
- moved 217 5.14 mm to (434.7, 51.0), turned to 0 degrees
- moved 900 4.28 mm to (439.0, 47.6), turned to 180 degrees
- moved 218 4.27 mm to (430.6, 47.6), turned to 180 degrees
- moved 221 4.24 mm to (422.4, 47.6), turned to 180 degrees
- moved C204 3.67 mm to (298.3, 77.7)
- moved Q200 3.58 mm to (303.9, 85.0)
- moved R204 3.50 mm to (295.5, 87.9)
- moved R206 3.11 mm to (289.5, 87.9)
- moved R205 3.02 mm to (292.5, 87.9)
- moved C322 2.91 mm to (342.1, 57.0)
- moved R241 2.67 mm to (286.5, 87.9)
- moved C221 2.60 mm to (278.7, 77.7)
- moved C241 2.56 mm to (281.3, 87.7)
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- renumbered FB217 to 217, FB218 to 218, FB219 to 219, FB220 to 220, FB221 to 221, FB900 to 900, FB901 to 901, FB902 to 902, FB903 to 903

Commit message: Makes the DRC happy
Parts:
- EMI201, EMI206, EMI207, EMI208, EMI209, EMI210, EMI211, EMI229, EMI230, EMI231, EMI232, EMI233, EMI234, EMI235, EMI236, EMI237, EMI238, EMI239, EMI240, EMI241, EMI242, EMI243, EMI300, EMI301, EMI302, EMI303, EMI304, EMI305, EMI306, EMI307, EMI308, EMI309, EMI310, EMI311, EMI312, EMI313, EMI314, EMI315, EMI316, EMI317, EMI318, EMI319, EMI320, EMI321, EMI322, EMI323, EMI324, EMI325, EMI326, EMI327, EMI328, EMI329, EMI330, EMI331, EMI332, EMI333, EMI334, EMI335, EMI336, EMI337, EMI338, EMI339, EMI340, EMI341: footprint Connector_PinSocket_2.54mm:PinSocket_1x03_P2.54mm_Vertical -> d_amiga:EMI_FILTER
- moved C223 4.58 mm to (277.7, 58.4)
- moved FB902 1.40 mm to (426.3, 52.4)
- moved FB220 1.40 mm to (418.1, 52.4)
- moved FB217 1.40 mm to (434.7, 52.4)
- moved FB218 0.89 mm to (430.6, 48.5)
- moved FB221 0.89 mm to (422.4, 48.5)
- moved FB900 0.89 mm to (439.0, 48.5)
- moved C244 0.70 mm to (269.2, 47.0)
- moved R805 0.63 mm to (207.9, 101.9)
- moved R802 0.63 mm to (210.9, 101.9)
- moved R233 0.62 mm to (248.1, 47.1)
- moved R243 0.55 mm to (266.5, 57.2)
- moved C805 0.47 mm to (200.5, 101.9)
- moved C815 0.47 mm to (197.9, 101.9)
- moved C243 0.36 mm to (270.2, 67.5)
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- renumbered 217 to FB217, 218 to FB218, 219 to FB219, 220 to FB220, 221 to FB221, 900 to FB900, 901 to FB901, 902 to FB902, 903 to FB903

Commit message: Add explanation for jumpers
Parts:
- moved F2 39.3 mm to (199.4, 46.6), turned to 270 degrees
- moved F1 13.1 mm to (339.4, 364.1), turned to 90 degrees
- moved R804 10.2 mm to (163.4, 355.6), turned to 270 degrees
- moved R901 10.2 mm to (79.3, 229.7), turned to 180 degrees
- moved R233 10.2 mm to (247.9, 57.2), turned to 90 degrees
- moved R234 10.2 mm to (251.0, 47.1), turned to 270 degrees
- moved R308 10.2 mm to (152.4, 355.6), turned to 270 degrees
- moved R801 10.2 mm to (155.4, 355.6), turned to 270 degrees
- moved R803 10.1 mm to (212.2, 360.0), turned to 0 degrees
- moved FB102 10.1 mm to (357.5, 170.6), turned to 270 degrees
- moved C704 10.1 mm to (128.7, 69.1), turned to 180 degrees
- moved C218 10.0 mm to (331.7, 353.9), turned to 270 degrees
- moved C917 10.0 mm to (79.3, 227.0), turned to 180 degrees
- moved EMI235 5.08 mm to (354.8, 354.6), turned to 0 degrees
- moved EMI231 5.07 mm to (394.3, 354.8), turned to 0 degrees
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Other:
- board text added: "J301: closed: A2000 override drive ID of 2nd drive even if none installed. 3.5’’ work open: drive should provide ID, no 2nd drive or special HD drive 150rpm"
- board text added: "TICK source: 1-2 : from PSU CN400 PIN 14 2-3: from AGNUS"
- board text added: "Trigger mode: A1000 1-2 A500 2-3"
- board text added: "close if J101 is 1-2"
- board text added: "closed: NTSC open: PAL depends on agnus vers"
- board text added: "dflt"
- board text added: "dflt open"
- board text added: "open dflt"
