File: amiga2000.kicad_pcb (KiCad board)
At the start: 2 copper layers, 416.3 x 345.8 mm, 558 parts, among them CN200 DB9P RIGHT(1), CN201 DB9P LEFT(0), CN202 DB23M, CN203 INTERNAL VIDEO SLOT TOP, CN204 RIGHT AUDIO, CN205 LEFT AUDIO, CN206 COMPOSITE, CN207 INTERNAL VIDEO SLOT BOT, CN300 KEYBOARD, CN301 DB25F, CN302 DB23F, CN303 Conn_02x17_Odd_Even, CN304 Conn_02x13_Odd_Even, CN305 DB25M, CN306 Conn_01x03_Male, CN400 POWER_CONN, CN600 CO-PROCESSOR_SLOT, CN601 zorro_socket, CN602 zorro_socket, CN603 zorro_socket, CN604 zorro_socket, CN605 zorro_socket, CN606 Conn_01x04_Male, CN700 IBM_8_BIT_EXPANSION_BUS, CN701 IBM_8_BIT_EXPANSION_BUS, CN702 IBM_8_BIT_EXPANSION_BUS, CN703 IBM_8_BIT_EXPANSION_BUS, CN704 IBM_16_BIT_EXTENDED_BUS, CN705 IBM_16_BIT_EXTENDED_BUS, CN706 IBM_16_BIT_EXTENDED_BUS, CN707 IBM_16_BIT_EXTENDED_BUS, J1 Conn_01x03_Male, J101 Conn_01x03_Male, J102 Jumper_2_Open, J2 Conn_01x03_Male, J200 Conn_01x03_Male, J3 ACCEL, J300 Conn_01x03_Male, J301 DF1:, J500 Jumper_2_Bridged, J900 Jumper_2_Bridged, Q200 MPF102, Q201 MPF102, Q202 2N3906, Q300 2SC945, Q301 2N3904, Q302 2N3906, U1 PST518B, U100 MC68000, U101 AGNUS8372, U102 GARY5719, U103 74F245, U104 74LS373, U105 74F245, U106 74LS373, U107 74F04, U108 74LS74A, U200 PAULA, U201 DENISE8373, U202 74LS157, U203 74LS38, U204 LF347, U205 74LS244, U206 74LS244, U300 CIA8520, U301 8520, U302 74LS32, U303 74F08, U304 1488, U305 1489, U500 62402, U501 XX4256-15, U502 XX4256-15, U503 XX4256-15, U504 XX4256-15, U505 XX4256-15, U506 XX4256-15, U507 XX4256-15, U508 XX4256-15, U540 74F244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

Commit message: Switch footprints for suitable modern replacements
Parts:
- C1, C100, C101, C102, C103, C104, C105, C106, C107, C108, C110, C200, C202, C203, C205, C206, C210, C211, C212, C213, C218, C230, C231, C232, C234, C240, C241, C242, C244, C259, C260, C261, C300, C301, C302, C303, C304, C306, C322, C323, C401, C407, C409, C411, C413, C414, C540, C541, C600, C601, C602, C603, C604, C605, C606, C607, C617, C619, C620, C621, C622, C623, C624, C625, C626, C627, C628, C629, C630, C631, C632, C633, C635, C637, C639, C641, C645, C647, C649, C650, C651, C652, C654, C655, C657, C658, C659, C660, C661, C662, C663, C664, C665, C666, C667, C668, C669, C670, C671, C672, C673, C674, C678, C711, C713, C714, C716, C717, C719, C720, C722, C726, C728, C730, C732, C734, C736, C738, C740, C742, C744, C746, C748, C750, C752, C754, C756, C758, C760, C762, C764, C766, C768, C770, C776, C778, C780, C782, C784, C786, C787, C789, C790, C791, C793, C794, C796, C800, C802, C803, C804, C805, C810, C812, C815, C900, C901, C903, C904, C905, C906, C907, C908, C909, C910, C913, C914, C915, C916, C918, C919, C920: footprint Capacitor_THT:C_Rect_L11.5mm_W2.0mm_P10.00mm_MKT -> Capacitor_THT:C_Rect_L11.5mm_W2.6mm_P10.00mm_MKT
- C201, C215, C216, C217, C219, C220, C221, C500, C501, C502, C503, C504, C505, C506, C507, C508, C700, C702, C703, C704, C705: footprint Capacitor_THT:C_Rect_L11.5mm_W2.0mm_P10.00mm_MKT -> Capacitor_THT:C_Rect_L11.5mm_W4.0mm_P10.00mm_MKT
- C214: value 470uF 16v -> 470uF 16/25v; footprint Capacitor_THT:CP_Radial_D8.0mm_P5.00mm -> Capacitor_THT:CP_Radial_D10.0mm_P5.00mm
- C224, C415, C811: footprint Capacitor_THT:CP_Radial_D8.0mm_P5.00mm -> Capacitor_THT:CP_Radial_D5.0mm_P2.50mm
- C225, C226: value 470uF 16v -> 470uF 16/25v
- C233: footprint Capacitor_THT:CP_Radial_D6.3mm_P2.50mm -> Capacitor_THT:CP_Radial_D8.0mm_P5.00mm
- C310, C311, C312, C313, C314, C315, C316, C320, C321: footprint Capacitor_THT:C_Rect_L7.0mm_W2.0mm_P5.00mm -> Capacitor_THT:C_Rect_L7.0mm_W4.5mm_P5.00mm
- C416, C417, C418, C419: footprint Capacitor_THT:C_Axial_L12.0mm_D7.5mm_P20.00mm_Horizontal -> Capacitor_THT:C_Axial_L12.0mm_D8.5mm_P15.00mm_Horizontal
- C912: footprint Capacitor_THT:CP_Radial_D8.0mm_P5.00mm -> Capacitor_THT:CP_Radial_D10.0mm_P5.00mm
- X1: value 28.63636MHz -> 28.37516MHz (pal)
- Y800: footprint Crystal:Crystal_DS10_D1.0mm_L4.3mm_Horizontal -> Crystal:Crystal_DS15_D1.5mm_L5.0mm_Horizontal
- moved C412 4.96 mm to (222.1, 187.1), turned to 0 degrees
- moved C912 3.21 mm to (291.4, 344.5)
- moved C405 2.92 mm to (430.6, 240.7)
- moved C210 1.77 mm to (445.2, 197.8)
- moved C211 1.15 mm to (442.1, 197.8)
- moved Q302 0.62 mm to (141.9, 362.1)
- moved R801 0.62 mm to (154.8, 355.6)
- moved R804 0.62 mm to (162.8, 355.6)
- moved D800 0.62 mm to (157.5, 358.1)
- moved D801 0.62 mm to (160.0, 358.1)
- moved R307 0.62 mm to (148.7, 355.6)
- moved R308 0.62 mm to (151.8, 365.7)
- moved R902 0.62 mm to (145.7, 365.7)
- moved C212 0.55 mm to (439.0, 197.8)
- moved C810 0.34 mm to (165.8, 355.7)
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Connections:
- C412 pad 1: -5V -> GND
- C412 pad 2: GND -> -5V

Commit message: Some footprints updates; Add all Mouser references
Parts:
- C912: value 470uF 25v -> 470uF 16/25v
- EMI201: value C_Feedthrough -> Fitted with a double ferrite beads...
- EMI206, EMI207, EMI210, EMI211, EMI229, EMI322, EMI323, EMI324, EMI339, EMI340, EMI341: value C_Feedthrough -> 100pF (Type C 101)
- EMI208, EMI311, EMI312, EMI313, EMI314, EMI315, EMI316, EMI317, EMI318, EMI319, EMI320, EMI321: value C_Feedthrough -> 100pF (Type F 101)
- EMI209: value C_Feedthrough -> 3.8nF (Type F 382)
- EMI230, EMI231, EMI232, EMI233, EMI234, EMI235, EMI236, EMI237, EMI238, EMI239, EMI240, EMI241, EMI242, EMI243: value C_Feedthrough -> 6.8nF (Type F 682)
- EMI300, EMI301, EMI302, EMI303, EMI304, EMI305, EMI306, EMI307, EMI308, EMI309, EMI310, EMI325, EMI326, EMI327, EMI328, EMI329, EMI330, EMI331, EMI332, EMI333, EMI334, EMI335, EMI336, EMI337, EMI338: value C_Feedthrough -> 330pF (Type F 331)
- F1, F2, F3, F4, F5: value Fuse -> 4A
- RP100, RP101: value 4.7K -> 4.7k
- RP102, RP201, RP203, RP500, RP501, RP902, RP907: value 47 -> 47 (isolated, pack)
- RP204: value 68 (Dx4) -> 68 (isolated, pack)
- RP502: value 22 -> 22 (isolated, pack)
- RP802: value 1k -> 1k (isolated, pack)

Commit message: Got the components, reduce some footprints
Parts:
- C201, C215, C216, C217, C219, C220, C221, C500, C700, C702, C703, C704, C705: footprint Capacitor_THT:C_Rect_L11.5mm_W4.0mm_P10.00mm_MKT -> Capacitor_THT:C_Rect_L11.5mm_W2.6mm_P10.00mm_MKT
- C204, C305: footprint Capacitor_THT:C_Rect_L11.5mm_W2.0mm_P10.00mm_MKT -> Capacitor_THT:C_Rect_L11.5mm_W2.6mm_P10.00mm_MKT
- C222, C223, C402, C403, C404, C405, C406, C408, C410, C412, C420, C421, C422: footprint Capacitor_THT:CP_Radial_D8.0mm_P5.00mm -> Capacitor_THT:CP_Radial_Tantal_D5.5mm_P5.00mm
- C233, C243, C317, C318, C701, C813, C814: footprint Capacitor_THT:CP_Radial_D8.0mm_P5.00mm -> Capacitor_THT:CP_Radial_Tantal_D5.0mm_P5.00mm
- C310, C311, C312, C313, C314, C315, C316, C320, C321: footprint Capacitor_THT:C_Rect_L7.0mm_W4.5mm_P5.00mm -> Capacitor_THT:C_Rect_L7.0mm_W2.0mm_P5.00mm
- C400: footprint Capacitor_THT:CP_Radial_D8.0mm_P5.00mm -> Capacitor_THT:CP_Radial_Tantal_D6.0mm_P5.00mm
- C416, C417, C418, C419: footprint Capacitor_THT:C_Axial_L12.0mm_D8.5mm_P15.00mm_Horizontal -> Capacitor_THT:C_Axial_L19.0mm_D8.0mm_P25.00mm_Horizontal
- FB216, FB217, FB218, FB219, FB220, FB221, FB900, FB901, FB902, FB903: footprint Inductor_THT:L_Axial_L7.0mm_D3.3mm_P5.08mm_Vertical_Fastron_MICC -> d_amiga:FERRITE_BEADS_DOUBLE

Commit message: Some footprint changes; Tidy pcb
Parts:
- C617, C619, C620, C621, C622, C623, C624, C625, C626, C627, C628, C629, C630, C631, C632, C633, C635, C637, C639, C641, C645, C647, C649, C650, C651, C652, C654, C655, C657, C658, C659, C660, C661, C662, C663, C664, C665, C666, C667, C668, C669, C670, C671, C672, C673, C674, C678, C711, C713, C714, C716, C717, C719, C720, C722, C726, C728, C730, C732, C734, C736, C738, C740, C742, C744, C746, C748, C750, C752, C754, C756, C758, C760, C762, C764, C766, C768, C770, C776, C778, C780, C782, C784, C786, C787, C789, C790, C791, C793, C794, C796: footprint Capacitor_THT:C_Rect_L11.5mm_W2.6mm_P10.00mm_MKT -> Capacitor_THT:C_Rect_L11.5mm_W2.0mm_P10.00mm_MKT
- moved Q200 6.02 mm to (309.9, 85.0)
- moved C204 5.54 mm to (303.9, 77.5)
- moved R204 5.23 mm to (300.8, 87.7)
- moved R206 5.23 mm to (294.8, 77.5)
- moved R241 5.22 mm to (291.8, 87.7)
- moved R205 5.22 mm to (297.8, 87.7)
- moved C240 4.92 mm to (288.7, 77.7)
- moved C418 4.86 mm to (116.8, 237.7)
- moved C419 4.86 mm to (96.5, 237.7)
- moved C416 4.86 mm to (157.6, 237.7)
- moved C417 4.86 mm to (136.6, 237.7)
- moved C241 4.32 mm to (285.6, 87.7)
- moved C221 3.74 mm to (282.5, 77.7)
- moved R213 3.44 mm to (276.4, 87.7)
- moved R230 3.44 mm to (279.4, 87.7)
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