File: denise.sch (KiCad schematic (older format))
At the start: 50 parts, among them CN202 DB23M, CN203 INTERNAL VIDEO SLOT TOP, CN206 COMPOSITE, CN207 INTERNAL VIDEO SLOT BOT, U201 DENISE8373, U205 74LS244, U206 74LS244, U303 74F08

Commit message: Update footprints
Parts:
- C201, C205, C206, C215, C216, C217, C913, C914, C915: footprint (none) -> Capacitor_THT:C_Rect_L11.0mm_W2.8mm_P10.00mm_MKT
- CN203: footprint Connector_PinSocket_2.54mm:PinSocket_2x18_P2.54mm_Vertical -> d_amiga:VIDEOSLOT
- CN207: footprint (none) -> d_amiga:VIDEOSLOT
Changed lines of the file:
@@
 F 0 "CN207" V 5496 3830 50  0000 L CNN
 F 1 "INTERNAL VIDEO SLOT BOT" V 5450 750 50  0000 L CNN
-F 2 "" H 5400 2950 50  0001 C CNN
+F 2 "d_amiga:VIDEOSLOT" H 5400 2950 50  0001 C CNN
 F 3 "~" H 5400 2950 50  0001 C CNN
 	1    5400 2950
@@
 F 0 "CN203" V 9250 4179 50  0000 L CNN
 F 1 "INTERNAL VIDEO SLOT TOP" V 9205 4179 50  0001 L CNN
-F 2 "Connector_PinSocket_2.54mm:PinSocket_2x18_P2.54mm_Vertical" H 9200 3300 50  0001 C CNN
+F 2 "d_amiga:VIDEOSLOT" H 9200 3300 50  0001 C CNN
 F 3 "~" H 9200 3300 50  0001 C CNN
 	1    9200 3300
@@
 F 0 "C915" H 2715 2446 50  0000 L CNN
 F 1 "0.1uF" H 2715 2355 50  0000 L CNN
-F 2 "" H 2638 2250 50  0001 C CNN
+F 2 "Capacitor_THT:C_Rect_L11.0mm_W2.8mm_P10.00mm_MKT" H 2638 2250 50  0001 C CNN
 F 3 "~" H 2600 2400 50  0001 C CNN
 	1    2600 2400
@@
 F 0 "C913" V 10198 3200 50  0000 C CNN
 F 1 "47pF" V 10289 3200 50  0000 C CNN
-F 2 "" H 10488 3050 50  0001 C CNN
+F 2 "Capacitor_THT:C_Rect_L11.0mm_W2.8mm_P10.00mm_MKT" H 10488 3050 50  0001 C CNN
 F 3 "~" H 10450 3200 50  0001 C CNN
 	1    10450 3200
@@
 F 0 "C215" H 14615 6996 50  0000 L CNN
 F 1 "0.22uF" H 14615 6905 50  0000 L CNN
-F 2 "" H 14538 6800 50  0001 C CNN
+F 2 "Capacitor_THT:C_Rect_L11.0mm_W2.8mm_P10.00mm_MKT" H 14538 6800 50  0001 C CNN
 F 3 "~" H 14500 6950 50  0001 C CNN
 	1    14500 6950
@@
 F 0 "C216" H 14515 8096 50  0000 L CNN
 F 1 "0.22uF" H 14515 8005 50  0000 L CNN
-F 2 "" H 14438 7900 50  0001 C CNN
+F 2 "Capacitor_THT:C_Rect_L11.0mm_W2.8mm_P10.00mm_MKT" H 14438 7900 50  0001 C CNN
 F 3 "~" H 14400 8050 50  0001 C CNN
 	1    14400 8050
@@
 F 0 "C217" H 14315 8746 50  0000 L CNN
 F 1 "0.22uF" H 14315 8655 50  0000 L CNN
-F 2 "" H 14238 8550 50  0001 C CNN
+F 2 "Capacitor_THT:C_Rect_L11.0mm_W2.8mm_P10.00mm_MKT" H 14238 8550 50  0001 C CNN
 F 3 "~" H 14200 8700 50  0001 C CNN
 	1    14200 8700
@@
 F 0 "C914" H 10315 7846 50  0000 L CNN
 F 1 "100pF" H 10315 7755 50  0000 L CNN
-F 2 "" H 10238 7650 50  0001 C CNN
+F 2 "Capacitor_THT:C_Rect_L11.0mm_W2.8mm_P10.00mm_MKT" H 10238 7650 50  0001 C CNN
 F 3 "~" H 10200 7800 50  0001 C CNN
 	1    10200 7800
@@
 F 0 "C201" V 3502 8150 50  0000 C CNN
 F 1 "0.22uF" V 3411 8150 50  0000 C CNN
-F 2 "" H 3288 8000 50  0001 C CNN
+F 2 "Capacitor_THT:C_Rect_L11.0mm_W2.8mm_P10.00mm_MKT" H 3288 8000 50  0001 C CNN
 F 3 "~" H 3250 8150 50  0001 C CNN
 	1    3250 8150
@@
 F 0 "C205" V 5698 5450 50  0000 C CNN
 F 1 "0.1uF" V 5789 5450 50  0000 C CNN
-F 2 "" H 5988 5300 50  0001 C CNN
+F 2 "Capacitor_THT:C_Rect_L11.0mm_W2.8mm_P10.00mm_MKT" H 5988 5300 50  0001 C CNN
 F 3 "~" H 5950 5450 50  0001 C CNN
 	1    5950 5450
@@
 F 0 "C206" V 5698 5750 50  0000 C CNN
 F 1 "0.1uF" V 5789 5750 50  0000 C CNN
-F 2 "" H 5988 5600 50  0001 C CNN
+F 2 "Capacitor_THT:C_Rect_L11.0mm_W2.8mm_P10.00mm_MKT" H 5988 5600 50  0001 C CNN
 F 3 "~" H 5950 5750 50  0001 C CNN
 	1    5950 5750
@@
 Text GLabel 7150 5850 2    50   Input ~ 0
 +5V_USER
-Wire Bus Line
-	12050 4450 12050 4600
-Wire Bus Line
-	3400 2100 3500 2100
-Wire Bus Line
-	4200 2400 4600 2400
-Wire Bus Line
-	3750 2350 3750 2500
-Wire Bus Line
-	7950 5150 8300 5150
-Wire Bus Line
-	8100 7300 8450 7300
-Wire Bus Line
-	7350 7300 7700 7300
-Wire Bus Line
-	5800 2300 6900 2300
-Wire Bus Line
-	5800 3500 6900 3500
-Wire Bus Line
-	2450 5900 2450 6700
-Wire Bus Line
-	2450 4050 2450 5650
 Text Notes 13750 6150 1    197  ~ 0
 VIDEO
+Wire Bus Line
+	12050 4450 12050 4600
+Wire Bus Line
+	3400 2100 3500 2100
+Wire Bus Line
+	4200 2400 4600 2400
+Wire Bus Line
+	3750 2350 3750 2500
+Wire Bus Line
+	7950 5150 8300 5150
+Wire Bus Line
+	8100 7300 8450 7300
+Wire Bus Line
+	7350 7300 7700 7300
+Wire Bus Line
+	5800 2300 6900 2300
+Wire Bus Line
+	5800 3500 6900 3500
+Wire Bus Line
+	2450 5900 2450 6700
+Wire Bus Line
+	2450 4050 2450 5650
 $EndSCHEMATC

Commit message: RCA
Parts:
- CN206: footprint (none) -> d_amiga:RCA
Changed lines of the file:
@@
 F 0 "CN206" H 14250 3625 50  0000 L CNN
 F 1 "COMPOSITE" H 14250 3534 50  0000 L CNN
-F 2 "" H 14150 3650 50  0001 C CNN
+F 2 "d_amiga:RCA" H 14150 3650 50  0001 C CNN
 F 3 " ~" H 14150 3650 50  0001 C CNN
 	1    14150 3650

Commit message: Components associations finished; regenered netlist and pdf
Parts:
- CN202: footprint (none) -> d_amiga:DSUB-23_Male_Horizontal_P2.77x2.84mm_EdgePinOffset7.70mm_Housed_MountingHolesOffset9.12mm
Changed lines of the file:
@@
 F 0 "CN202" H 13022 6350 50  0000 R CNN
 F 1 "DB23M" H 13000 6250 50  0000 R CNN
-F 2 "" H 13200 6250 50  0001 C CNN
+F 2 "d_amiga:DSUB-23_Male_Horizontal_P2.77x2.84mm_EdgePinOffset7.70mm_Housed_MountingHolesOffset9.12mm" H 13200 6250 50  0001 C CNN
 F 3 " ~" H 13200 6250 50  0001 C CNN
 F 4 "Male" H 13250 6350 50  0001 C CNN "Gender"

Commit message: first placement pass is done
Parts:
- C214: footprint Capacitor_THT:CP_Radial_D10.0mm_P5.00mm -> Capacitor_THT:CP_Radial_D8.0mm_P5.00mm
Changed lines of the file:
@@
 F 0 "C214" H 11218 7396 50  0000 L CNN
 F 1 "470uF 16v" H 11218 7305 50  0000 L CNN
-F 2 "Capacitor_THT:CP_Radial_D10.0mm_P5.00mm" H 11138 7200 50  0001 C CNN
+F 2 "Capacitor_THT:CP_Radial_D8.0mm_P5.00mm" H 11138 7200 50  0001 C CNN
 F 3 "~" H 11100 7350 50  0001 C CNN
 	1    11100 7350

Commit message: Make caps footprint smaller
Parts:
- C201, C205, C206, C215, C216, C217, C913, C914, C915: footprint Capacitor_THT:C_Rect_L11.0mm_W2.8mm_P10.00mm_MKT -> Capacitor_THT:C_Rect_L11.5mm_W2.0mm_P10.00mm_MKT
Changed lines of the file:
@@
 F 0 "C915" H 2715 2446 50  0000 L CNN
 F 1 "0.1uF" H 2715 2355 50  0000 L CNN
-F 2 "Capacitor_THT:C_Rect_L11.0mm_W2.8mm_P10.00mm_MKT" H 2638 2250 50  0001 C CNN
+F 2 "Capacitor_THT:C_Rect_L11.5mm_W2.0mm_P10.00mm_MKT" H 2638 2250 50  0001 C CNN
 F 3 "~" H 2600 2400 50  0001 C CNN
 	1    2600 2400
@@
 F 0 "C913" V 10198 3200 50  0000 C CNN
 F 1 "47pF" V 10289 3200 50  0000 C CNN
-F 2 "Capacitor_THT:C_Rect_L11.0mm_W2.8mm_P10.00mm_MKT" H 10488 3050 50  0001 C CNN
+F 2 "Capacitor_THT:C_Rect_L11.5mm_W2.0mm_P10.00mm_MKT" H 10488 3050 50  0001 C CNN
 F 3 "~" H 10450 3200 50  0001 C CNN
 	1    10450 3200
@@
 F 0 "C215" H 14615 6996 50  0000 L CNN
 F 1 "0.22uF" H 14615 6905 50  0000 L CNN
-F 2 "Capacitor_THT:C_Rect_L11.0mm_W2.8mm_P10.00mm_MKT" H 14538 6800 50  0001 C CNN
+F 2 "Capacitor_THT:C_Rect_L11.5mm_W2.0mm_P10.00mm_MKT" H 14538 6800 50  0001 C CNN
 F 3 "~" H 14500 6950 50  0001 C CNN
 	1    14500 6950
@@
 F 0 "C216" H 14515 8096 50  0000 L CNN
 F 1 "0.22uF" H 14515 8005 50  0000 L CNN
-F 2 "Capacitor_THT:C_Rect_L11.0mm_W2.8mm_P10.00mm_MKT" H 14438 7900 50  0001 C CNN
+F 2 "Capacitor_THT:C_Rect_L11.5mm_W2.0mm_P10.00mm_MKT" H 14438 7900 50  0001 C CNN
 F 3 "~" H 14400 8050 50  0001 C CNN
 	1    14400 8050
@@
 F 0 "C217" H 14315 8746 50  0000 L CNN
 F 1 "0.22uF" H 14315 8655 50  0000 L CNN
-F 2 "Capacitor_THT:C_Rect_L11.0mm_W2.8mm_P10.00mm_MKT" H 14238 8550 50  0001 C CNN
+F 2 "Capacitor_THT:C_Rect_L11.5mm_W2.0mm_P10.00mm_MKT" H 14238 8550 50  0001 C CNN
 F 3 "~" H 14200 8700 50  0001 C CNN
 	1    14200 8700
@@
 F 0 "C914" H 10315 7846 50  0000 L CNN
 F 1 "100pF" H 10315 7755 50  0000 L CNN
-F 2 "Capacitor_THT:C_Rect_L11.0mm_W2.8mm_P10.00mm_MKT" H 10238 7650 50  0001 C CNN
+F 2 "Capacitor_THT:C_Rect_L11.5mm_W2.0mm_P10.00mm_MKT" H 10238 7650 50  0001 C CNN
 F 3 "~" H 10200 7800 50  0001 C CNN
 	1    10200 7800
@@
 F 0 "C201" V 3502 8150 50  0000 C CNN
 F 1 "0.22uF" V 3411 8150 50  0000 C CNN
-F 2 "Capacitor_THT:C_Rect_L11.0mm_W2.8mm_P10.00mm_MKT" H 3288 8000 50  0001 C CNN
+F 2 "Capacitor_THT:C_Rect_L11.5mm_W2.0mm_P10.00mm_MKT" H 3288 8000 50  0001 C CNN
 F 3 "~" H 3250 8150 50  0001 C CNN
 	1    3250 8150
@@
 F 0 "C205" V 5698 5450 50  0000 C CNN
 F 1 "0.1uF" V 5789 5450 50  0000 C CNN
-F 2 "Capacitor_THT:C_Rect_L11.0mm_W2.8mm_P10.00mm_MKT" H 5988 5300 50  0001 C CNN
+F 2 "Capacitor_THT:C_Rect_L11.5mm_W2.0mm_P10.00mm_MKT" H 5988 5300 50  0001 C CNN
 F 3 "~" H 5950 5450 50  0001 C CNN
 	1    5950 5450
@@
 F 0 "C206" V 5698 5750 50  0000 C CNN
 F 1 "0.1uF" V 5789 5750 50  0000 C CNN
-F 2 "Capacitor_THT:C_Rect_L11.0mm_W2.8mm_P10.00mm_MKT" H 5988 5600 50  0001 C CNN
+F 2 "Capacitor_THT:C_Rect_L11.5mm_W2.0mm_P10.00mm_MKT" H 5988 5600 50  0001 C CNN
 F 3 "~" H 5950 5750 50  0001 C CNN
 	1    5950 5750

Commit message: All components have been realigned; plus small sizes changes
Parts:
- F5: footprint Fuse:Fuse_Littelfuse-LVR100 -> Capacitor_THT:C_Rect_L11.5mm_W2.0mm_P10.00mm_MKT
Changed lines of the file:
@@
 F 0 "F5" V 14045 7900 50  0000 C CNN
 F 1 "Fuse" V 14044 7900 50  0001 C CNN
-F 2 "Fuse:Fuse_Littelfuse-LVR100" V 14080 7900 50  0001 C CNN
+F 2 "Capacitor_THT:C_Rect_L11.5mm_W2.0mm_P10.00mm_MKT" V 14080 7900 50  0001 C CNN
 F 3 "~" H 14150 7900 50  0001 C CNN
 	1    14150 7900

Commit message: Makes the DRC happy
Parts:
- EMI201, EMI206, EMI207, EMI208, EMI209, EMI210, EMI211, EMI229: footprint Connector_PinSocket_2.54mm:PinSocket_1x03_P2.54mm_Vertical -> d_amiga:EMI_FILTER
Changed lines of the file:
@@
 F 0 "EMI201" H 11300 3463 50  0000 C CNN
 F 1 "C_Feedthrough" H 11300 3464 50  0001 C CNN
-F 2 "Connector_PinSocket_2.54mm:PinSocket_1x03_P2.54mm_Vertical" V 11300 3250 50  0001 C CNN
+F 2 "d_amiga:EMI_FILTER" V 11300 3250 50  0001 C CNN
 F 3 "~" V 11300 3250 50  0001 C CNN
 	1    11300 3250
@@
 F 0 "EMI208" H 13750 3963 50  0000 C CNN
 F 1 "C_Feedthrough" H 13750 3964 50  0001 C CNN
-F 2 "Connector_PinSocket_2.54mm:PinSocket_1x03_P2.54mm_Vertical" V 13750 3750 50  0001 C CNN
+F 2 "d_amiga:EMI_FILTER" V 13750 3750 50  0001 C CNN
 F 3 "~" V 13750 3750 50  0001 C CNN
 	1    13750 3750
@@
 F 0 "EMI206" H 12300 7350 50  0000 C CNN
 F 1 "C_Feedthrough" H 12200 7564 50  0001 C CNN
-F 2 "Connector_PinSocket_2.54mm:PinSocket_1x03_P2.54mm_Vertical" V 12200 7350 50  0001 C CNN
+F 2 "d_amiga:EMI_FILTER" V 12200 7350 50  0001 C CNN
 F 3 "~" V 12200 7350 50  0001 C CNN
 	1    12200 7350
@@
 F 0 "EMI207" H 12400 7600 50  0000 C CNN
 F 1 "C_Feedthrough" H 12300 7814 50  0001 C CNN
-F 2 "Connector_PinSocket_2.54mm:PinSocket_1x03_P2.54mm_Vertical" V 12300 7600 50  0001 C CNN
+F 2 "d_amiga:EMI_FILTER" V 12300 7600 50  0001 C CNN
 F 3 "~" V 12300 7600 50  0001 C CNN
 	1    12300 7600
@@
 F 0 "EMI209" H 13800 8813 50  0000 C CNN
 F 1 "C_Feedthrough" H 13800 8814 50  0001 C CNN
-F 2 "Connector_PinSocket_2.54mm:PinSocket_1x03_P2.54mm_Vertical" V 13800 8600 50  0001 C CNN
+F 2 "d_amiga:EMI_FILTER" V 13800 8600 50  0001 C CNN
 F 3 "~" V 13800 8600 50  0001 C CNN
 	1    13800 8600
@@
 F 0 "EMI229" H 2400 8263 50  0000 C CNN
 F 1 "C_Feedthrough" H 2400 8264 50  0001 C CNN
-F 2 "Connector_PinSocket_2.54mm:PinSocket_1x03_P2.54mm_Vertical" V 2400 8050 50  0001 C CNN
+F 2 "d_amiga:EMI_FILTER" V 2400 8050 50  0001 C CNN
 F 3 "~" V 2400 8050 50  0001 C CNN
 	1    2400 8050
@@
 F 0 "EMI210" H 13800 8213 50  0000 C CNN
 F 1 "C_Feedthrough" H 13800 8214 50  0001 C CNN
-F 2 "Connector_PinSocket_2.54mm:PinSocket_1x03_P2.54mm_Vertical" V 13800 8000 50  0001 C CNN
+F 2 "d_amiga:EMI_FILTER" V 13800 8000 50  0001 C CNN
 F 3 "~" V 13800 8000 50  0001 C CNN
 	1    13800 8000
@@
 F 0 "EMI211" H 14150 7363 50  0000 C CNN
 F 1 "C_Feedthrough" H 14150 7364 50  0001 C CNN
-F 2 "Connector_PinSocket_2.54mm:PinSocket_1x03_P2.54mm_Vertical" V 14150 7150 50  0001 C CNN
+F 2 "d_amiga:EMI_FILTER" V 14150 7150 50  0001 C CNN
 F 3 "~" V 14150 7150 50  0001 C CNN
 	1    14150 7150

Commit message: Add DoNotPopulate field for components which shouldn't be fitted
Parts:
- RP904, RP905, RP906: DoNotPopulate (none) -> yes
Changed lines of the file:
@@
 F 2 "Resistor_THT:R_Array_SIP6" V 4625 8300 50  0001 C CNN
 F 3 "http://www.vishay.com/docs/31509/csc.pdf" H 4250 8300 50  0001 C CNN
+F 4 "yes" H 4250 8300 50  0001 C CNN "DoNotPopulate"
 	1    4250 8300
 	-1   0    0    1
@@
 F 2 "Resistor_THT:R_Array_SIP6" V 5175 8300 50  0001 C CNN
 F 3 "http://www.vishay.com/docs/31509/csc.pdf" H 4800 8300 50  0001 C CNN
+F 4 "yes" H 4800 8300 50  0001 C CNN "DoNotPopulate"
 	1    4800 8300
 	1    0    0    1
@@
 F 2 "Resistor_THT:R_Array_SIP6" V 5825 8300 50  0001 C CNN
 F 3 "http://www.vishay.com/docs/31509/csc.pdf" H 5450 8300 50  0001 C CNN
+F 4 "yes" H 5450 8300 50  0001 C CNN "DoNotPopulate"
 	1    5450 8300
 	1    0    0    1
